File: can-transceiver.kicad_sch (KiCad schematic)
At the start: 4 parts, among them U6 TJA1044GTK_3Z

Commit message: Add HVSON83x3 library with 3d model
Parts:
- U4: renamed from U6; footprint Package_SON:HVSON-8-1EP_3x3mm_P0.65mm_EP1.6x2.4mm -> HVSON-8-EP(3x3):HVSON-8-1EP_3x3mm_P0.65mm_EP1.6x2.4mm
- renumbered C21 to C17, C22 to C18, R24 to R22
Changed lines of the file:
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@@
 		(on_board yes)
 		(dnp no)
-		(property "Reference" "#PWR055"
+		(property "Reference" "#PWR043"
 			(at 163.83 93.98 0)
 			(effects
@@
 			(project "base-module"
 				(path "/090a8e41-87a8-4fb1-998b-60a2c0dc4cee/ae074854-c02c-496b-964f-ecb8956e53f8/7ee3192a-2c17-43bb-b41c-3a68ad8e606c"
-					(reference "#PWR055")
-					(unit 1)
-				)
-				(path "/090a8e41-87a8-4fb1-998b-60a2c0dc4cee/ae074854-c02c-496b-964f-ecb8956e53f8/9aa56239-1a3a-4aac-8799-c057bacf336d"
-					(reference "#PWR061")
+					(reference "#PWR043")
+					(unit 1)
+				)
+				(path "/090a8e41-87a8-4fb1-998b-60a2c0dc4cee/ae074854-c02c-496b-964f-ecb8956e53f8/9aa56239-1a3a-4aac-8799-c057bacf336d"
+					(reference "#PWR049")
 					(unit 1)
 				)
@@
 		(on_board yes)
 		(dnp no)
-		(property "Reference" "C22"
+		(property "Reference" "C18"
 			(at 172.72 91.44 90)
 			(effects
@@
 			(project "base-module"
 				(path "/090a8e41-87a8-4fb1-998b-60a2c0dc4cee/ae074854-c02c-496b-964f-ecb8956e53f8/7ee3192a-2c17-43bb-b41c-3a68ad8e606c"
-					(reference "C22")
-					(unit 1)
-				)
-				(path "/090a8e41-87a8-4fb1-998b-60a2c0dc4cee/ae074854-c02c-496b-964f-ecb8956e53f8/9aa56239-1a3a-4aac-8799-c057bacf336d"
-					(reference "C24")
+					(reference "C18")
+					(unit 1)
+				)
+				(path "/090a8e41-87a8-4fb1-998b-60a2c0dc4cee/ae074854-c02c-496b-964f-ecb8956e53f8/9aa56239-1a3a-4aac-8799-c057bacf336d"
+					(reference "C20")
 					(unit 1)
 				)
@@
 		(on_board yes)
 		(dnp no)
-		(property "Reference" "U6"
+		(property "Reference" "U4"
 			(at 151.13 89.535 0)
 			(effects
@@
 			)
 		)
-		(property "Footprint" "Package_SON:HVSON-8-1EP_3x3mm_P0.65mm_EP1.6x2.4mm"
+		(property "Footprint" "HVSON-8-EP(3x3):HVSON-8-1EP_3x3mm_P0.65mm_EP1.6x2.4mm"
 			(at 165.1 191.44 0)
 			(effects
@@
 			(project "base-module"
 				(path "/090a8e41-87a8-4fb1-998b-60a2c0dc4cee/ae074854-c02c-496b-964f-ecb8956e53f8/7ee3192a-2c17-43bb-b41c-3a68ad8e606c"
-					(reference "U6")
-					(unit 1)
-				)
-				(path "/090a8e41-87a8-4fb1-998b-60a2c0dc4cee/ae074854-c02c-496b-964f-ecb8956e53f8/9aa56239-1a3a-4aac-8799-c057bacf336d"
-					(reference "U7")
+					(reference "U4")
+					(unit 1)
+				)
+				(path "/090a8e41-87a8-4fb1-998b-60a2c0dc4cee/ae074854-c02c-496b-964f-ecb8956e53f8/9aa56239-1a3a-4aac-8799-c057bacf336d"
+					(reference "U5")
 					(unit 1)
 				)
@@
 		(on_board yes)
 		(dnp no)
-		(property "Reference" "#PWR054"
+		(property "Reference" "#PWR042"
 			(at 138.43 93.98 0)
 			(effects
@@
 			(project "base-module"
 				(path "/090a8e41-87a8-4fb1-998b-60a2c0dc4cee/ae074854-c02c-496b-964f-ecb8956e53f8/7ee3192a-2c17-43bb-b41c-3a68ad8e606c"
-					(reference "#PWR054")
-					(unit 1)
-				)
-				(path "/090a8e41-87a8-4fb1-998b-60a2c0dc4cee/ae074854-c02c-496b-964f-ecb8956e53f8/9aa56239-1a3a-4aac-8799-c057bacf336d"
-					(reference "#PWR060")
+					(reference "#PWR042")
+					(unit 1)
+				)
+				(path "/090a8e41-87a8-4fb1-998b-60a2c0dc4cee/ae074854-c02c-496b-964f-ecb8956e53f8/9aa56239-1a3a-4aac-8799-c057bacf336d"
+					(reference "#PWR048")
 					(unit 1)
 				)
@@
 		(on_board yes)
 		(dnp no)
-		(property "Reference" "R24"
+		(property "Reference" "R22"
 			(at 165.1 111.76 0)
 			(effects
@@
 			(project "base-module"
 				(path "/090a8e41-87a8-4fb1-998b-60a2c0dc4cee/ae074854-c02c-496b-964f-ecb8956e53f8/7ee3192a-2c17-43bb-b41c-3a68ad8e606c"
-					(reference "R24")
-					(unit 1)
-				)
-				(path "/090a8e41-87a8-4fb1-998b-60a2c0dc4cee/ae074854-c02c-496b-964f-ecb8956e53f8/9aa56239-1a3a-4aac-8799-c057bacf336d"
-					(reference "R25")
+					(reference "R22")
+					(unit 1)
+				)
+				(path "/090a8e41-87a8-4fb1-998b-60a2c0dc4cee/ae074854-c02c-496b-964f-ecb8956e53f8/9aa56239-1a3a-4aac-8799-c057bacf336d"
+					(reference "R23")
 					(unit 1)
 				)
@@
 		(on_board yes)
 		(dnp no)
-		(property "Reference" "#PWR056"
+		(property "Reference" "#PWR044"
 			(at 125.73 100.33 0)
 			(effects
@@
 			(project "base-module"
 				(path "/090a8e41-87a8-4fb1-998b-60a2c0dc4cee/ae074854-c02c-496b-964f-ecb8956e53f8/7ee3192a-2c17-43bb-b41c-3a68ad8e606c"
-					(reference "#PWR056")
-					(unit 1)
-				)
-				(path "/090a8e41-87a8-4fb1-998b-60a2c0dc4cee/ae074854-c02c-496b-964f-ecb8956e53f8/9aa56239-1a3a-4aac-8799-c057bacf336d"
-					(reference "#PWR062")
+					(reference "#PWR044")
+					(unit 1)
+				)
+				(path "/090a8e41-87a8-4fb1-998b-60a2c0dc4cee/ae074854-c02c-496b-964f-ecb8956e53f8/9aa56239-1a3a-4aac-8799-c057bacf336d"
+					(reference "#PWR050")
 					(unit 1)
 				)
@@
 		(on_board yes)
 		(dnp no)
-		(property "Reference" "#PWR059"
+		(property "Reference" "#PWR047"
 			(at 163.83 123.19 0)
 			(effects
@@
 			(project "base-module"
 				(path "/090a8e41-87a8-4fb1-998b-60a2c0dc4cee/ae074854-c02c-496b-964f-ecb8956e53f8/7ee3192a-2c17-43bb-b41c-3a68ad8e606c"
-					(reference "#PWR059")
-					(unit 1)
-				)
-				(path "/090a8e41-87a8-4fb1-998b-60a2c0dc4cee/ae074854-c02c-496b-964f-ecb8956e53f8/9aa56239-1a3a-4aac-8799-c057bacf336d"
-					(reference "#PWR065")
+					(reference "#PWR047")
+					(unit 1)
+				)
+				(path "/090a8e41-87a8-4fb1-998b-60a2c0dc4cee/ae074854-c02c-496b-964f-ecb8956e53f8/9aa56239-1a3a-4aac-8799-c057bacf336d"
+					(reference "#PWR053")
 					(unit 1)
 				)
@@
 		(on_board yes)
 		(dnp no)
-		(property "Reference" "C21"
+		(property "Reference" "C17"
 			(at 129.54 91.44 90)
 			(effects
@@
 			(project "base-module"
 				(path "/090a8e41-87a8-4fb1-998b-60a2c0dc4cee/ae074854-c02c-496b-964f-ecb8956e53f8/7ee3192a-2c17-43bb-b41c-3a68ad8e606c"
-					(reference "C21")
-					(unit 1)
-				)
-				(path "/090a8e41-87a8-4fb1-998b-60a2c0dc4cee/ae074854-c02c-496b-964f-ecb8956e53f8/9aa56239-1a3a-4aac-8799-c057bacf336d"
-					(reference "C23")
+					(reference "C17")
+					(unit 1)
+				)
+				(path "/090a8e41-87a8-4fb1-998b-60a2c0dc4cee/ae074854-c02c-496b-964f-ecb8956e53f8/9aa56239-1a3a-4aac-8799-c057bacf336d"
+					(reference "C19")
 					(unit 1)
 				)
@@
 		(on_board yes)
 		(dnp no)
-		(property "Reference" "#PWR057"
+		(property "Reference" "#PWR045"
 			(at 176.53 100.33 0)
 			(effects
@@
 			(project "base-module"
 				(path "/090a8e41-87a8-4fb1-998b-60a2c0dc4cee/ae074854-c02c-496b-964f-ecb8956e53f8/7ee3192a-2c17-43bb-b41c-3a68ad8e606c"
-					(reference "#PWR057")
-					(unit 1)
-				)
-				(path "/090a8e41-87a8-4fb1-998b-60a2c0dc4cee/ae074854-c02c-496b-964f-ecb8956e53f8/9aa56239-1a3a-4aac-8799-c057bacf336d"
-					(reference "#PWR063")
+					(reference "#PWR045")
+					(unit 1)
+				)
+				(path "/090a8e41-87a8-4fb1-998b-60a2c0dc4cee/ae074854-c02c-496b-964f-ecb8956e53f8/9aa56239-1a3a-4aac-8799-c057bacf336d"
+					(reference "#PWR051")
 					(unit 1)
 				)
@@
 		(on_board yes)
 		(dnp no)
-		(property "Reference" "#PWR058"
+		(property "Reference" "#PWR046"
 			(at 138.43 123.19 0)
 			(effects
@@
 			(project "base-module"
 				(path "/090a8e41-87a8-4fb1-998b-60a2c0dc4cee/ae074854-c02c-496b-964f-ecb8956e53f8/7ee3192a-2c17-43bb-b41c-3a68ad8e606c"
-					(reference "#PWR058")
-					(unit 1)
-				)
-				(path "/090a8e41-87a8-4fb1-998b-60a2c0dc4cee/ae074854-c02c-496b-964f-ecb8956e53f8/9aa56239-1a3a-4aac-8799-c057bacf336d"
-					(reference "#PWR064")
-					(unit 1)
-				)
+					(reference "#PWR046")
+					(unit 1)
+				)
+				(path "/090a8e41-87a8-4fb1-998b-60a2c0dc4cee/ae074854-c02c-496b-964f-ecb8956e53f8/9aa56239-1a3a-4aac-8799-c057bacf336d"
+					(reference "#PWR052")
+					(unit 1)
+				)

Commit message: [#3] Annotate power and CAN transceiver sheets
Parts:
- renumbered C17 to C501, C18 to C502, R22 to R501, U4 to U501
Other:
- note added: "CAN TRANSCEIVER"
Changed lines of the file:
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@@
+		)
+	)
+	(text "CAN TRANSCEIVER"
+		(exclude_from_sim no)
+		(at 149.86 76.835 0)
+		(effects
+			(font
+				(size 2.54 2.54)
+				(thickness 0.508)
+				(bold yes)
+			)
 		)
 	)
@@
 		(on_board yes)
 		(dnp no)
-		(property "Reference" "#PWR043"
+		(property "Reference" "#PWR0502"
 			(at 163.83 93.98 0)
 			(effects
@@
 			(project "base-module"
 				(path "/090a8e41-87a8-4fb1-998b-60a2c0dc4cee/ae074854-c02c-496b-964f-ecb8956e53f8/7ee3192a-2c17-43bb-b41c-3a68ad8e606c"
-					(reference "#PWR043")
-					(unit 1)
-				)
-				(path "/090a8e41-87a8-4fb1-998b-60a2c0dc4cee/ae074854-c02c-496b-964f-ecb8956e53f8/9aa56239-1a3a-4aac-8799-c057bacf336d"
-					(reference "#PWR049")
+					(reference "#PWR0502")
+					(unit 1)
+				)
+				(path "/090a8e41-87a8-4fb1-998b-60a2c0dc4cee/ae074854-c02c-496b-964f-ecb8956e53f8/9aa56239-1a3a-4aac-8799-c057bacf336d"
+					(reference "#PWR0608")
 					(unit 1)
 				)
@@
 		(on_board yes)
 		(dnp no)
-		(property "Reference" "C18"
+		(property "Reference" "C502"
 			(at 172.72 91.44 90)
 			(effects
@@
 			(project "base-module"
 				(path "/090a8e41-87a8-4fb1-998b-60a2c0dc4cee/ae074854-c02c-496b-964f-ecb8956e53f8/7ee3192a-2c17-43bb-b41c-3a68ad8e606c"
-					(reference "C18")
-					(unit 1)
-				)
-				(path "/090a8e41-87a8-4fb1-998b-60a2c0dc4cee/ae074854-c02c-496b-964f-ecb8956e53f8/9aa56239-1a3a-4aac-8799-c057bacf336d"
-					(reference "C20")
+					(reference "C502")
+					(unit 1)
+				)
+				(path "/090a8e41-87a8-4fb1-998b-60a2c0dc4cee/ae074854-c02c-496b-964f-ecb8956e53f8/9aa56239-1a3a-4aac-8799-c057bacf336d"
+					(reference "C604")
 					(unit 1)
 				)
@@
 		(on_board yes)
 		(dnp no)
-		(property "Reference" "U4"
+		(property "Reference" "U501"
 			(at 151.13 89.535 0)
 			(effects
@@
 			(project "base-module"
 				(path "/090a8e41-87a8-4fb1-998b-60a2c0dc4cee/ae074854-c02c-496b-964f-ecb8956e53f8/7ee3192a-2c17-43bb-b41c-3a68ad8e606c"
-					(reference "U4")
-					(unit 1)
-				)
-				(path "/090a8e41-87a8-4fb1-998b-60a2c0dc4cee/ae074854-c02c-496b-964f-ecb8956e53f8/9aa56239-1a3a-4aac-8799-c057bacf336d"
-					(reference "U5")
+					(reference "U501")
+					(unit 1)
+				)
+				(path "/090a8e41-87a8-4fb1-998b-60a2c0dc4cee/ae074854-c02c-496b-964f-ecb8956e53f8/9aa56239-1a3a-4aac-8799-c057bacf336d"
+					(reference "U602")
 					(unit 1)
 				)
@@
 		(on_board yes)
 		(dnp no)
-		(property "Reference" "#PWR042"
+		(property "Reference" "#PWR0501"
 			(at 138.43 93.98 0)
 			(effects
@@
 			(project "base-module"
 				(path "/090a8e41-87a8-4fb1-998b-60a2c0dc4cee/ae074854-c02c-496b-964f-ecb8956e53f8/7ee3192a-2c17-43bb-b41c-3a68ad8e606c"
-					(reference "#PWR042")
-					(unit 1)
-				)
-				(path "/090a8e41-87a8-4fb1-998b-60a2c0dc4cee/ae074854-c02c-496b-964f-ecb8956e53f8/9aa56239-1a3a-4aac-8799-c057bacf336d"
-					(reference "#PWR048")
+					(reference "#PWR0501")
+					(unit 1)
+				)
+				(path "/090a8e41-87a8-4fb1-998b-60a2c0dc4cee/ae074854-c02c-496b-964f-ecb8956e53f8/9aa56239-1a3a-4aac-8799-c057bacf336d"
+					(reference "#PWR0607")
 					(unit 1)
 				)
@@
 		(on_board yes)
 		(dnp no)
-		(property "Reference" "R22"
+		(property "Reference" "R501"
 			(at 165.1 111.76 0)
 			(effects
@@
 			(project "base-module"
 				(path "/090a8e41-87a8-4fb1-998b-60a2c0dc4cee/ae074854-c02c-496b-964f-ecb8956e53f8/7ee3192a-2c17-43bb-b41c-3a68ad8e606c"
-					(reference "R22")
-					(unit 1)
-				)
-				(path "/090a8e41-87a8-4fb1-998b-60a2c0dc4cee/ae074854-c02c-496b-964f-ecb8956e53f8/9aa56239-1a3a-4aac-8799-c057bacf336d"
-					(reference "R23")
+					(reference "R501")
+					(unit 1)
+				)
+				(path "/090a8e41-87a8-4fb1-998b-60a2c0dc4cee/ae074854-c02c-496b-964f-ecb8956e53f8/9aa56239-1a3a-4aac-8799-c057bacf336d"
+					(reference "R602")
 					(unit 1)
 				)
@@
 		(on_board yes)
 		(dnp no)
-		(property "Reference" "#PWR044"
+		(property "Reference" "#PWR0503"
 			(at 125.73 100.33 0)
 			(effects
@@
 			(project "base-module"
 				(path "/090a8e41-87a8-4fb1-998b-60a2c0dc4cee/ae074854-c02c-496b-964f-ecb8956e53f8/7ee3192a-2c17-43bb-b41c-3a68ad8e606c"
-					(reference "#PWR044")
-					(unit 1)
-				)
-				(path "/090a8e41-87a8-4fb1-998b-60a2c0dc4cee/ae074854-c02c-496b-964f-ecb8956e53f8/9aa56239-1a3a-4aac-8799-c057bacf336d"
-					(reference "#PWR050")
+					(reference "#PWR0503")
+					(unit 1)
+				)
+				(path "/090a8e41-87a8-4fb1-998b-60a2c0dc4cee/ae074854-c02c-496b-964f-ecb8956e53f8/9aa56239-1a3a-4aac-8799-c057bacf336d"
+					(reference "#PWR0609")
 					(unit 1)
 				)
@@
 		(on_board yes)
 		(dnp no)
-		(property "Reference" "#PWR047"
+		(property "Reference" "#PWR0506"
 			(at 163.83 123.19 0)
 			(effects
@@
 			(project "base-module"
 				(path "/090a8e41-87a8-4fb1-998b-60a2c0dc4cee/ae074854-c02c-496b-964f-ecb8956e53f8/7ee3192a-2c17-43bb-b41c-3a68ad8e606c"
-					(reference "#PWR047")
-					(unit 1)
-				)
-				(path "/090a8e41-87a8-4fb1-998b-60a2c0dc4cee/ae074854-c02c-496b-964f-ecb8956e53f8/9aa56239-1a3a-4aac-8799-c057bacf336d"
-					(reference "#PWR053")
+					(reference "#PWR0506")
+					(unit 1)
+				)
+				(path "/090a8e41-87a8-4fb1-998b-60a2c0dc4cee/ae074854-c02c-496b-964f-ecb8956e53f8/9aa56239-1a3a-4aac-8799-c057bacf336d"
+					(reference "#PWR0612")
 					(unit 1)
 				)
@@
 		(on_board yes)
 		(dnp no)
-		(property "Reference" "C17"
+		(property "Reference" "C501"
 			(at 129.54 91.44 90)
 			(effects
@@
 			(project "base-module"
 				(path "/090a8e41-87a8-4fb1-998b-60a2c0dc4cee/ae074854-c02c-496b-964f-ecb8956e53f8/7ee3192a-2c17-43bb-b41c-3a68ad8e606c"
-					(reference "C17")
-					(unit 1)
-				)
-				(path "/090a8e41-87a8-4fb1-998b-60a2c0dc4cee/ae074854-c02c-496b-964f-ecb8956e53f8/9aa56239-1a3a-4aac-8799-c057bacf336d"
-					(reference "C19")
+					(reference "C501")
+					(unit 1)
+				)
+				(path "/090a8e41-87a8-4fb1-998b-60a2c0dc4cee/ae074854-c02c-496b-964f-ecb8956e53f8/9aa56239-1a3a-4aac-8799-c057bacf336d"
+					(reference "C603")
 					(unit 1)
 				)
@@
 		(on_board yes)
 		(dnp no)
-		(property "Reference" "#PWR045"
+		(property "Reference" "#PWR0504"
 			(at 176.53 100.33 0)
 			(effects
@@
 			(project "base-module"
 				(path "/090a8e41-87a8-4fb1-998b-60a2c0dc4cee/ae074854-c02c-496b-964f-ecb8956e53f8/7ee3192a-2c17-43bb-b41c-3a68ad8e606c"
-					(reference "#PWR045")
-					(unit 1)
-				)
-				(path "/090a8e41-87a8-4fb1-998b-60a2c0dc4cee/ae074854-c02c-496b-964f-ecb8956e53f8/9aa56239-1a3a-4aac-8799-c057bacf336d"
-					(reference "#PWR051")
+					(reference "#PWR0504")
+					(unit 1)
+				)
+				(path "/090a8e41-87a8-4fb1-998b-60a2c0dc4cee/ae074854-c02c-496b-964f-ecb8956e53f8/9aa56239-1a3a-4aac-8799-c057bacf336d"
+					(reference "#PWR0610")
 					(unit 1)
 				)
@@
 		(on_board yes)
 		(dnp no)
-		(property "Reference" "#PWR046"
+		(property "Reference" "#PWR0505"
 			(at 138.43 123.19 0)
 			(effects
@@
 			(project "base-module"
 				(path "/090a8e41-87a8-4fb1-998b-60a2c0dc4cee/ae074854-c02c-496b-964f-ecb8956e53f8/7ee3192a-2c17-43bb-b41c-3a68ad8e606c"
-					(reference "#PWR046")
-					(unit 1)
-				)
-				(path "/090a8e41-87a8-4fb1-998b-60a2c0dc4cee/ae074854-c02c-496b-964f-ecb8956e53f8/9aa56239-1a3a-4aac-8799-c057bacf336d"
-					(reference "#PWR052")
-					(unit 1)
-				)
+					(reference "#PWR0505")
+					(unit 1)
+				)
+				(path "/090a8e41-87a8-4fb1-998b-60a2c0dc4cee/ae074854-c02c-496b-964f-ecb8956e53f8/9aa56239-1a3a-4aac-8799-c057bacf336d"
+					(reference "#PWR0611")
+					(unit 1)
+				)
