File: can-transceiver.kicad_sch (KiCad schematic)
At the start: 4 parts, among them U4 TJA1044GTK_3Z

Commit message: Add usb schematic
Parts:
- renumbered C17 to C501, C18 to C502, R22 to R501, U4 to U501
Other:
- note added: "CAN TRANSCEIVER"
Changed lines of the file:
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@@
+		)
+	)
+	(text "CAN TRANSCEIVER"
+		(exclude_from_sim no)
+		(at 149.86 76.835 0)
+		(effects
+			(font
+				(size 2.54 2.54)
+				(thickness 0.508)
+				(bold yes)
+			)
 		)
 	)
@@
 		(on_board yes)
 		(dnp no)
-		(property "Reference" "#PWR043"
+		(property "Reference" "#PWR0502"
 			(at 163.83 93.98 0)
 			(effects
@@
 			(project "base-module"
 				(path "/090a8e41-87a8-4fb1-998b-60a2c0dc4cee/ae074854-c02c-496b-964f-ecb8956e53f8/7ee3192a-2c17-43bb-b41c-3a68ad8e606c"
-					(reference "#PWR043")
-					(unit 1)
-				)
-				(path "/090a8e41-87a8-4fb1-998b-60a2c0dc4cee/ae074854-c02c-496b-964f-ecb8956e53f8/9aa56239-1a3a-4aac-8799-c057bacf336d"
-					(reference "#PWR049")
+					(reference "#PWR0502")
+					(unit 1)
+				)
+				(path "/090a8e41-87a8-4fb1-998b-60a2c0dc4cee/ae074854-c02c-496b-964f-ecb8956e53f8/9aa56239-1a3a-4aac-8799-c057bacf336d"
+					(reference "#PWR0608")
 					(unit 1)
 				)
@@
 		(on_board yes)
 		(dnp no)
-		(property "Reference" "C18"
+		(property "Reference" "C502"
 			(at 172.72 91.44 90)
 			(effects
@@
 			(project "base-module"
 				(path "/090a8e41-87a8-4fb1-998b-60a2c0dc4cee/ae074854-c02c-496b-964f-ecb8956e53f8/7ee3192a-2c17-43bb-b41c-3a68ad8e606c"
-					(reference "C18")
-					(unit 1)
-				)
-				(path "/090a8e41-87a8-4fb1-998b-60a2c0dc4cee/ae074854-c02c-496b-964f-ecb8956e53f8/9aa56239-1a3a-4aac-8799-c057bacf336d"
-					(reference "C20")
+					(reference "C502")
+					(unit 1)
+				)
+				(path "/090a8e41-87a8-4fb1-998b-60a2c0dc4cee/ae074854-c02c-496b-964f-ecb8956e53f8/9aa56239-1a3a-4aac-8799-c057bacf336d"
+					(reference "C604")
 					(unit 1)
 				)
@@
 		(on_board yes)
 		(dnp no)
-		(property "Reference" "U4"
+		(property "Reference" "U501"
 			(at 151.13 89.535 0)
 			(effects
@@
 			(project "base-module"
 				(path "/090a8e41-87a8-4fb1-998b-60a2c0dc4cee/ae074854-c02c-496b-964f-ecb8956e53f8/7ee3192a-2c17-43bb-b41c-3a68ad8e606c"
-					(reference "U4")
-					(unit 1)
-				)
-				(path "/090a8e41-87a8-4fb1-998b-60a2c0dc4cee/ae074854-c02c-496b-964f-ecb8956e53f8/9aa56239-1a3a-4aac-8799-c057bacf336d"
-					(reference "U5")
+					(reference "U501")
+					(unit 1)
+				)
+				(path "/090a8e41-87a8-4fb1-998b-60a2c0dc4cee/ae074854-c02c-496b-964f-ecb8956e53f8/9aa56239-1a3a-4aac-8799-c057bacf336d"
+					(reference "U602")
 					(unit 1)
 				)
@@
 		(on_board yes)
 		(dnp no)
-		(property "Reference" "#PWR042"
+		(property "Reference" "#PWR0501"
 			(at 138.43 93.98 0)
 			(effects
@@
 			(project "base-module"
 				(path "/090a8e41-87a8-4fb1-998b-60a2c0dc4cee/ae074854-c02c-496b-964f-ecb8956e53f8/7ee3192a-2c17-43bb-b41c-3a68ad8e606c"
-					(reference "#PWR042")
-					(unit 1)
-				)
-				(path "/090a8e41-87a8-4fb1-998b-60a2c0dc4cee/ae074854-c02c-496b-964f-ecb8956e53f8/9aa56239-1a3a-4aac-8799-c057bacf336d"
-					(reference "#PWR048")
+					(reference "#PWR0501")
+					(unit 1)
+				)
+				(path "/090a8e41-87a8-4fb1-998b-60a2c0dc4cee/ae074854-c02c-496b-964f-ecb8956e53f8/9aa56239-1a3a-4aac-8799-c057bacf336d"
+					(reference "#PWR0607")
 					(unit 1)
 				)
@@
 		(on_board yes)
 		(dnp no)
-		(property "Reference" "R22"
+		(property "Reference" "R501"
 			(at 165.1 111.76 0)
 			(effects
@@
 			(project "base-module"
 				(path "/090a8e41-87a8-4fb1-998b-60a2c0dc4cee/ae074854-c02c-496b-964f-ecb8956e53f8/7ee3192a-2c17-43bb-b41c-3a68ad8e606c"
-					(reference "R22")
-					(unit 1)
-				)
-				(path "/090a8e41-87a8-4fb1-998b-60a2c0dc4cee/ae074854-c02c-496b-964f-ecb8956e53f8/9aa56239-1a3a-4aac-8799-c057bacf336d"
-					(reference "R23")
+					(reference "R501")
+					(unit 1)
+				)
+				(path "/090a8e41-87a8-4fb1-998b-60a2c0dc4cee/ae074854-c02c-496b-964f-ecb8956e53f8/9aa56239-1a3a-4aac-8799-c057bacf336d"
+					(reference "R602")
 					(unit 1)
 				)
@@
 		(on_board yes)
 		(dnp no)
-		(property "Reference" "#PWR044"
+		(property "Reference" "#PWR0503"
 			(at 125.73 100.33 0)
 			(effects
@@
 			(project "base-module"
 				(path "/090a8e41-87a8-4fb1-998b-60a2c0dc4cee/ae074854-c02c-496b-964f-ecb8956e53f8/7ee3192a-2c17-43bb-b41c-3a68ad8e606c"
-					(reference "#PWR044")
-					(unit 1)
-				)
-				(path "/090a8e41-87a8-4fb1-998b-60a2c0dc4cee/ae074854-c02c-496b-964f-ecb8956e53f8/9aa56239-1a3a-4aac-8799-c057bacf336d"
-					(reference "#PWR050")
+					(reference "#PWR0503")
+					(unit 1)
+				)
+				(path "/090a8e41-87a8-4fb1-998b-60a2c0dc4cee/ae074854-c02c-496b-964f-ecb8956e53f8/9aa56239-1a3a-4aac-8799-c057bacf336d"
+					(reference "#PWR0609")
 					(unit 1)
 				)
@@
 		(on_board yes)
 		(dnp no)
-		(property "Reference" "#PWR047"
+		(property "Reference" "#PWR0506"
 			(at 163.83 123.19 0)
 			(effects
@@
 			(project "base-module"
 				(path "/090a8e41-87a8-4fb1-998b-60a2c0dc4cee/ae074854-c02c-496b-964f-ecb8956e53f8/7ee3192a-2c17-43bb-b41c-3a68ad8e606c"
-					(reference "#PWR047")
-					(unit 1)
-				)
-				(path "/090a8e41-87a8-4fb1-998b-60a2c0dc4cee/ae074854-c02c-496b-964f-ecb8956e53f8/9aa56239-1a3a-4aac-8799-c057bacf336d"
-					(reference "#PWR053")
+					(reference "#PWR0506")
+					(unit 1)
+				)
+				(path "/090a8e41-87a8-4fb1-998b-60a2c0dc4cee/ae074854-c02c-496b-964f-ecb8956e53f8/9aa56239-1a3a-4aac-8799-c057bacf336d"
+					(reference "#PWR0612")
 					(unit 1)
 				)
@@
 		(on_board yes)
 		(dnp no)
-		(property "Reference" "C17"
+		(property "Reference" "C501"
 			(at 129.54 91.44 90)
 			(effects
@@
 			(project "base-module"
 				(path "/090a8e41-87a8-4fb1-998b-60a2c0dc4cee/ae074854-c02c-496b-964f-ecb8956e53f8/7ee3192a-2c17-43bb-b41c-3a68ad8e606c"
-					(reference "C17")
-					(unit 1)
-				)
-				(path "/090a8e41-87a8-4fb1-998b-60a2c0dc4cee/ae074854-c02c-496b-964f-ecb8956e53f8/9aa56239-1a3a-4aac-8799-c057bacf336d"
-					(reference "C19")
+					(reference "C501")
+					(unit 1)
+				)
+				(path "/090a8e41-87a8-4fb1-998b-60a2c0dc4cee/ae074854-c02c-496b-964f-ecb8956e53f8/9aa56239-1a3a-4aac-8799-c057bacf336d"
+					(reference "C603")
 					(unit 1)
 				)
@@
 		(on_board yes)
 		(dnp no)
-		(property "Reference" "#PWR045"
+		(property "Reference" "#PWR0504"
 			(at 176.53 100.33 0)
 			(effects
@@
 			(project "base-module"
 				(path "/090a8e41-87a8-4fb1-998b-60a2c0dc4cee/ae074854-c02c-496b-964f-ecb8956e53f8/7ee3192a-2c17-43bb-b41c-3a68ad8e606c"
-					(reference "#PWR045")
-					(unit 1)
-				)
-				(path "/090a8e41-87a8-4fb1-998b-60a2c0dc4cee/ae074854-c02c-496b-964f-ecb8956e53f8/9aa56239-1a3a-4aac-8799-c057bacf336d"
-					(reference "#PWR051")
+					(reference "#PWR0504")
+					(unit 1)
+				)
+				(path "/090a8e41-87a8-4fb1-998b-60a2c0dc4cee/ae074854-c02c-496b-964f-ecb8956e53f8/9aa56239-1a3a-4aac-8799-c057bacf336d"
+					(reference "#PWR0610")
 					(unit 1)
 				)
@@
 		(on_board yes)
 		(dnp no)
-		(property "Reference" "#PWR046"
+		(property "Reference" "#PWR0505"
 			(at 138.43 123.19 0)
 			(effects
@@
 			(project "base-module"
 				(path "/090a8e41-87a8-4fb1-998b-60a2c0dc4cee/ae074854-c02c-496b-964f-ecb8956e53f8/7ee3192a-2c17-43bb-b41c-3a68ad8e606c"
-					(reference "#PWR046")
-					(unit 1)
-				)
-				(path "/090a8e41-87a8-4fb1-998b-60a2c0dc4cee/ae074854-c02c-496b-964f-ecb8956e53f8/9aa56239-1a3a-4aac-8799-c057bacf336d"
-					(reference "#PWR052")
-					(unit 1)
-				)
+					(reference "#PWR0505")
+					(unit 1)
+				)
+				(path "/090a8e41-87a8-4fb1-998b-60a2c0dc4cee/ae074854-c02c-496b-964f-ecb8956e53f8/9aa56239-1a3a-4aac-8799-c057bacf336d"
+					(reference "#PWR0611")
+					(unit 1)
+				)

Commit message: [3] Add USB power + data schematic
Other:
- note added: "It's pretty empty here ... here's meme to fill some space:"

Commit message: [3] Add DIN41612 connector
Parts:
- U501: footprint HVSON-8-EP(3x3):HVSON-8-1EP_3x3mm_P0.65mm_EP1.6x2.4mm -> Package_SON:HVSON-8-1EP_3x3mm_P0.65mm_EP1.6x2.4mm
Changed lines of the file:
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@@
 	(wire
 		(pts
-			(xy 163.83 104.14) (xy 161.29 104.14)
+			(xy 182.88 104.14) (xy 161.29 104.14)
 		)
 		(stroke
@@
 	(wire
 		(pts
-			(xy 163.83 101.6) (xy 161.29 101.6)
+			(xy 182.88 101.6) (xy 161.29 101.6)
 		)
 		(stroke
@@
 	(hierarchical_label "CAN-"
 		(shape bidirectional)
-		(at 163.83 104.14 0)
+		(at 182.88 104.14 0)
 		(fields_autoplaced yes)
 		(effects
@@
 	(hierarchical_label "CAN+"
 		(shape bidirectional)
-		(at 163.83 101.6 0)
+		(at 182.88 101.6 0)
 		(fields_autoplaced yes)
 		(effects
@@
 			)
 		)
-		(property "Footprint" "HVSON-8-EP(3x3):HVSON-8-1EP_3x3mm_P0.65mm_EP1.6x2.4mm"
+		(property "Footprint" "Package_SON:HVSON-8-1EP_3x3mm_P0.65mm_EP1.6x2.4mm"
 			(at 165.1 191.44 0)
 			(effects

Commit message: Add QSPI flash to MCU
Parts:
- renumbered C501 to C423, C502 to C424, R501 to R405, U501 to U408
Connections:
- net CAN+ renamed CAN1.+
- net CAN- renamed CAN1.-
- net RX renamed CAN1.RX
- net TX renamed CAN1.TX
