File: base-module.kicad_sch (KiCad schematic)
At the start: 0 parts

Commit message: [3] Add USB hub, draft new MCU
Other:
- added sheet USBhub (USBhub.kicad_sch)
- sheet MCU ports: added USBIN1.{+ -}; removed none
Changed lines of the file:
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@@
 	(bus
 		(pts
-			(xy 110.49 59.69) (xy 104.14 59.69)
-		)
-		(stroke
-			(width 0)
-			(type default)
-		)
-	)
-	(bus
-		(pts
-			(xy 97.79 53.34) (xy 110.49 53.34)
-		)
-		(stroke
-			(width 0)
-			(type default)
-		)
-	)
-	(bus
-		(pts
-			(xy 104.14 59.69) (xy 104.14 82.55)
+			(xy 110.49 64.77) (xy 104.14 64.77)
+		)
+		(stroke
+			(width 0)
+			(type default)
+		)
+	)
+	(bus
+		(pts
+			(xy 110.49 41.91) (xy 104.14 41.91)
+		)
+		(stroke
+			(width 0)
+			(type default)
+		)
+	)
+	(bus
+		(pts
+			(xy 97.79 35.56) (xy 110.49 35.56)
 		)
 		(stroke
@@
 		)
 	)
+	(bus
+		(pts
+			(xy 135.89 54.61) (xy 148.59 54.61)
+		)
+		(stroke
+			(width 0)
+			(type default)
+		)
+	)
 	(wire
 		(pts
@@
 		(pts
 			(xy 104.14 82.55) (xy 110.49 82.55)
+		)
+		(stroke
+			(width 0)
+			(type default)
+		)
+	)
+	(bus
+		(pts
+			(xy 104.14 41.91) (xy 104.14 58.42)
+		)
+		(stroke
+			(width 0)
+			(type default)
+		)
+	)
+	(bus
+		(pts
+			(xy 104.14 58.42) (xy 110.49 58.42)
+		)
+		(stroke
+			(width 0)
+			(type default)
+		)
+	)
+	(bus
+		(pts
+			(xy 104.14 64.77) (xy 104.14 82.55)
 		)
 		(stroke
@@
 	)
 	(sheet
-		(at 110.49 48.26)
+		(at 110.49 30.48)
 		(size 25.4 13.97)
 		(fields_autoplaced yes)
@@
 		)
 		(property "Sheetname" "USB"
-			(at 110.49 47.5484 0)
+			(at 110.49 29.7684 0)
 			(effects
 				(font
@@
 		)
 		(property "Sheetfile" "USB.kicad_sch"
-			(at 110.49 62.8146 0)
+			(at 110.49 45.0346 0)
 			(effects
 				(font
@@
 		)
 		(pin "USB{SWIN}" input
-			(at 110.49 53.34 180)
+			(at 110.49 35.56 180)
 			(effects
 				(font
@@
 		)
 		(pin "USB{SWOUT}" input
-			(at 110.49 59.69 180)
+			(at 110.49 41.91 180)
 			(effects
 				(font
@@
 	)
 	(sheet
-		(at 148.59 74.93)
-		(size 44.45 54.61)
+		(at 148.59 30.48)
+		(size 44.45 99.06)
 		(fields_autoplaced yes)
 		(stroke
@@
 		)
 		(property "Sheetname" "MCU"
-			(at 148.59 74.2184 0)
+			(at 148.59 29.7684 0)
 			(effects
 				(font
@@
 		(pin "CAN{CAN1}" input
 			(at 148.59 90.17 180)
+			(effects
+				(font
+					(size 1.27 1.27)
+				)
+				(justify left)
+			)
+		)
+		(pin "USBIN1.{+ -}" input
+			(at 148.59 54.61 180)
 			(effects
 				(font
@@
 	)
 	(sheet
+		(at 110.49 52.07)
+		(size 25.4 16.51)
+		(fields_autoplaced yes)
+		(stroke
+			(width 0.1524)
+			(type solid)
+		)
+		(fill
+			(color 0 0 0 0.0000)
+		)
+		(property "Sheetname" "USBhub"
+			(at 110.49 51.3584 0)
+			(effects
+				(font
+					(size 1.27 1.27)
+				)
+				(justify left bottom)
+			)
+		)
+		(property "Sheetfile" "USBhub.kicad_sch"
+			(at 110.49 69.1646 0)
+			(effects
+				(font
+					(size 1.27 1.27)
+				)
+				(justify left top)
+			)
+		)
+		(pin "USBIN1.{+ -}" input
+			(at 110.49 58.42 180)
+			(effects
+				(font
+					(size 1.27 1.27)
+				)
+				(justify left)
+			)
+		)
+		(pin "USBOUT1.{+ -}" input
+			(at 110.49 64.77 180)
+			(effects
+				(font
+					(size 1.27 1.27)
+				)
+				(justify left)
+			)
+		)
+		(pin "USBOUT2.{+ -}" input
+			(at 135.89 54.61 0)
+			(effects
+				(font
+					(size 1.27 1.27)
+				)
+				(justify right)
+			)
+		)
+		(instances
+			(project "base-module"
+				(path "/090a8e41-87a8-4fb1-998b-60a2c0dc4cee"
+					(page "9")
+				)
+			)
+		)
+	)
+	(sheet
 		(at 110.49 74.93)
 		(size 25.4 10.16)
@@
 	)
 	(sheet
-		(at 72.39 48.26)
-		(size 25.4 64.77)
+		(at 72.39 30.48)
+		(size 25.4 82.55)
 		(fields_autoplaced yes)
 		(stroke
@@
 		)
 		(property "Sheetname" "Backplane"
-			(at 72.39 47.5484 0)
+			(at 72.39 29.7684 0)
 			(effects
 				(font
@@
 		)
 		(pin "USB{BACKPLANE}" input
-			(at 97.79 53.34 0)
-			(effects
-				(font
+			(at 97.79 35.56 0)
+			(effects
+				(font
