File: base-module.kicad_sch (KiCad schematic)
At the start: 0 parts

Commit message: [3] Rename USB hub sheet
Other:
- sheet USBhub renamed USB-hub
- sheet USB-hub: file USBhub.kicad_sch -> USB-hub.kicad_sch
Changed lines of the file:
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@@
 			(color 0 0 0 0.0000)
 		)
-		(property "Sheetname" "USBhub"
+		(property "Sheetname" "USB-hub"
 			(at 110.49 51.3584 0)
 			(effects
@@
 			)
 		)
-		(property "Sheetfile" "USBhub.kicad_sch"
+		(property "Sheetfile" "USB-hub.kicad_sch"
 			(at 110.49 69.1646 0)
 			(effects

Commit message: [3] Add DIN41612 connector
Other:
- sheet Backplane ports: added CAN1{CAN}, CAN2{CAN}; removed CAN{CAN1}, CAN{CAN2}
- sheet MCU ports: added CAN1{CAN}, CAN2{CAN}; removed CAN{CAN1}, CAN{CAN2}
Changed lines of the file:
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@@
 		(comment 2 "Project author: <author>")
 	)
-	(bus_alias "CAN1"
-		(members "1+" "1-")
-	)
-	(bus_alias "CAN2"
-		(members "2+" "2-")
+	(bus_alias "CAN"
+		(members "+" "-")
 	)
 	(bus_alias "ST-LINK"
@@
 	(bus
 		(pts
+			(xy 97.79 92.71) (xy 148.59 92.71)
+		)
+		(stroke
+			(width 0)
+			(type default)
+		)
+	)
+	(bus
+		(pts
+			(xy 97.79 90.17) (xy 148.59 90.17)
+		)
+		(stroke
+			(width 0)
+			(type default)
+		)
+	)
+	(bus
+		(pts
 			(xy 110.49 41.91) (xy 104.14 41.91)
 		)
@@
 		(pts
 			(xy 135.89 77.47) (xy 148.59 77.47)
-		)
-		(stroke
-			(width 0)
-			(type default)
-		)
-	)
-	(bus
-		(pts
-			(xy 97.79 92.71) (xy 148.59 92.71)
-		)
-		(stroke
-			(width 0)
-			(type default)
-		)
-	)
-	(bus
-		(pts
-			(xy 97.79 90.17) (xy 148.59 90.17)
 		)
 		(stroke
@@
 			)
 		)
-		(pin "CAN{CAN2}" input
-			(at 148.59 92.71 180)
-			(effects
-				(font
-					(size 1.27 1.27)
-				)
-				(justify left)
-			)
-		)
-		(pin "CAN{CAN1}" input
-			(at 148.59 90.17 180)
-			(effects
-				(font
-					(size 1.27 1.27)
-				)
-				(justify left)
-			)
-		)
 		(pin "USBIN1.{+ -}" input
 			(at 148.59 54.61 180)
+			(effects
+				(font
+					(size 1.27 1.27)
+				)
+				(justify left)
+			)
+		)
+		(pin "CAN2{CAN}" input
+			(at 148.59 92.71 180)
+			(effects
+				(font
+					(size 1.27 1.27)
+				)
+				(justify left)
+			)
+		)
+		(pin "CAN1{CAN}" input
+			(at 148.59 90.17 180)
 			(effects
 				(font
@@
 			)
 		)
-		(pin "CAN{CAN2}" input
-			(at 97.79 92.71 0)
-			(effects
-				(font
-					(size 1.27 1.27)
-				)
-				(justify right)
-			)
-		)
-		(pin "CAN{CAN1}" input
-			(at 97.79 90.17 0)
-			(effects
-				(font
-					(size 1.27 1.27)
-				)
-				(justify right)
-			)
-		)
 		(pin "USB{BACKPLANE}" input
 			(at 97.79 35.56 0)
 			(effects
 				(font
+					(size 1.27 1.27)
+				)
+				(justify right)
+			)
+		)
+		(pin "CAN1{CAN}" input
+			(at 97.79 90.17 0)
+			(effects
+				(font
+					(size 1.27 1.27)
+				)
+				(justify right)
+			)
+		)
+		(pin "CAN2{CAN}" input
+			(at 97.79 92.71 0)
+			(effects
+				(font

Commit message: Add QSPI flash to MCU
Other:
- added sheet CAN transceiver 1 (can-transceiver.kicad_sch)
- added sheet CAN transceiver 2 (can-transceiver.kicad_sch)
- added sheet QSPI FLASH (QSPI FLASH.kicad_sch)
- sheet MCU ports: added CAN1{RX TX}, CAN2{RX TX}, QSPI1{QSPI}, SWD1{SWD}; removed CAN1{CAN}, CAN2{CAN}, NRST, SWCLK, SWDIO
- sheet ST-LINK ports: added SWD1{SWD}; removed NRST, SWCLK, SWDIO

Commit message: [3] Fix usb bus issue
Other:
- sheet MCU ports: added USB_MCU{USB}; removed USBIN1.{+ -}
- sheet USB-hub ports: added USBOUT1{USB}, USB_MCU{USB}; removed USBOUT1.{+ -}, USBOUT2.{+ -}
Changed lines of the file:
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@@
+	(bus
+		(pts
+			(xy 135.89 55.88) (xy 148.59 55.88)
+		)
+		(stroke
+			(width 0)
+			(type default)
+		)
+	)
 	(bus
 		(pts
@@
 	(bus
 		(pts
-			(xy 135.89 54.61) (xy 148.59 54.61)
-		)
-		(stroke
-			(width 0)
-			(type default)
-		)
-	)
-	(bus
-		(pts
 			(xy 193.04 73.66) (xy 204.47 73.66)
 		)
@@
 	(bus
 		(pts
-			(xy 104.14 41.91) (xy 104.14 58.42)
-		)
-		(stroke
-			(width 0)
-			(type default)
-		)
-	)
-	(bus
-		(pts
-			(xy 104.14 58.42) (xy 110.49 58.42)
+			(xy 104.14 41.91) (xy 104.14 59.69)
+		)
+		(stroke
+			(width 0)
+			(type default)
+		)
+	)
+	(bus
+		(pts
+			(xy 104.14 59.69) (xy 110.49 59.69)
 		)
 		(stroke
@@
 			)
 		)
-		(pin "USBIN1.{+ -}" input
-			(at 148.59 54.61 180)
-			(effects
-				(font
-					(size 1.27 1.27)
-				)
-				(justify left)
-			)
-		)
 		(pin "QSPI1{QSPI}" input
 			(at 193.04 73.66 0)
@@
 		(pin "SWD1{SWD}" input
 			(at 148.59 77.47 180)
+			(effects
+				(font
+					(size 1.27 1.27)
+				)
+				(justify left)
+			)
+		)
+		(pin "USB_MCU{USB}" input
+			(at 148.59 55.88 180)
 			(effects
 				(font
@@
 		)
 		(pin "USBIN1.{+ -}" input
-			(at 110.49 58.42 180)
-			(effects
-				(font
-					(size 1.27 1.27)
-				)
-				(justify left)
-			)
-		)
-		(pin "USBOUT1.{+ -}" input
+			(at 110.49 59.69 180)
+			(effects
+				(font
+					(size 1.27 1.27)
+				)
+				(justify left)
+			)
+		)
+		(pin "USBOUT1{USB}" input
 			(at 110.49 64.77 180)
 			(effects
@@
 			)
 		)
-		(pin "USBOUT2.{+ -}" input
-			(at 135.89 54.61 0)
-			(effects
-				(font
+		(pin "USB_MCU{USB}" input
+			(at 135.89 55.88 0)
+			(effects
+				(font
