File: st-link.kicad_sch (KiCad schematic)
At the start: 33 parts, among them U2 STM32F103CBTx, Y2 Crystal

Commit message: Add usb schematic
Parts:
- removed Y2: Crystal, symbol Device:Crystal
- added Y501: 8MHz, symbol Device:Crystal_Small
- renumbered C6 to C12, C2 to C13, C4 to C14, C1 to C15, C3 to C16, C5 to C17, C12 to C18, C10 to C19, C11 to C20, D1 to D6, D2 to D7, R13 to R10, R16 to R11, R2 to R12, R10 to R13, R15 to R14, R3 to R15, R4 to R16, R11 to R17, R12 to R18, R1 to R19, R6 to R20, R14 to R21, R7 to R9, TP3 to TP10, TP4 to TP11, TP5 to TP12, TP1 to TP8, TP2 to TP9, U2 to U4
Connections:
- net STLINK-OSC_IN: now also Y501.1
- net STLINK-OSC_OUT: now also Y501.2

Commit message: [3] Add USB power + data schematic
Parts:
- R10, R11: value 4k7 -> 10k
Other:
- note added: "ACTIVE LED"
- note added: "Alternative GD32F103CB"
- note added: "CAUTION:"
- note added: "Credit to:"
- note added: "MANDATORY CB VERSION"
- note added: "NOTICE:"
- note added: "Populate with STM32F103C8, STM32F103CB"
- note added: "for providing amazing reverse engeenering of ST-link"
- note removed: "Works with STM32F103C8 STM32F103CB or GD32F103CB But CB should be used"
- moved on the sheet: C12, C13, C14, C15, C16, C17, C18, C19, C20, D6, D7, R10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

Commit message: [3] Finish ST-LINK schematic
Parts:
- removed C12: 1u, Capacitor_SMD:C_0402_1005Metric, symbol Device:C_Small
- removed C13, C14, C15, C16, C17, C18: 100n, Capacitor_SMD:C_0402_1005Metric, symbol Device:C_Small
- removed C19, C20: 22p, Capacitor_SMD:C_0402_1005Metric, symbol Device:C_Small
- removed D6: BLUE, LED_SMD:LED_0603_1608Metric, symbol Device:LED
- removed D7: RED, LED_SMD:LED_0603_1608Metric, symbol Device:LED
- removed R10, R11, R15, R16: 10k, Resistor_SMD:R_0402_1005Metric, symbol Device:R_Small
- removed R12, R14, R18, R9: 100k, Resistor_SMD:R_0402_1005Metric, symbol Device:R_Small
- removed R13, R17, R20, R21: 22R, Resistor_SMD:R_0402_1005Metric, symbol Device:R_Small
- removed R19: 100R, Resistor_SMD:R_0402_1005Metric, symbol Device:R_Small
- removed Y501: 8MHz, symbol Device:Crystal_Small
- added C428, C429, C430, C431, C432, C434: 100nF, PCM_JLCPCB:C_0402, symbol PCM_JLCPCB-Capacitors:0402,100nF,(2)
- added C433: 1uF, PCM_JLCPCB:C_0402, symbol PCM_JLCPCB-Capacitors:0402,1uF
- added C435, C437: 33pF, PCM_JLCPCB:C_0402, symbol PCM_JLCPCB-Capacitors:0402,33pF
- added D406: Green, PCM_JLCPCB:D_0603, symbol PCM_JLCPCB-Diodes:LED,0603,Green
- added D407: Blue, PCM_JLCPCB:D_0603, symbol PCM_JLCPCB-Diodes:LED,0603,Blue
- added Q403: S9013, PCM_JLCPCB:Q_SOT-23, symbol PCM_JLCPCB-Transistors:NPN,S9013
- added R424: 39kΩ, PCM_JLCPCB:R_0402, symbol PCM_JLCPCB-Resistors:0402,39kΩ
- added R425, R427, R429, R432, R433, R439, R440: 10kΩ, PCM_JLCPCB:R_0402, symbol PCM_JLCPCB-Resistors:0402,10kΩ
- added R426: 1.2kΩ, PCM_JLCPCB:R_0402, symbol PCM_JLCPCB-Resistors:0402,1.2kΩ
- added R428, R438: 100Ω, PCM_JLCPCB:R_0402, symbol PCM_JLCPCB-Resistors:0402,100Ω
- added R430, R431: 100kΩ, PCM_JLCPCB:R_0402, symbol PCM_JLCPCB-Resistors:0402,100kΩ
- added R434, R435, R436, R437: 22Ω, PCM_JLCPCB:R_0402, symbol PCM_JLCPCB-Resistors:0402,22Ω
- added X401: X50328MSB2GI, PCM_JLCPCB:CRYSTAL-SMD_L5.0-W3.2, symbol PCM_JLCPCB-Crystals:Crystal, 8MHz, 20pF, ±10ppm
Connections:
- net +3V3: now also C428.1, C429.1, C430.1, C431.1, C432.1, C433.1, Q403.3 (C), R430.1, R439.1, R440.1
- net GND: now also C428.2, C429.2, C430.2, C431.2, C432.2, C433.2, C434.2, C435.2, C437.2, R424.2, R427.2, R429.2, R431.1, R432.1, R433.1; no longer U4.20 (PB2)
- net LED: now also D406.2, D407.1
- net NRST: now also R434.1
- net STLINK-BOOT0: now also R431.2
- net STLINK-OSC_IN: now also C437.1, X401.1
- net STLINK-OSC_OUT: now also C435.1, X401.2
- net STLINK-RST: now also C434.1, R430.2
- net SWCLK: now also R435.1, R437.2
- net SWDIO: now also R436.1
- net USB_RENUM: now also R428.2
- net at U4.2 (PC13): now also R432.2
- net at U4.26 (PB13): now also R435.2
- net at U4.10 (PA0): now also R429.1, R440.2
- net at U4.15 (PA5): now also R437.1
- net at U4.18 (PB0): now also R434.2
- net at U4.25 (PB12): now also R438.2
- net at U4.27 (PB14): now also R436.2, R438.1
- net at U4.3 (PC14): now also R433.2
- new net: Q403.2 (E), R426.1
- new net: Q403.1 (B), R424.1, R425.2, R428.1
- new net: D406.1, R427.1
- new net: D407.2, R439.2
- new net +5V: R425.1
- new net USB_D+: R426.2
- no-connect marks 18 -> 19
Other:
- note added: "C406=C407 = (CL - 4pF) * 2"
- note added: "FORCE RENUMERATION OF USB DEVICES"
- note added: "Should be 1k5, but we try 1k2 because it is in basic parts"
- moved on the sheet: TP10, TP11, TP12, TP6, TP7, TP8, TP9, U4

Commit message: [3] Annotate ST-LINK schematic, fix minor text missalignments
Parts:
- renumbered C433 to C700, C432 to C701, C431 to C702, C430 to C703, C429 to C704, C428 to C705, C434 to C706, C437 to C707, C435 to C708, D407 to D700, D406 to D701, Q403 to Q700, R430 to R700, R440 to R701, R431 to R702, R429 to R703, R437 to R704, R432 to R705, R433 to R706, R439 to R707, R434 to R708, R425 to R709, R428 to R710, R424 to R711, R426 to R712, R427 to R713, R438 to R714, R435 to R715, R436 to R716, TP6 to TP700, TP7 to TP701, TP8 to TP702, TP9 to TP703, TP10 to TP704, TP11 to TP705, TP12 to TP706, U4 to U700, X401 to X700
Other:
- note added: "ACTIVITY LED"
- note removed: "ACTIVE LED"
- moved on the sheet: Q700, R709, R710, R711, R712

Commit message: [3] Add resistor and test points footprints
Parts:
- TP702, TP703, TP704, TP705, TP706: footprint TestPoint:TestPoint_Pad_1.0x1.0mm -> TestPoint:TestPoint_Pad_D1.0mm
Changed lines of the file:
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@@
 	(label "STLINK_RX"
 		(at 115.57 62.23 180)
-		(fields_autoplaced yes)
 		(effects
 			(font
@@
 	(label "SWO"
 		(at 115.57 80.01 180)
-		(fields_autoplaced yes)
 		(effects
 			(font
@@
 	(label "USB.D-"
 		(at 115.57 82.55 180)
-		(fields_autoplaced yes)
 		(effects
 			(font
@@
 	(label "USB_RENUM"
 		(at 115.57 92.71 180)
-		(fields_autoplaced yes)
 		(effects
 			(font
@@
 	(label "STLINK_TX"
 		(at 115.57 59.69 180)
-		(fields_autoplaced yes)
 		(effects
 			(font
@@
 	(label "STLINK-BOOT0"
 		(at 53.34 59.69 0)
-		(fields_autoplaced yes)
 		(effects
 			(font
@@
 	(label "CLK"
 		(at 181.61 96.52 0)
-		(fields_autoplaced yes)
 		(effects
 			(font
@@
 	(label "LED"
 		(at 115.57 77.47 180)
-		(fields_autoplaced yes)
 		(effects
 			(font
@@
 	(label "LED"
 		(at 156.21 93.98 0)
-		(fields_autoplaced yes)
 		(effects
 			(font
@@
 	(label "STLINK-RST"
 		(at 55.88 54.61 0)
-		(fields_autoplaced yes)
 		(effects
 			(font
@@
 	(label "STLINK-OSC_OUT"
 		(at 52.07 67.31 0)
-		(fields_autoplaced yes)
 		(effects
 			(font
@@
 	(label "USB.D+"
 		(at 115.57 85.09 180)
-		(fields_autoplaced yes)
 		(effects
 			(font
@@
 	(label "USB_RENUM"
 		(at 259.08 91.44 180)
-		(fields_autoplaced yes)
 		(effects
 			(font
@@
 	(label "STLINK-OSC_IN"
 		(at 52.07 64.77 0)
-		(fields_autoplaced yes)
 		(effects
 			(font
@@
 	(label "BOOT"
 		(at 181.61 88.9 0)
-		(fields_autoplaced yes)
 		(effects
 			(font
@@
 	(label "DIO"
 		(at 181.61 92.71 0)
-		(fields_autoplaced yes)
 		(effects
 			(font
@@
 	(label "CLK"
 		(at 115.57 90.17 180)
-		(fields_autoplaced yes)
 		(effects
 			(font
@@
 	(label "DIO"
 		(at 115.57 87.63 180)
-		(fields_autoplaced yes)
 		(effects
 			(font
@@
 		(shape bidirectional)
 		(at 38.1 118.11 180)
-		(fields_autoplaced yes)
 		(effects
 			(font
@@
 		(shape input)
 		(at 38.1 115.57 180)
-		(fields_autoplaced yes)
 		(effects
 			(font
@@
 		(shape input)
 		(at 121.92 88.9 0)
-		(fields_autoplaced yes)
 		(effects
 			(font
@@
 		(shape input)
 		(at 116.84 67.31 0)
-		(fields_autoplaced yes)
 		(effects
 			(font
@@
 		(shape input)
 		(at 220.98 116.84 0)
-		(fields_autoplaced yes)
 		(effects
 			(font
@@
 		(shape output)
 		(at 55.88 82.55 180)
-		(fields_autoplaced yes)
 		(effects
 			(font
@@
 			)
 		)
-		(property "Footprint" "TestPoint:TestPoint_Pad_1.0x1.0mm"
+		(property "Footprint" "TestPoint:TestPoint_Pad_D1.0mm"
 			(at 190.5 97.79 0)
 			(effects
@@
 			)
 		)
-		(property "Footprint" "TestPoint:TestPoint_Pad_1.0x1.0mm"
+		(property "Footprint" "TestPoint:TestPoint_Pad_D1.0mm"
 			(at 190.5 101.6 0)
 			(effects
@@
 			)
 		)
-		(property "Footprint" "TestPoint:TestPoint_Pad_1.0x1.0mm"
+		(property "Footprint" "TestPoint:TestPoint_Pad_D1.0mm"
 			(at 190.5 90.17 0)
 			(effects
@@
 			)
 		)
-		(property "Footprint" "TestPoint:TestPoint_Pad_1.0x1.0mm"
+		(property "Footprint" "TestPoint:TestPoint_Pad_D1.0mm"
 			(at 190.5 93.98 0)
 			(effects
@@
 			)
 		)
-		(property "Footprint" "TestPoint:TestPoint_Pad_1.0x1.0mm"
+		(property "Footprint" "TestPoint:TestPoint_Pad_D1.0mm"
 			(at 190.5 105.41 0)
 			(effects
