File: st-link.kicad_sch (KiCad schematic)
At the start: 38 parts, among them Q700 S9013, U700 STM32F103CBTx, X700 X50328MSB2GI

Commit message: [3] Fix schematic typos
Connections:
- net BOOT renamed BOOT0
Changed lines of the file:
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@@
 	(label "STLINK_RX"
 		(at 115.57 62.23 180)
+		(fields_autoplaced yes)
 		(effects
 			(font
@@
 	(label "SWO"
 		(at 115.57 80.01 180)
+		(fields_autoplaced yes)
 		(effects
 			(font
@@
 	(label "USB.D-"
 		(at 115.57 82.55 180)
+		(fields_autoplaced yes)
 		(effects
 			(font
@@
 	(label "USB_RENUM"
 		(at 115.57 92.71 180)
+		(fields_autoplaced yes)
 		(effects
 			(font
@@
 	(label "STLINK_TX"
 		(at 115.57 59.69 180)
+		(fields_autoplaced yes)
 		(effects
 			(font
@@
 	(label "STLINK-BOOT0"
 		(at 53.34 59.69 0)
+		(fields_autoplaced yes)
 		(effects
 			(font
@@
 	(label "CLK"
 		(at 181.61 96.52 0)
+		(fields_autoplaced yes)
 		(effects
 			(font
@@
 	(label "LED"
 		(at 115.57 77.47 180)
+		(fields_autoplaced yes)
 		(effects
 			(font
@@
 	(label "LED"
 		(at 156.21 93.98 0)
+		(fields_autoplaced yes)
 		(effects
 			(font
@@
 	(label "STLINK-RST"
 		(at 55.88 54.61 0)
+		(fields_autoplaced yes)
 		(effects
 			(font
@@
 	(label "STLINK-OSC_OUT"
 		(at 52.07 67.31 0)
+		(fields_autoplaced yes)
 		(effects
 			(font
@@
 	(label "USB.D+"
 		(at 115.57 85.09 180)
+		(fields_autoplaced yes)
 		(effects
 			(font
@@
 	(label "USB_RENUM"
 		(at 259.08 91.44 180)
+		(fields_autoplaced yes)
 		(effects
 			(font
@@
 	(label "STLINK-OSC_IN"
 		(at 52.07 64.77 0)
-		(effects
-			(font
-				(size 1.27 1.27)
-			)
-			(justify left bottom)
-		)
-	)
-	(label "BOOT"
+		(fields_autoplaced yes)
+		(effects
+			(font
+				(size 1.27 1.27)
+			)
+			(justify left bottom)
+		)
+	)
+	(label "BOOT0"
 		(at 181.61 88.9 0)
+		(fields_autoplaced yes)
 		(effects
 			(font
@@
 	(label "DIO"
 		(at 181.61 92.71 0)
+		(fields_autoplaced yes)
 		(effects
 			(font
@@
 	(label "CLK"
 		(at 115.57 90.17 180)
+		(fields_autoplaced yes)
 		(effects
 			(font
@@
 	(label "DIO"
 		(at 115.57 87.63 180)
+		(fields_autoplaced yes)
 		(effects
 			(font
@@
 		(shape bidirectional)
 		(at 38.1 118.11 180)
+		(fields_autoplaced yes)
 		(effects
 			(font
@@
 		(shape input)
 		(at 38.1 115.57 180)
+		(fields_autoplaced yes)
 		(effects
 			(font
@@
 		(shape input)
 		(at 121.92 88.9 0)
+		(fields_autoplaced yes)
 		(effects
 			(font
@@
 		(shape input)
 		(at 116.84 67.31 0)
+		(fields_autoplaced yes)
 		(effects
 			(font
@@
 		(shape input)
 		(at 220.98 116.84 0)
+		(fields_autoplaced yes)
 		(effects
 			(font
@@
 		(shape output)
 		(at 55.88 82.55 180)
-		(effects
-			(font
+		(fields_autoplaced yes)
+		(effects
+			(font

Commit message: Fix St-link schematic errors
Connections:
- net BOOT0 is gone; now on net STLINK-BOOT0: TP703.1
- net USB_D+ is gone; now on net USB.D+: R712.2
Changed lines of the file:
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@@
 	(wire
 		(pts
-			(xy 181.61 88.9) (xy 190.5 88.9)
+			(xy 179.07 88.9) (xy 190.5 88.9)
 		)
 		(stroke
@@
 	(wire
 		(pts
-			(xy 181.61 96.52) (xy 190.5 96.52)
+			(xy 179.07 96.52) (xy 190.5 96.52)
 		)
 		(stroke
@@
 	(wire
 		(pts
-			(xy 181.61 92.71) (xy 190.5 92.71)
+			(xy 179.07 92.71) (xy 190.5 92.71)
 		)
 		(stroke
@@
 		)
 	)
+	(label "STLINK-BOOT0"
+		(at 179.07 88.9 0)
+		(fields_autoplaced yes)
+		(effects
+			(font
+				(size 1.27 1.27)
+			)
+			(justify left bottom)
+		)
+	)
 	(label "SWO"
 		(at 115.57 80.01 180)
@@
 	)
 	(label "CLK"
-		(at 181.61 96.52 0)
+		(at 179.07 96.52 0)
 		(fields_autoplaced yes)
 		(effects
@@
 		)
 	)
+	(label "USB.D+"
+		(at 220.98 116.84 0)
+		(fields_autoplaced yes)
+		(effects
+			(font
+				(size 1.27 1.27)
+			)
+			(justify left bottom)
+		)
+	)
 	(label "STLINK-OSC_IN"
 		(at 52.07 64.77 0)
@@
 		)
 	)
-	(label "BOOT0"
-		(at 181.61 88.9 0)
-		(fields_autoplaced yes)
-		(effects
-			(font
-				(size 1.27 1.27)
-			)
-			(justify left bottom)
-		)
-	)
 	(label "DIO"
-		(at 181.61 92.71 0)
+		(at 179.07 92.71 0)
 		(fields_autoplaced yes)
 		(effects
@@
 		(fields_autoplaced yes)
 		(effects
-			(font
-				(size 1.27 1.27)
-			)
-			(justify left)
-		)
-	)
-	(hierarchical_label "USB_D+"
-		(shape input)
-		(at 220.98 116.84 0)
-		(fields_autoplaced yes)
-		(effects

Commit message: Add QSPI flash to MCU
Connections:
- net NRST renamed ~{RST}
- net SWCLK renamed SWD.SWCLK
- net SWDIO renamed SWD.SWDIO
Other:
- moved on the sheet: R701, R703
