File: st-link.kicad_sch (KiCad schematic)
At the start: 38 parts, among them Q700 MMST3904, U700 STM32F103CBTx, Y700 8 MHz

Commit message: [#12] Add missing Y700 data
Parts:
- Y700: LCSC (none) -> C7424755; MPN (none) -> 3225-8.00-20-10-10/4B
Changed lines of the file:
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@@
 			)
 		)
-		(property "Description" "Four pin crystal, GND on pins 2 and 4"
+		(property "Description" "8MHz 20pF ±10ppm SMD3225 Crystals ROHS"
 			(at 41.91 85.09 0)
 			(effects
+				(font
+					(size 1.27 1.27)
+				)
+				(hide yes)
+			)
+		)
+		(property "MPN" "3225-8.00-20-10-10/4B"
+			(at 41.91 85.09 0)
+			(effects
+				(font
+					(size 1.27 1.27)
+				)
+				(hide yes)
+			)
+		)
+		(property "LCSC" "C7424755"
+			(at 41.91 85.09 0)
+			(effects

Commit message: Change MCU and update library
Changed MCU from H7 to H5 series due to programming issues with external
loader. Also updated JLCPCB components (not all tho there are still
arround 18 components to fix)
Parts:
- C700: Stock 8480407 -> 6453835
- C701, C702, C703, C704, C705, C706: Stock 5427590 -> 5436546
- C707, C708: Stock 1088254 -> 1049076
- Q700: Stock 32529 -> 19064
- R700, R702: Stock 5666023 -> 5804343
- R701, R703, R705, R706, R707, R709, R713: Stock 7034931 -> 13746052
- R704, R708, R715, R716: Stock 2545567 -> 2158519
- R710, R714: Stock 2831654 -> 3389382
- R711: Stock 415990 -> 134046
- R712: Stock 236021 -> 191144
- TP702, TP703, TP704, TP705, TP706: value ~ -> TestPoint
- Y700: value 8 MHz -> Crystal_GND24
Other:
- title: ModuCard base module -> ModuCard BM STM32H562VGT6
- moved on the sheet: C700, C701, C702, C703, C704, C705, C706, C707, C708, R700, R701, R702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

Commit message: [1] Change MCU schematic ERC pass
Parts:
- removed D700: Blue, PCM_JLCPCB:D_0603, symbol PCM_JLCPCB-Diodes:LED,0603,Blue
- removed D701: Green, PCM_JLCPCB:D_0603, symbol PCM_JLCPCB-Diodes:LED,0603,Green
- added D700, D701: Red, PCM_JLCPCB:D_0603, symbol PCM_JLCPCB-Diodes:LED,0603,Red
Connections:
- net LED: now also D700.1, D701.2
- net at R713.1: now also D701.1
- net at R707.2: now also D700.2
Other:
- note added: "Do weryfikackji"

Commit message: [REV2] board finshed, schematics and leyout
Other:
- title: ModuCard BM STM32H562VGT6 -> ModuCard nav module
Changed lines of the file:
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@@
 	(paper "A4")
 	(title_block
-		(title "ModuCard BM STM32H562VGT6")
-		(date "2025-04-18")
+		(title "ModuCard nav module")
+		(date "2025-04-20")
 		(rev "1.1.0")
 		(company "KoNaR")
 		(comment 1 "Base project authors: Dominik Pluta, Artem Horiunov")
-		(comment 2 "Project author: <author>")
+		(comment 2 "Project author: Patryk Dudziński")
 	)
 	(rectangle

Commit message: changed shity resisrto to smaller one on LEDs  fixed level shifting
Parts:
- removed R707, R713: 10kΩ, PCM_JLCPCB:R_0402, symbol PCM_JLCPCB-Resistors:0402,10kΩ
- added R409, R429: 220Ω, PCM_JLCPCB:R_0402, symbol PCM_JLCPCB-Resistors:0402,220Ω
Connections:
- net +3V3: now also R409.1
- net GND: now also R429.2
- net at D701.1: now also R429.1
- net at D700.2: now also R409.2
Other:
- note removed: "Do weryfikackji"
