File: backplane.kicad_sch (KiCad schematic)
At the start: 0 parts

Commit message: Add usb schematic
Parts:
- added U403: IP4234CZ6,115, Package_TO_SOT_SMD:SC-74-6_1.55x2.9mm_P0.95mm, symbol Power_Protection:IP4234CZ6
Connections:
- new net USB1U.D+: U403.4, U403.6
- new net USB1U.D-: U403.1, U403.3
Changed lines of the file:
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@@
 	)
 	(bus_entry
-		(at 236.22 137.16)
+		(at 229.87 138.43)
 		(size 2.54 2.54)
 		(stroke
@@
 	)
 	(bus_entry
-		(at 236.22 139.7)
+		(at 229.87 143.51)
 		(size 2.54 2.54)
 		(stroke
@@
 	(bus
 		(pts
-			(xy 238.76 142.24) (xy 238.76 148.59)
+			(xy 232.41 149.86) (xy 232.41 146.05)
 		)
 		(stroke
@@
 	(wire
 		(pts
-			(xy 222.25 137.16) (xy 236.22 137.16)
+			(xy 208.28 138.43) (xy 229.87 138.43)
 		)
 		(stroke
@@
 		)
 	)
+	(wire
+		(pts
+			(xy 182.88 138.43) (xy 187.96 138.43)
+		)
+		(stroke
+			(width 0)
+			(type default)
+		)
+	)
 	(bus
 		(pts
@@
 	(bus
 		(pts
-			(xy 238.76 139.7) (xy 238.76 142.24)
+			(xy 232.41 140.97) (xy 232.41 146.05)
 		)
 		(stroke
@@
 		)
 	)
+	(wire
+		(pts
+			(xy 182.88 143.51) (xy 187.96 143.51)
+		)
+		(stroke
+			(width 0)
+			(type default)
+		)
+	)
 	(bus
 		(pts
@@
 	(bus
 		(pts
-			(xy 238.76 148.59) (xy 252.73 148.59)
+			(xy 232.41 149.86) (xy 243.84 149.86)
 		)
 		(stroke
@@
 	(wire
 		(pts
-			(xy 222.25 139.7) (xy 236.22 139.7)
+			(xy 208.28 143.51) (xy 229.87 143.51)
 		)
 		(stroke
@@
 	)
 	(rectangle
-		(start 210.185 124.46)
+		(start 170.18 124.46)
 		(end 270.51 153.67)
 		(stroke
@@
 	(text "USB\n"
 		(exclude_from_sim no)
-		(at 216.154 130.556 0)
+		(at 263.906 129.032 0)
 		(effects
 			(font
@@
 		)
 	)
+	(label "USB1U.D-"
+		(at 222.25 143.51 180)
+		(fields_autoplaced yes)
+		(effects
+			(font
+				(size 1.27 1.27)
+				(italic yes)
+			)
+			(justify right bottom)
+		)
+	)
 	(label "CAN.1+"
 		(at 242.57 101.6 180)
@@
 		)
 	)
+	(label "USB1U.D+"
+		(at 182.88 138.43 180)
+		(fields_autoplaced yes)
+		(effects
+			(font
+				(size 1.27 1.27)
+				(italic yes)
+			)
+			(justify right bottom)
+		)
+	)
 	(label "GPIOR7"
 		(at 77.47 46.99 0)
@@
 		)
 	)
+	(label "USB1U.D-"
+		(at 182.88 143.51 180)
+		(fields_autoplaced yes)
+		(effects
+			(font
+				(size 1.27 1.27)
+				(italic yes)
+			)
+			(justify right bottom)
+		)
+	)
 	(label "GPIOL15"
 		(at 57.15 121.92 0)
@@
 		)
 	)
-	(label "USB.D-"
-		(at 222.25 139.7 180)
-		(fields_autoplaced yes)
-		(effects
-			(font
-				(size 1.27 1.27)
-				(italic yes)
-			)
-			(justify right bottom)
-		)
-	)
 	(label "GPIOC2"
 		(at 57.15 144.78 0)
@@
 		)
 	)
-	(label "USB.D+"
-		(at 222.25 137.16 180)
+	(label "USB1U.D+"
+		(at 222.25 138.43 180)
 		(fields_autoplaced yes)
 		(effects
@@
 	(hierarchical_label "USB{ST-LINK}"
 		(shape input)
-		(at 252.73 148.59 0)
+		(at 243.84 149.86 0)
 		(fields_autoplaced yes)
 		(effects
@@
 		)
 	)
+	(symbol
+		(lib_id "Power_Protection:IP4234CZ6")
+		(at 198.12 140.97 0)
+		(unit 1)
+		(exclude_from_sim no)
+		(in_bom yes)
+		(on_board yes)
+		(dnp no)
+		(property "Reference" "U403"
+			(at 201.93 130.302 0)
+			(effects
+				(font
+					(size 1.27 1.27)
+				)
+				(justify left)
+			)
+		)
+		(property "Value" "IP4234CZ6,115"
+			(at 201.93 132.08 0)
+			(effects
+				(font
+					(size 1.27 1.27)
+				)
+				(justify left)
+			)
+		)
+		(property "Footprint" "Package_TO_SOT_SMD:SC-74-6_1.55x2.9mm_P0.95mm"
+			(at 198.12 156.718 0)
+			(effects
+				(font
+					(size 1.27 1.27)
+				)
+				(hide yes)
+			)
+		)
+		(property "Datasheet" "https://assets.nexperia.com/documents/data-sheet/IP4234CZ6.pdf"
+			(at 198.12 161.036 0)
+			(effects
+				(font
+					(size 1.27 1.27)
+				)
+				(hide yes)
+			)
+		)
+		(property "Description" "ESD Protection, 2 channel, USB 2.0 to IEC 61000-4-2 level 4, 5.5V, SOT457 (SC-74-6)"
+			(at 198.12 159.004 0)
+			(effects
+				(font
+					(size 1.27 1.27)
+				)
+				(hide yes)
+			)
+		)
+		(pin "3"
+		)
+		(pin "4"
+		)
+		(pin "5"
+		)
+		(pin "1"
+		)
+		(pin "6"
+		)
+		(pin "2"
+		)
+		(instances
+			(project "base-module"
+				(path "/090a8e41-87a8-4fb1-998b-60a2c0dc4cee/ff3476d7-2f10-4f79-9864-988601c7ce1b"
+					(reference "U403")
+					(unit 1)
+				)
+			)
+		)
+	)

Commit message: [3] Add USB power + data schematic
Changed lines of the file:
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@@
 		)
 	)
-	(hierarchical_label "USB{ST-LINK}"
+	(hierarchical_label "USB{BACKPLANE}"
 		(shape input)
 		(at 243.84 149.86 0)
@@
 					(unit 1)
 				)
+			)
+		)
+	)
+	(symbol
+		(lib_id "power:+12V")
+		(at 186.69 76.2 0)
+		(unit 1)
+		(exclude_from_sim no)
+		(in_bom yes)
+		(on_board yes)
+		(dnp no)
+		(fields_autoplaced yes)
+		(property "Reference" "#PWR0427"
+			(at 186.69 80.01 0)
+			(effects
+				(font
+					(size 1.27 1.27)
+				)
+				(hide yes)
+			)
+		)
+		(property "Value" "+12V_Unprotec"
+			(at 186.69 71.12 0)
+			(effects
+				(font
+					(size 1.27 1.27)
+				)
+			)
+		)
+		(property "Footprint" ""
+			(at 186.69 76.2 0)
+			(effects
+				(font
+					(size 1.27 1.27)
+				)
+				(hide yes)
+			)
+		)
+		(property "Datasheet" ""
+			(at 186.69 76.2 0)
+			(effects
+				(font
+					(size 1.27 1.27)
+				)
+				(hide yes)
+			)
+		)
+		(property "Description" "Power symbol creates a global label with name \"+12V\""
+			(at 186.69 76.2 0)
+			(effects
+				(font
+					(size 1.27 1.27)
+				)
+				(hide yes)
+			)
+		)
+		(pin "1"
+		)
+		(instances
+			(project ""
+				(path "/090a8e41-87a8-4fb1-998b-60a2c0dc4cee/ff3476d7-2f10-4f79-9864-988601c7ce1b"
+					(reference "#PWR0427")
+					(unit 1)
+				)

Commit message: WIP: Add backplane connector
Parts:
- added J200: 09031967921, Connector_DIN:DIN41612_R_3x32_Female_Horizontal_THT, symbol DIN41612_3x32:09031967921
Connections:
- net GPIOC0: now also J200.b16
- net GPIOC1: now also J200.b17
- net GPIOC10: now also J200.b26
- net GPIOC11: now also J200.b27
- net GPIOC12: now also J200.b28
- net GPIOC13: now also J200.b29
- net GPIOC14: now also J200.b30
- net GPIOC15: now also J200.b31
- net GPIOC2: now also J200.b18
- net GPIOC3: now also J200.b19
- net GPIOC4: now also J200.b20
- net GPIOC5: now also J200.b21
- net GPIOC6: now also J200.b22
- net GPIOC7: now also J200.b23
- net GPIOC8: now also J200.b24
- net GPIOC9: now also J200.b25
- net GPIOL0: now also J200.a16
- net GPIOL1: now also J200.a17
- net GPIOL10: now also J200.a26
- net GPIOL11: now also J200.a27
- net GPIOL12: now also J200.a28
- net GPIOL13: now also J200.a29
- net GPIOL14: now also J200.a30
- net GPIOL15: now also J200.a31
- net GPIOL2: now also J200.a18
- net GPIOL3: now also J200.a19
- net GPIOL4: now also J200.a20
- net GPIOL5: now also J200.a21
- net GPIOL6: now also J200.a22
- net GPIOL7: now also J200.a23
- net GPIOL8: now also J200.a24
- net GPIOL9: now also J200.a25
- net GPIOR0: now also J200.c16
- net GPIOR1: now also J200.c17
- net GPIOR10: now also J200.c26
- net GPIOR11: now also J200.c27
- net GPIOR12: now also J200.c28
- net GPIOR13: now also J200.c29
- net GPIOR14: now also J200.c30
- net GPIOR15: now also J200.c31
- net GPIOR2: now also J200.c18
- net GPIOR3: now also J200.c19
- net GPIOR4: now also J200.c20
- net GPIOR5: now also J200.c21
- net GPIOR6: now also J200.c22
- net GPIOR7: now also J200.c23
- net GPIOR8: now also J200.c24
- net GPIOR9: now also J200.c25
- net USB1U.D+: now also J200.c2
- net USB1U.D-: now also J200.a2
- new net +12V: J200.a11, J200.a12, J200.b11, J200.b12, J200.c11, J200.c12
- new net +24V: J200.a14, J200.b14, J200.c14
- new net +5v_stdby: J200.a3, J200.b3, J200.c3
- new net CAN1.+: J200.a5, J200.b5, J200.c5
- new net CAN1.-: J200.a6, J200.b6, J200.c6
- new net CAN2.+: J200.a8, J200.b8, J200.c8
- new net CAN2.-: J200.a9, J200.b9, J200.c9
- new net GND: J200.a1, J200.a10, J200.a13, J200.a15, J200.a32, J200.a4, J200.a7, J200.b1, J200.b10, J200.b13, J200.b15, J200.b2, J200.b32, J200.b4, J200.b7, J200.c1, J200.c10, J200.c13, J200.c15, J200.c32, J200.c4, J200.c7

Commit message: [3] Add DIN41612 connector
Connections:
- net CAN1.+: no longer J200.b5, J200.c5
- net CAN1.-: no longer J200.b6, J200.c6
- net CAN2.+: no longer J200.b8, J200.c8
- net CAN2.-: no longer J200.b9, J200.c9
- new net CAN1..+: J200.b5, J200.c5
- new net CAN1..-: J200.b6, J200.c6
- new net CAN2..+: J200.b8, J200.c8
- new net CAN2..-: J200.b9, J200.c9
Other:
- moved on the sheet: J200, U403
