File: backplane.kicad_sch (KiCad schematic)
At the start: 2 parts, among them J200 09031967921, U200 IP4234CZ6,115

Commit message: [#2] WIP: Layout DC-DC converters, MCU
Connections:
- net BACKPLANE.D+: now also U200.3; no longer U200.4
- net BACKPLANE.D-: now also U200.4; no longer U200.3
- net BACKPLANE_U.D+: now also U200.1; no longer U200.6
- net BACKPLANE_U.D-: now also U200.6; no longer U200.1
Changed lines of the file:
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@@
+		)
+	)
+	(label "BACKPLANE.D+"
+		(at 231.14 148.59 180)
+		(effects
+			(font
+				(size 1.27 1.27)
+				(italic yes)
+			)
+			(justify right bottom)
 		)
 	)
@@
 		)
 	)
+	(label "BACKPLANE_U.D-"
+		(at 175.26 143.51 0)
+		(effects
+			(font
+				(size 1.27 1.27)
+				(italic yes)
+			)
+			(justify left bottom)
+		)
+	)
 	(label "GPIOL15"
 		(at 53.34 99.06 0)
@@
 		)
 	)
-	(label "BACKPLANE.D-"
-		(at 228.6 148.59 180)
-		(effects
-			(font
-				(size 1.27 1.27)
-				(italic yes)
-			)
-			(justify right bottom)
-		)
-	)
 	(label "BACKPLANE_U.D+"
 		(at 53.34 25.4 0)
@@
 		)
 	)
-	(label "BACKPLANE_U.D+"
-		(at 175.26 143.51 0)
-		(effects
-			(font
-				(size 1.27 1.27)
-				(italic yes)
-			)
-			(justify left bottom)
-		)
-	)
 	(label "GPIOR0"
 		(at 153.67 60.96 0)
@@
 		)
 	)
-	(label "BACKPLANE_U.D-"
-		(at 175.26 148.59 0)
-		(effects
-			(font
-				(size 1.27 1.27)
-				(italic yes)
-			)
-			(justify left bottom)
-		)
-	)
 	(label "GPIOL10"
 		(at 53.34 86.36 0)
@@
 		)
 	)
+	(label "BACKPLANE_U.D+"
+		(at 175.26 148.59 0)
+		(effects
+			(font
+				(size 1.27 1.27)
+				(italic yes)
+			)
+			(justify left bottom)
+		)
+	)
 	(label "GPIOC0"
 		(at 53.34 144.78 0)
@@
 		)
 	)
-	(label "BACKPLANE.D+"
-		(at 229.87 143.51 180)
-		(effects
-			(font
-				(size 1.27 1.27)
-				(italic yes)
-			)
-			(justify right bottom)
-		)
-	)
 	(label "CAN2.-"
 		(at 220.98 107.95 0)
@@
 		)
 	)
+	(label "BACKPLANE.D-"
+		(at 231.14 143.51 180)
+		(effects
+			(font
+				(size 1.27 1.27)
+				(italic yes)
+			)
+			(justify right bottom)
+		)
+	)

Commit message: [#2] WIP: Layout USB, ST-LINK, move CAN transcievers
Connections:
- net +5v_stdby: no longer U200.5 (VP)
- new net +5V: U200.5 (VP)
Changed lines of the file:
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@@
 			)
 		)
-		(property "Value" "+5v_stdby"
+		(property "Value" "+5V"
 			(at 201.93 130.81 0)
 			(effects

Commit message: [#4] Replace ESD protection with PESD5V0S2BT
Parts:
- removed U200: IP4234CZ6,115, Package_TO_SOT_SMD:SC-74-6_1.55x2.9mm_P0.95mm, symbol Power_Protection:IP4234CZ6
- added U303: PESD5V0S2BT, Package_TO_SOT_SMD:SOT-23, symbol PESD5V0S2BT:PESD5V0S2BT
Connections:
- net BACKPLANE_U.D+ is gone; now on net BACKPLANE.D+: J200.a2
- net BACKPLANE_U.D- is gone; now on net BACKPLANE.D-: J200.c2
- net BACKPLANE.D+: now also U303.2
- net BACKPLANE.D-: now also U303.1
- net GND: now also U303.3

Commit message: [#4] Improve schematic aesthetics, color nets
Parts:
- renumbered U303 to U200
Connections:
- net +5v_stdby renamed +5V_STDBY
Other:
- note added: "CAN"
- note added: "POWER FLAGS"
