File: USB.kicad_sch (KiCad schematic)
At the start: 10 parts, among them J900 USB_C_Receptacle_USB2.0_16P, U800 IP4234CZ6,115, U801 TS3USB30ERSWR

Commit message: [#2] Replace USB switch and power indicator LEDs
Parts:
- removed R800, R801: 10kΩ, PCM_JLCPCB:R_0402, symbol PCM_JLCPCB-Resistors:0402,10kΩ
- removed U801: TS3USB30ERSWR, Package_DFN_QFN:UQFN-10_1.4x1.8mm_P0.4mm, symbol Interface_USB:TS3USB30ERSWR
- added R802, R804: 10kΩ, PCM_JLCPCB:R_0402, symbol PCM_JLCPCB-Resistors:0402,10kΩ
- added R803: 22kΩ, PCM_JLCPCB:R_0402, symbol PCM_JLCPCB-Resistors:0402,22kΩ
- added U801: FSUSB42UMX, Package_DFN_QFN:UQFN-10_1.4x1.8mm_P0.4mm, symbol FSUSB42UMX:FSUSB42UMX
- renumbered J900 to J800, R904 to R800, R905 to R801, R802 to R805
Connections:
- net BACKPLANE.D+: now also U801.5 (HSD1+)
- net BACKPLANE.D-: now also U801.4 (HSD1-)
- net EXTUSB.D+: now also U801.1 (D+)
- net EXTUSB.D-: now also U801.2 (D-)
- net GND: now also R803.2, R804.2, U801.3 (GND)
- net USB2S.D+: now also U801.7 (HSD2+)
- net USB2S.D-: now also U801.6 (HSD2-)
- net VBUS_IN: now also R802.1
- net CC1: now reaches J800.A5 (CC1), R801.1
- net CC2: now reaches J800.B5 (CC2), R800.1
- new net: R802.2, R803.1, U801.10 (SEL)
- new net: R804.1, U801.8 (~{OE})
- new net +3V3: U801.9 (VCC)

Commit message: [#2] WIP: Layout USB
Parts:
- added C312: 100nF, PCM_JLCPCB:C_0402, symbol PCM_JLCPCB-Capacitors:0402,100nF,(2)
Connections:
- net +3V3: now also C312.1
- net GND: now also C312.2
- net USB2S.D+: now also U800.3; no longer U800.4
- net USB2S.D-: now also U800.4; no longer U800.3
- net USB2U.D+: now also J800.A6 (D+), J800.B6 (D+), U800.1; no longer J800.A7 (D-), J800.B7 (D-), U800.6
- net USB2U.D-: now also J800.A7 (D-), J800.B7 (D-), U800.6; no longer J800.A6 (D+), J800.B6 (D+), U800.1
Other:
- moved on the sheet: C800

Commit message: [#4] Replace ESD protection with PESD5V0S2BT
Parts:
- removed U800: IP4234CZ6,115, Package_TO_SOT_SMD:SC-74-6_1.55x2.9mm_P0.95mm, symbol Power_Protection:IP4234CZ6
- added U802: PESD5V0S2BT, Package_TO_SOT_SMD:SOT-23, symbol PESD5V0S2BT:PESD5V0S2BT
Connections:
- net USB2U.D+ is gone; now on net USB2S.D+: J800.A6 (D+), J800.B6 (D+)
- net USB2U.D- is gone; now on net USB2S.D-: J800.A7 (D-), J800.B7 (D-)
- net GND: now also U802.3
- net USB2S.D+: now also U802.2
- net USB2S.D-: now also U802.1
Changed lines of the file:
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@@
+	)
+	(junction
+		(at 123.19 81.28)
+		(diameter 0)
+		(color 0 0 0 0)
+	)
+	(junction
+		(at 118.11 86.36)
+		(diameter 0)
+		(color 0 0 0 0)
 	)
 	(junction
@@
 	(wire
 		(pts
-			(xy 146.05 86.36) (xy 137.16 86.36)
-		)
-		(stroke
-			(width 0)
-			(type default)
-		)
-	)
-	(wire
-		(pts
 			(xy 149.86 85.09) (xy 168.91 85.09)
 		)
@@
 	(wire
 		(pts
-			(xy 81.28 81.28) (xy 116.84 81.28)
+			(xy 81.28 81.28) (xy 123.19 81.28)
 		)
 		(stroke
@@
 	(wire
 		(pts
+			(xy 123.19 81.28) (xy 123.19 87.63)
+		)
+		(stroke
+			(width 0)
+			(type default)
+		)
+	)
+	(wire
+		(pts
 			(xy 223.52 66.04) (xy 223.52 68.58)
 		)
@@
 	(wire
 		(pts
+			(xy 118.11 86.36) (xy 146.05 86.36)
+		)
+		(stroke
+			(width 0)
+			(type default)
+		)
+	)
+	(wire
+		(pts
 			(xy 58.42 120.65) (xy 58.42 121.92)
 		)
@@
 	(wire
 		(pts
-			(xy 146.05 81.28) (xy 137.16 81.28)
-		)
-		(stroke
-			(width 0)
-			(type default)
-		)
-	)
-	(wire
-		(pts
-			(xy 81.28 86.36) (xy 116.84 86.36)
+			(xy 81.28 86.36) (xy 118.11 86.36)
 		)
 		(stroke
@@
 	(wire
 		(pts
-			(xy 127 93.98) (xy 127 96.52)
+			(xy 120.65 100.33) (xy 120.65 102.87)
 		)
 		(stroke
@@
 	(wire
 		(pts
+			(xy 123.19 81.28) (xy 146.05 81.28)
+		)
+		(stroke
+			(width 0)
+			(type default)
+		)
+	)
+	(wire
+		(pts
 			(xy 81.28 73.66) (xy 93.98 73.66)
 		)
@@
 		(pts
 			(xy 127 66.04) (xy 223.52 66.04)
+		)
+		(stroke
+			(width 0)
+			(type default)
+		)
+	)
+	(wire
+		(pts
+			(xy 118.11 87.63) (xy 118.11 86.36)
 		)
 		(stroke
@@
 	(symbol
 		(lib_id "power:GND")
-		(at 127 96.52 0)
+		(at 120.65 102.87 0)
 		(mirror y)
 		(unit 1)
@@
 		(dnp no)
 		(property "Reference" "#PWR0802"
-			(at 127 102.87 0)
+			(at 120.65 109.22 0)
 			(effects
 				(font
@@
 		)
 		(property "Value" "GND"
-			(at 127 100.33 0)
+			(at 120.65 106.68 0)
 			(effects
 				(font
@@
 		)
 		(property "Footprint" ""
-			(at 127 96.52 0)
+			(at 120.65 102.87 0)
 			(effects
 				(font
@@
 		)
 		(property "Datasheet" ""
-			(at 127 96.52 0)
+			(at 120.65 102.87 0)
 			(effects
 				(font
@@
 		)
 		(property "Description" "Power symbol creates a global label with name \"GND\" , ground"
-			(at 127 96.52 0)
+			(at 120.65 102.87 0)
 			(effects
 				(font
@@
 	)
 	(symbol
+		(lib_id "PESD5V0S2BT:PESD5V0S2BT")
+		(at 120.65 95.25 180)
+		(unit 1)
+		(exclude_from_sim no)
+		(in_bom yes)
+		(on_board yes)
+		(dnp no)
+		(property "Reference" "U802"
+			(at 125.73 91.44 0)
+			(effects
+				(font
+					(size 1.27 1.27)
+				)
+				(justify right)
+			)
+		)
+		(property "Value" "PESD5V0S2BT"
+			(at 125.73 93.98 0)
+			(effects
+				(font
+					(size 1.27 1.27)
+				)
+				(justify right)
+			)
+		)
+		(property "Footprint" "Package_TO_SOT_SMD:SOT-23"
+			(at 120.65 95.25 0)
+			(effects
+				(font
+					(size 1.27 1.27)
+				)
+				(hide yes)
+			)
+		)
+		(property "Datasheet" "https://www.lcsc.com/datasheet/lcsc_datasheet_2501101716_HXY-MOSFET-PESD5V0S2BT_C5451656.pdf"
+			(at 120.65 95.25 0)
+			(effects
+				(font
+					(size 1.27 1.27)
+				)
+				(hide yes)
+			)
+		)
+		(property "Description" "11A 8V 8V Bidirectional 5V SOT-23 ESD and Surge Protection (TVS/ESD)"
+			(at 120.65 95.25 0)
+			(effects
+				(font
+					(size 1.27 1.27)
+				)
+				(hide yes)
+			)
+		)
+		(pin "3"
+		)
+		(pin "1"
+		)
+		(pin "2"
+		)
+		(instances
+			(project ""
+				(path "/090a8e41-87a8-4fb1-998b-60a2c0dc4cee/8fd5ae83-0658-4178-9e81-18085647e2bb"
+					(reference "U802")
+					(unit 1)
+				)
+			)
+		)
+	)
+	(symbol
 		(lib_id "power:GND")
 		(at 201.93 110.49 0)
@@
 					(unit 1)
 				)
-			)
-		)
-	)
-	(symbol
-		(lib_id "Power_Protection:IP4234CZ6")
-		(at 127 83.82 0)
-		(unit 1)
-		(exclude_from_sim no)
-		(in_bom yes)
-		(on_board yes)
-		(dnp no)
-		(property "Reference" "U800"
-			(at 130.81 73.152 0)
-			(effects
-				(font
-					(size 1.27 1.27)
-				)
-				(justify left)
-			)
-		)
-		(property "Value" "IP4234CZ6,115"
-			(at 130.81 74.93 0)
-			(effects
-				(font
-					(size 1.27 1.27)
-				)
-				(justify left)
-			)
-		)
-		(property "Footprint" "Package_TO_SOT_SMD:SC-74-6_1.55x2.9mm_P0.95mm"
-			(at 127 99.568 0)
-			(effects
-				(font
-					(size 1.27 1.27)
-				)
-				(hide yes)
-			)
-		)
-		(property "Datasheet" "https://assets.nexperia.com/documents/data-sheet/IP4234CZ6.pdf"
-			(at 127 103.886 0)
-			(effects
-				(font
-					(size 1.27 1.27)
-				)
-				(hide yes)
-			)
-		)
-		(property "Description" "ESD Protection, 2 channel, USB 2.0 to IEC 61000-4-2 level 4, 5.5V, SOT457 (SC-74-6)"
-			(at 127 101.854 0)
-			(effects
-				(font
-					(size 1.27 1.27)
-				)
-				(hide yes)
-			)
-		)
-		(pin "3"
-		)
-		(pin "4"
-		)
-		(pin "5"
-		)
-		(pin "1"
-		)
-		(pin "6"
-		)
-		(pin "2"
-		)
-		(instances
-			(project "base-module"
-				(path "/090a8e41-87a8-4fb1-998b-60a2c0dc4cee/8fd5ae83-0658-4178-9e81-18085647e2bb"
-					(reference "U800")
-					(unit 1)
-				)

Commit message: [#4] Rotate USB connector ESD protection
Connections:
- net USB2S.D+: now also U802.1; no longer U802.2
- net USB2S.D-: now also U802.2; no longer U802.1
Changed lines of the file:
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@@
-	)
-	(junction
-		(at 123.19 81.28)
-		(diameter 0)
-		(color 0 0 0 0)
-	)
-	(junction
-		(at 118.11 86.36)
-		(diameter 0)
-		(color 0 0 0 0)
 	)
 	(junction
@@
 	)
 	(junction
+		(at 123.19 86.36)
+		(diameter 0)
+		(color 0 0 0 0)
+	)
+	(junction
 		(at 207.01 76.2)
 		(diameter 0)
@@
 	)
 	(junction
-		(at 127 66.04)
-		(diameter 0)
-		(color 0 0 0 0)
-	)
-	(junction
 		(at 81.28 86.36)
+		(diameter 0)
+		(color 0 0 0 0)
+	)
+	(junction
+		(at 118.11 81.28)
 		(diameter 0)
 		(color 0 0 0 0)
@@
 	(wire
 		(pts
-			(xy 81.28 81.28) (xy 123.19 81.28)
+			(xy 81.28 81.28) (xy 118.11 81.28)
 		)
 		(stroke
@@
 	(wire
 		(pts
-			(xy 123.19 81.28) (xy 123.19 87.63)
-		)
-		(stroke
-			(width 0)
-			(type default)
-		)
-	)
-	(wire
-		(pts
 			(xy 223.52 66.04) (xy 223.52 68.58)
 		)
@@
 	(wire
 		(pts
-			(xy 118.11 86.36) (xy 146.05 86.36)
-		)
-		(stroke
-			(width 0)
-			(type default)
-		)
-	)
-	(wire
-		(pts
 			(xy 58.42 120.65) (xy 58.42 121.92)
 		)
@@
 	(wire
 		(pts
-			(xy 81.28 66.04) (xy 127 66.04)
-		)
-		(stroke
-			(width 0)
-			(type default)
-		)
-	)
-	(wire
-		(pts
 			(xy 207.01 74.93) (xy 207.01 76.2)
 		)
@@
 	(wire
 		(pts
+			(xy 123.19 86.36) (xy 146.05 86.36)
+		)
+		(stroke
+			(width 0)
+			(type default)
+		)
+	)
+	(wire
+		(pts
 			(xy 58.42 121.92) (xy 58.42 127)
 		)
@@
 	(wire
 		(pts
-			(xy 81.28 86.36) (xy 118.11 86.36)
-		)
-		(stroke
-			(width 0)
-			(type default)
-		)
-	)
-	(wire
-		(pts
 			(xy 149.86 82.55) (xy 146.05 86.36)
 		)
@@
 	(wire
 		(pts
+			(xy 118.11 81.28) (xy 146.05 81.28)
+		)
+		(stroke
+			(width 0)
+			(type default)
+		)
+	)
+	(wire
+		(pts
 			(xy 81.28 83.82) (xy 81.28 86.36)
 		)
@@
 	(wire
 		(pts
+			(xy 81.28 86.36) (xy 123.19 86.36)
+		)
+		(stroke
+			(width 0)
+			(type default)
+		)
+	)
+	(wire
+		(pts
 			(xy 120.65 100.33) (xy 120.65 102.87)
 		)
@@
 	(wire
 		(pts
+			(xy 123.19 86.36) (xy 123.19 87.63)
+		)
+		(stroke
+			(width 0)
+			(type default)
+		)
+	)
+	(wire
+		(pts
 			(xy 201.93 110.49) (xy 201.93 107.95)
 		)
@@
 	(wire
 		(pts
-			(xy 123.19 81.28) (xy 146.05 81.28)
-		)
-		(stroke
-			(width 0)
-			(type default)
-		)
-	)
-	(wire
-		(pts
 			(xy 81.28 73.66) (xy 93.98 73.66)
 		)
@@
 	(wire
 		(pts
-			(xy 127 66.04) (xy 223.52 66.04)
-		)
-		(stroke
-			(width 0)
-			(type default)
-		)
-	)
-	(wire
-		(pts
-			(xy 118.11 87.63) (xy 118.11 86.36)
+			(xy 81.28 66.04) (xy 223.52 66.04)
+		)
+		(stroke
+			(width 0)
+			(type default)
+		)
+	)
+	(wire
+		(pts
+			(xy 118.11 81.28) (xy 118.11 87.63)
 		)
 		(stroke
@@
 		)
 		(stroke
-			(width 0)
-			(type default)
-		)
-	)
-	(wire
-		(pts
-			(xy 127 66.04) (xy 127 73.66)
-		)
-		(stroke

Commit message: [#4] Improve schematic aesthetics, color nets
Connections:
- no-connect marks 0 -> 2
Other:
- moved on the sheet: C800
