File: USB.kicad_sch (KiCad schematic)
At the start: 12 parts, among them J800 USB_C_Receptacle_USB2.0_16P, U801 FSUSB42UMX, U802 PESD5V0S2BT

Commit message: [#12] Change USB TVS
Parts:
- removed U802: PESD5V0S2BT, Package_TO_SOT_SMD:SOT-23, symbol PESD5V0S2BT:PESD5V0S2BT
- added U401: TPD2E2U06DCK, Package_TO_SOT_SMD:SOT-323_SC-70, symbol Power_Protection:TPD2E2U06DCK
Connections:
- net GND: now also U401.3
- net USB2S.D+: now also U401.1
- net USB2S.D-: now also U401.2
Changed lines of the file:
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@@
 	)
 	(junction
-		(at 123.19 86.36)
+		(at 207.01 76.2)
 		(diameter 0)
 		(color 0 0 0 0)
 	)
 	(junction
-		(at 207.01 76.2)
+		(at 110.49 86.36)
 		(diameter 0)
 		(color 0 0 0 0)
@@
 	)
 	(junction
-		(at 118.11 81.28)
+		(at 106.68 81.28)
 		(diameter 0)
 		(color 0 0 0 0)
@@
 	(wire
 		(pts
-			(xy 81.28 81.28) (xy 118.11 81.28)
-		)
-		(stroke
-			(width 0)
-			(type default)
-		)
-	)
-	(wire
-		(pts
 			(xy 201.93 107.95) (xy 199.39 107.95)
 		)
@@
 	(wire
 		(pts
-			(xy 93.98 100.33) (xy 93.98 102.87)
+			(xy 93.98 100.33) (xy 93.98 104.14)
 		)
 		(stroke
@@
 	(wire
 		(pts
-			(xy 118.11 81.28) (xy 146.05 81.28)
+			(xy 106.68 81.28) (xy 146.05 81.28)
+		)
+		(stroke
+			(width 0)
+			(type default)
+		)
+	)
+	(wire
+		(pts
+			(xy 81.28 81.28) (xy 106.68 81.28)
 		)
 		(stroke
@@
 	(wire
 		(pts
+			(xy 110.49 86.36) (xy 110.49 91.44)
+		)
+		(stroke
+			(width 0)
+			(type default)
+		)
+	)
+	(wire
+		(pts
 			(xy 152.4 96.52) (xy 168.91 96.52)
 		)
@@
 	(wire
 		(pts
-			(xy 123.19 86.36) (xy 146.05 86.36)
+			(xy 81.28 86.36) (xy 110.49 86.36)
 		)
 		(stroke
@@
 	(wire
 		(pts
-			(xy 81.28 86.36) (xy 123.19 86.36)
+			(xy 110.49 86.36) (xy 146.05 86.36)
 		)
 		(stroke
@@
 	(wire
 		(pts
-			(xy 120.65 100.33) (xy 120.65 102.87)
+			(xy 119.38 101.6) (xy 119.38 104.14)
 		)
 		(stroke
@@
 	(wire
 		(pts
-			(xy 123.19 86.36) (xy 123.19 87.63)
+			(xy 201.93 119.38) (xy 201.93 107.95)
 		)
 		(stroke
@@
 		)
 	)
-	(wire
+	(bus
 		(pts
-			(xy 201.93 119.38) (xy 201.93 107.95)
+			(xy 149.86 96.52) (xy 149.86 99.06)
 		)
 		(stroke
@@
 		)
 	)
-	(bus
+	(wire
 		(pts
-			(xy 149.86 96.52) (xy 149.86 99.06)
+			(xy 111.76 96.52) (xy 106.68 96.52)
 		)
 		(stroke
@@
 	(wire
 		(pts
-			(xy 118.11 81.28) (xy 118.11 87.63)
+			(xy 139.7 107.95) (xy 148.59 107.95)
 		)
 		(stroke
@@
 	(wire
 		(pts
-			(xy 139.7 107.95) (xy 148.59 107.95)
+			(xy 97.79 90.17) (xy 97.79 71.12)
 		)
 		(stroke
@@
 	(wire
 		(pts
-			(xy 97.79 90.17) (xy 97.79 71.12)
+			(xy 66.04 120.65) (xy 66.04 121.92)
 		)
 		(stroke
@@
 	(wire
 		(pts
-			(xy 66.04 120.65) (xy 66.04 121.92)
+			(xy 157.48 107.95) (xy 168.91 107.95)
 		)
 		(stroke
@@
 	(wire
 		(pts
-			(xy 157.48 107.95) (xy 168.91 107.95)
+			(xy 166.37 105.41) (xy 166.37 110.49)
 		)
 		(stroke
@@
 	(wire
 		(pts
-			(xy 166.37 105.41) (xy 166.37 110.49)
+			(xy 166.37 105.41) (xy 168.91 105.41)
 		)
 		(stroke
@@
 	(wire
 		(pts
-			(xy 166.37 105.41) (xy 168.91 105.41)
+			(xy 106.68 81.28) (xy 106.68 96.52)
 		)
 		(stroke
@@
 	(wire
 		(pts
+			(xy 111.76 91.44) (xy 110.49 91.44)
+		)
+		(stroke
+			(width 0)
+			(type default)
+		)
+	)
+	(wire
+		(pts
 			(xy 93.98 100.33) (xy 97.79 100.33)
 		)
@@
 	(symbol
 		(lib_id "power:GND")
-		(at 120.65 102.87 0)
+		(at 119.38 104.14 0)
 		(mirror y)
 		(unit 1)
@@
 		(dnp no)
 		(property "Reference" "#PWR0802"
-			(at 120.65 109.22 0)
+			(at 119.38 110.49 0)
 			(effects
 				(font
@@
 		)
 		(property "Value" "GND"
-			(at 120.65 106.68 0)
+			(at 119.38 107.95 0)
 			(effects
 				(font
@@
 		)
 		(property "Footprint" ""
-			(at 120.65 102.87 0)
+			(at 119.38 104.14 0)
 			(effects
 				(font
@@
 		)
 		(property "Datasheet" ""
-			(at 120.65 102.87 0)
+			(at 119.38 104.14 0)
 			(effects
 				(font
@@
 		)
 		(property "Description" "Power symbol creates a global label with name \"GND\" , ground"
-			(at 120.65 102.87 0)
+			(at 119.38 104.14 0)
 			(effects
 				(font
@@
 	)
 	(symbol
-		(lib_id "PESD5V0S2BT:PESD5V0S2BT")
-		(at 120.65 95.25 180)
+		(lib_id "Power_Protection:TPD2E2U06DCK")
+		(at 119.38 93.98 0)
 		(unit 1)
 		(exclude_from_sim no)
@@
 		(on_board yes)
 		(dnp no)
-		(property "Reference" "U802"
-			(at 125.73 91.44 0)
+		(fields_autoplaced yes)
+		(property "Reference" "U401"
+			(at 123.19 92.7099 0)
 			(effects
 				(font
 					(size 1.27 1.27)
 				)
-				(justify right)
+				(justify left)
 			)
 		)
-		(property "Value" "PESD5V0S2BT"
-			(at 125.73 93.98 0)
+		(property "Value" "TPD2E2U06DCK"
+			(at 123.19 95.2499 0)
 			(effects
 				(font
 					(size 1.27 1.27)
 				)
-				(justify right)
+				(justify left)
 			)
 		)
-		(property "Footprint" "Package_TO_SOT_SMD:SOT-23"
-			(at 120.65 95.25 0)
+		(property "Footprint" "Package_TO_SOT_SMD:SOT-323_SC-70"
+			(at 99.06 100.33 0)
 			(effects
 				(font
@@
 			)
 		)
-		(property "Datasheet" "https://www.lcsc.com/datasheet/lcsc_datasheet_2501101716_HXY-MOSFET-PESD5V0S2BT_C5451656.pdf"
-			(at 120.65 95.25 0)
+		(property "Datasheet" "http://www.ti.com/lit/ds/symlink/tpd2e2u06.pdf"
+			(at 114.3 88.9 0)
 			(effects
 				(font
@@
 			)
 		)
-		(property "Description" "11A 8V 8V Bidirectional 5V SOT-23 ESD and Surge Protection (TVS/ESD)"
-			(at 120.65 95.25 0)
+		(property "Description" "Dual-Channel High-Speed ESD Protection, SC-70"
+			(at 119.38 93.98 0)
 			(effects
 				(font
@@
 			)
 		)
-		(pin "3"
+		(pin "2"
 		)
 		(pin "1"
 		)
-		(pin "2"
+		(pin "3"
 		)
 		(instances
 			(project ""
 				(path "/090a8e41-87a8-4fb1-998b-60a2c0dc4cee/8fd5ae83-0658-4178-9e81-18085647e2bb"
-					(reference "U802")
+					(reference "U401")
 					(unit 1)
 				)
@@
 	(symbol
 		(lib_id "power:GND")
-		(at 93.98 102.87 0)
+		(at 93.98 104.14 0)
 		(mirror y)
 		(unit 1)
@@
 		(dnp no)
 		(property "Reference" "#PWR0803"
-			(at 93.98 109.22 0)
+			(at 93.98 110.49 0)
 			(effects
 				(font
@@
 		)
 		(property "Value" "GND"
-			(at 93.98 106.68 0)
+			(at 93.98 107.95 0)
 			(effects
 				(font
@@
 		)
 		(property "Footprint" ""
-			(at 93.98 102.87 0)
+			(at 93.98 104.14 0)
 			(effects
 				(font
@@
 		)
 		(property "Datasheet" ""
-			(at 93.98 102.87 0)
+			(at 93.98 104.14 0)
 			(effects
 				(font
@@
 		)
 		(property "Description" "Power symbol creates a global label with name \"GND\" , ground"
-			(at 93.98 102.87 0)
+			(at 93.98 104.14 0)
 			(effects
 				(font

Commit message: Change MCU and update library
Changed MCU from H7 to H5 series due to programming issues with external
loader. Also updated JLCPCB components (not all tho there are still
arround 18 components to fix)
Parts:
- C312, C800, C801: Stock 3851753 -> 5436546
- R800, R801: Stock 2022176 -> 3416329
- R802, R804: Stock 14017682 -> 13746052
- R803: Stock 474609 -> 574595
- R805: Stock 399284 -> 577267
- U801: footprint Package_DFN_QFN:UQFN-10_1.4x1.8mm_P0.4mm -> kicad-footprints:UFQFN-10_1.4x1.8
Other:
- title: ModuCard base module -> ModuCard BM STM32H562VGT6
Changed lines of the file:
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@@
 (kicad_sch
-	(version 20231120)
+	(version 20250114)
 	(generator "eeschema")
-	(generator_version "8.0")
+	(generator_version "9.0")
 	(paper "A4")
 	(title_block
-		(title "ModuCard base module")
-		(date "2025-02-25")
-		(rev "1.0.1")
+		(title "ModuCard BM STM32H562VGT6")
+		(date "2025-04-18")
+		(rev "1.0.0")
 		(company "KoNaR")
 		(comment 1 "Base project authors: Dominik Pluta, Artem Horiunov")
@@
 			)
 		)
-		(property "Stock" "3851753"
+		(property "Stock" "5436546"
 			(at 104.14 69.85 0)
 			(effects
@@
 			)
 		)
-		(property "Stock" "474609"
+		(property "Stock" "574595"
 			(at 157.48 114.3 0)
 			(effects
@@
 			)
 		)
-		(property "Stock" "14017682"
+		(property "Stock" "13746052"
 			(at 166.37 114.3 0)
 			(effects
@@
 		(on_board yes)
 		(dnp no)
-		(property "Reference" "#PWR0802"
+		(property "Reference" "#PWR802"
 			(at 119.38 110.49 0)
 			(effects
@@
 			(project "base-module"
 				(path "/090a8e41-87a8-4fb1-998b-60a2c0dc4cee/8fd5ae83-0658-4178-9e81-18085647e2bb"
-					(reference "#PWR0802")
+					(reference "#PWR802")
 					(unit 1)
 				)
@@
 			)
 		)
-		(property "Stock" "3851753"
+		(property "Stock" "5436546"
 			(at 58.42 116.84 0)
 			(effects
@@
 		(on_board yes)
 		(dnp no)
-		(property "Reference" "#PWR0805"
+		(property "Reference" "#PWR805"
 			(at 201.93 125.73 0)
 			(effects
@@
 			(project "base-module"
 				(path "/090a8e41-87a8-4fb1-998b-60a2c0dc4cee/8fd5ae83-0658-4178-9e81-18085647e2bb"
-					(reference "#PWR0805")
+					(reference "#PWR805")
 					(unit 1)
 				)
@@
 		(on_board yes)
 		(dnp no)
-		(property "Reference" "#PWR0808"
+		(property "Reference" "#PWR808"
 			(at 58.42 133.35 0)
 			(effects
@@
 			(project "base-module"
 				(path "/090a8e41-87a8-4fb1-998b-60a2c0dc4cee/8fd5ae83-0658-4178-9e81-18085647e2bb"
-					(reference "#PWR0808")
+					(reference "#PWR808")
 					(unit 1)
 				)
@@
 		(on_board yes)
 		(dnp no)
-		(property "Reference" "#PWR0804"
+		(property "Reference" "#PWR804"
 			(at 66.04 110.49 0)
 			(effects
@@
 			(project "base-module"
 				(path "/090a8e41-87a8-4fb1-998b-60a2c0dc4cee/8fd5ae83-0658-4178-9e81-18085647e2bb"
-					(reference "#PWR0804")
+					(reference "#PWR804")
 					(unit 1)
 				)
@@
 		(on_board yes)
 		(dnp no)
-		(property "Reference" "#PWR0806"
+		(property "Reference" "#PWR806"
 			(at 157.48 125.73 0)
 			(effects
@@
 			(project "base-module"
 				(path "/090a8e41-87a8-4fb1-998b-60a2c0dc4cee/8fd5ae83-0658-4178-9e81-18085647e2bb"
-					(reference "#PWR0806")
+					(reference "#PWR806")
 					(unit 1)
 				)
@@
 		(on_board yes)
 		(dnp no)
-		(property "Reference" "#PWR0807"
+		(property "Reference" "#PWR807"
 			(at 166.37 125.73 0)
 			(effects
@@
 			(project "base-module"
 				(path "/090a8e41-87a8-4fb1-998b-60a2c0dc4cee/8fd5ae83-0658-4178-9e81-18085647e2bb"
-					(reference "#PWR0807")
+					(reference "#PWR807")
 					(unit 1)
 				)
@@
 		(on_board yes)
 		(dnp no)
-		(property "Reference" "#PWR0800"
+		(property "Reference" "#PWR800"
 			(at 104.14 81.28 0)
 			(effects
@@
 			(project "base-module"
 				(path "/090a8e41-87a8-4fb1-998b-60a2c0dc4cee/8fd5ae83-0658-4178-9e81-18085647e2bb"
-					(reference "#PWR0800")
+					(reference "#PWR800")
 					(unit 1)
 				)
@@
 		(on_board yes)
 		(dnp no)
-		(property "Reference" "#PWR0330"
+		(property "Reference" "#PWR330"
 			(at 207.01 91.44 0)
 			(effects
@@
 			(project "base-module"
 				(path "/090a8e41-87a8-4fb1-998b-60a2c0dc4cee/8fd5ae83-0658-4178-9e81-18085647e2bb"
-					(reference "#PWR0330")
+					(reference "#PWR330")
 					(unit 1)
 				)
@@
 			)
 		)
-		(property "Footprint" "Package_DFN_QFN:UQFN-10_1.4x1.8mm_P0.4mm"
+		(property "Footprint" "kicad-footprints:UFQFN-10_1.4x1.8"
 			(at 182.88 75.184 0)
 			(effects
@@
 			)
 		)
-		(property "Stock" "3851753"
+		(property "Stock" "5436546"
 			(at 207.01 80.01 0)
 			(effects
@@
 			)
 		)
-		(property "Stock" "399284"
+		(property "Stock" "577267"
 			(at 66.04 116.84 0)
 			(effects
@@
 	)
 	(symbol
-		(lib_name "USB_C_Receptacle_USB2.0_16P_1")
 		(lib_id "Connector:USB_C_Receptacle_USB2.0_16P")
 		(at 66.04 81.28 0)
@@
 			)
 		)
-		(property "Stock" "2022176"
+		(property "Stock" "3416329"
 			(at 97.79 93.98 0)
 			(effects
@@
 		(on_board yes)
 		(dnp no)
-		(property "Reference" "#PWR0801"
+		(property "Reference" "#PWR801"
 			(at 207.01 78.74 0)
 			(effects
@@
 			(project "base-module"
 				(path "/090a8e41-87a8-4fb1-998b-60a2c0dc4cee/8fd5ae83-0658-4178-9e81-18085647e2bb"
-					(reference "#PWR0801")
+					(reference "#PWR801")
 					(unit 1)
 				)
@@
 			)
 		)
-		(property "Stock" "2022176"
+		(property "Stock" "3416329"
 			(at 93.98 93.98 0)
 			(effects
@@
 			)
 		)
-		(property "Stock" "14017682"
+		(property "Stock" "13746052"
 			(at 152.4 107.95 0)
 			(effects
@@
 		(on_board yes)
 		(dnp no)
-		(property "Reference" "#PWR0803"
+		(property "Reference" "#PWR803"
 			(at 93.98 110.49 0)
 			(effects
@@
 			(project "base-module"
 				(path "/090a8e41-87a8-4fb1-998b-60a2c0dc4cee/8fd5ae83-0658-4178-9e81-18085647e2bb"
-					(reference "#PWR0803")
+					(reference "#PWR803")
 					(unit 1)
 				)

Commit message: [REV2] board finshed, schematics and leyout
Other:
- title: ModuCard BM STM32H562VGT6 -> ModuCard nav module
Changed lines of the file:
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@@
 	(paper "A4")
 	(title_block
-		(title "ModuCard BM STM32H562VGT6")
-		(date "2025-04-18")
+		(title "ModuCard nav module")
+		(date "2025-04-20")
 		(rev "1.1.0")
 		(company "KoNaR")
 		(comment 1 "Base project authors: Dominik Pluta, Artem Horiunov")
-		(comment 2 "Project author: <author>")
+		(comment 2 "Project author: Patryk Dudziński")
 	)
 	(junction
