File: mcu.kicad_sch (KiCad schematic)
At the start: 0 parts

Commit message: Add usb schematic
Parts:
- added C401, C408, C410, C412, C413: 4u7, Capacitor_SMD:C_0402_1005Metric, symbol Device:C_Small
- added C402, C403, C404, C405, C409, C411: 100nF, Capacitor_SMD:C_0402_1005Metric, symbol Device:C_Small
- added C406, C407, C414, C415: 22p, Capacitor_SMD:C_0402_1005Metric, symbol Device:C_Small
- added FB401: 1u, symbol Device:FerriteBead_Small
- added R401, R402: 10k, symbol Device:R_Small
- added R403: 100R, symbol Device:R_Small
- added R404, R405, R406, R409: 0R, symbol Device:R_Small
- added R407, R408: 1k, symbol Device:R_Small
- added SW401, SW402: SW_Push, symbol Switch:SW_Push
- added TP401, TP402: TestPoint, symbol Connector:TestPoint
- added U401: STM32F446RETx, Package_QFP:LQFP-64_10x10mm_P0.5mm, symbol MCU_ST_STM32F4:STM32F446RETx
- added Y401: 8MHz, symbol Device:Crystal_Small
- added Y402: 32.768kHz, symbol Device:Crystal_Small
Connections:
- net NRST: now also C409.2, R402.2, R403.1, R403.2, SW401.1, U401.7 (NRST)
- net SWCLK: now also TP402.1, U401.49 (PA14)
- net SWDIO: now also TP401.1, U401.46 (PA13)
- new net: C408.2, R405.1, R406.1
- new net: R404.2, R405.2, U401.31 (VSS)
- new net: C410.2, FB401.2, U401.13 (VDDA)
- new net: R406.2, U401.30 (VCAP_1)
- new net: C413.2, R409.2, U401.47 (VSS)
- new net: R408.2, SW402.2
- new net +3V3: C401.2, C402.2, C403.2, C404.2, C405.2, C411.2, FB401.1, R402.1, SW402.1, U401.1 (VBAT), U401.19 (VDD), U401.32 (VDD), U401.48 (VDD), U401.64 (VDD)
- new net BOOT0: C412.2, R401.1, R407.2, R408.1, U401.60 (BOOT0)
- new net BOOT_EN: R407.1, U401.59 (PB7)
- new net CAN1_RX: U401.57 (PB5)
- new net CAN1_TX: U401.58 (PB6)
- new net CAN2_RX: U401.61 (PB8)
- new net CAN2_TX: U401.62 (PB9)
- new net GND: C401.1, C402.1, C403.1, C404.1, C405.1, C406.1, C407.1, C408.1, C409.1, C410.1, C411.1, C412.1, C413.1, C414.1, C415.1, R401.2, R404.1, R409.1, SW401.2, U401.12 (VSSA), U401.18 (VSS), U401.63 (VSS)
- new net LSE_OSC_IN: C414.2, U401.3 (PC14), Y402.1
- new net LSE_OSC_OUT: C415.2, U401.4 (PC15), Y402.2
- new net OSC_IN: C406.2, U401.5 (PH0), Y401.1
- new net OSC_OUT: C407.2, U401.6 (PH1), Y401.2
- new net PA0: U401.14 (PA0)
- new net PA1: U401.15 (PA1)
- new net PA10: U401.43 (PA10)
- new net PA11: U401.44 (PA11)
- new net PA12: U401.45 (PA12)
- new net PA15: U401.50 (PA15)
- new net PA2: U401.16 (PA2)
- new net PA3: U401.17 (PA3)
- new net PA4: U401.20 (PA4)
- new net PA5: U401.21 (PA5)
- new net PA6: U401.22 (PA6)
- new net PA7: U401.23 (PA7)
- new net PA8: U401.41 (PA8)
- new net PA9: U401.42 (PA9)
- new net PB0: U401.26 (PB0)
- new net PB1: U401.27 (PB1)
- new net PB10: U401.29 (PB10)
- new net PB12: U401.33 (PB12)
- new net PB13: U401.34 (PB13)
- new net PB14: U401.35 (PB14)
- new net PB15: U401.36 (PB15)
- new net PB2: U401.28 (PB2)
- new net PB3: U401.55 (PB3)
- new net PB4: U401.56 (PB4)
- new net PC0: U401.8 (PC0)
- new net PC1: U401.9 (PC1)
- new net PC10: U401.51 (PC10)
- new net PC11: U401.52 (PC11)
- new net PC12: U401.53 (PC12)
- new net PC13: U401.2 (PC13)
- new net PC2: U401.10 (PC2)
- new net PC3: U401.11 (PC3)
- new net PC4: U401.24 (PC4)
- new net PC5: U401.25 (PC5)
- new net PC6: U401.37 (PC6)
- new net PC7: U401.38 (PC7)
- new net PC8: U401.39 (PC8)
- new net PC9: U401.40 (PC9)
- new net PD2: U401.54 (PD2)
Other:
- note added: "Boot EN can be pulled up with BOOT_EN pin C412 will retain voltage on boot0 pin during MCU reboot routine"
- note added: "C406=C407 = (CL - 4pF) * 2"
- note added: "C414=C415 = (CL - 4pF) * 2"
- note added: "NOTICE:"
- note added: "POPULATE:"
- note added: "REMOVE:"
- note added: "RESET BUTTON"
- note added: "To use STM32F405/STM32F415 line instead of STM32F446: C413 and R404 R406, R404 and R409"

Commit message: [3] Add USB power + data schematic
Connections:
- net PA5 renamed USER_LED1
- net PC13 renamed USER_BTN1
Other:
- moved on the sheet: C409, R402, R403, SW401

Commit message: [3] Add USB hub, draft new MCU
Parts:
- removed C406, C407, C414, C415: 22p, Capacitor_SMD:C_0402_1005Metric, symbol Device:C_Small
- removed C408, C413: 4u7, Capacitor_SMD:C_0402_1005Metric, symbol Device:C_Small
- removed R404, R405, R406, R409: 0R, symbol Device:R_Small
- removed TP401, TP402: TestPoint, symbol Connector:TestPoint
- removed U401: STM32F446RETx, Package_QFP:LQFP-64_10x10mm_P0.5mm, symbol MCU_ST_STM32F4:STM32F446RETx
- removed Y401: 8MHz, symbol Device:Crystal_Small
- removed Y402: 32.768kHz, symbol Device:Crystal_Small
- added C408, C413: 22pF, PCM_JLCPCB:C_0402, symbol PCM_JLCPCB-Capacitors:0402,22pF
- added U407: STM32F750V8Tx, Package_QFP:LQFP-100_14x14mm_P0.5mm, symbol MCU_ST_STM32F7:STM32F750V8Tx
- added X402: X322512MSB4SI, PCM_JLCPCB:CRYSTAL-SMD_4P-L3.2-W2.5-BL, symbol PCM_JLCPCB-Crystals:Crystal, 12MHz, 20pF
Connections:
- net +3V3: now also U407.100 (VDD), U407.11 (VDD), U407.27 (VDD), U407.50 (VDD), U407.75 (VDD)
- net BOOT_EN: now also U407.94 (BOOT0)
- net GND: now also C408.2, C413.2, U407.10 (VSS), U407.19 (VSSA), U407.26 (VSS), U407.49 (VSS), U407.74 (VSS), U407.99 (VSS), X402.2 (GND), X402.4 (GND)
- net NRST: now also U407.14 (NRST)
- net OSC_IN: now also C408.1, X402.1 (OSC)
- net OSC_OUT: now also C413.1, X402.3 (OSC)
- net PA0: now also U407.22 (PA0)
- net PA1: now also U407.23 (PA1)
- net PA10: now also U407.69 (PA10)
- net PA11: now also U407.70 (PA11)
- net PA12: now also U407.71 (PA12)
- net PA15: now also U407.77 (PA15)
- net PA2: now also U407.24 (PA2)
- net PA3: now also U407.25 (PA3)
- net PA4: now also U407.28 (PA4)
- net PA6: now also U407.30 (PA6)
- net PA7: now also U407.31 (PA7)
- net PA8: now also U407.67 (PA8)
- net PA9: now also U407.68 (PA9)
- net PB0: now also U407.34 (PB0)
- net PB1: now also U407.35 (PB1)
- net PB10: now also U407.46 (PB10)
- net PB12: now also U407.51 (PB12)
- net PB13: now also U407.52 (PB13)
- net PB14: now also U407.53 (PB14)
- net PB15: now also U407.54 (PB15)
- net PB2: now also U407.36 (PB2)
- net PB3: now also U407.89 (PB3)
- net PB4: now also U407.90 (PB4)
- net PC0: now also U407.15 (PC0)
- net PC1: now also U407.16 (PC1)
- net PC10: now also U407.78 (PC10)
- net PC11: now also U407.79 (PC11)
- net PC12: now also U407.80 (PC12)
- net PC2: now also U407.17 (PC2)
- net PC3: now also U407.18 (PC3)
- net PC4: now also U407.32 (PC4)
- net PC5: now also U407.33 (PC5)
- net PC6: now also U407.63 (PC6)
- net PC7: now also U407.64 (PC7)
- net PC8: now also U407.65 (PC8)
- net PC9: now also U407.66 (PC9)
- net at C410.2, FB401.2: now also U407.21 (VDDA)
- net BOOT0: no longer names the net of C412.2, R401.1, R407.2, R408.1
- new net PA13: U407.72 (PA13)
- new net PA14: U407.76 (PA14)
- new net PA5: U407.29 (PA5)
- new net PB11: U407.47 (PB11)
- new net PB5: U407.91 (PB5)
- new net PB6: U407.92 (PB6)
- new net PB7: U407.93 (PB7)
- new net PB8: U407.95 (PB8)
- new net PB9: U407.96 (PB9)
- new net PC13: U407.7 (PC13)
- new net PC14: U407.8 (PC14)
- new net PC15: U407.9 (PC15)
Other:
- note removed: "C406=C407 = (CL - 4pF) * 2"
- note removed: "C414=C415 = (CL - 4pF) * 2"
- note removed: "POPULATE:"
- note removed: "REMOVE:"
- note removed: "To use STM32F405/STM32F415 line instead of STM32F446: C413 and R404 R406, R404 and R409"
- moved on the sheet: C409, R402, R403, SW401

Commit message: [3] Add mcu pinout pt1
Connections:
- net BOOT_EN: no longer U407.94 (BOOT0)
- net BOOT0: now reaches C412.2, R401.1, R407.2, R408.1
- net BOOT0: now also U407.94 (BOOT0)
- net PE2: now reaches U407.1 (PE2)
- net PH0: now reaches U407.12 (PH0)
- net PH1: now reaches U407.13 (PH1)
- net PE3: now reaches U407.2 (PE3)
- net VREF+: now reaches U407.20 (VREF+)
- net PE4: now reaches U407.3 (PE4)
- net PE7: now reaches U407.37 (PE7)
- net PE8: now reaches U407.38 (PE8)
- net PE9: now reaches U407.39 (PE9)
- net PE5: now reaches U407.4 (PE5)
- net PE10: now reaches U407.40 (PE10)
- net PE11: now reaches U407.41 (PE11)
- net PE12: now reaches U407.42 (PE12)
- net PE13: now reaches U407.43 (PE13)
- net PE14: now reaches U407.44 (PE14)
- net PE15: now reaches U407.45 (PE15)
- net VCAP_1: now reaches U407.48 (VCAP_1)
- net PE6: now reaches U407.5 (PE6)
- net PD8: now reaches U407.55 (PD8)
- net PD9: now reaches U407.56 (PD9)
- net PD10: now reaches U407.57 (PD10)
- net PD11: now reaches U407.58 (PD11)
- net PD12: now reaches U407.59 (PD12)
- net PD13: now reaches U407.60 (PD13)
- net PD14: now reaches U407.61 (PD14)
- net PD15: now reaches U407.62 (PD15)
- net VCAP_2: now reaches U407.73 (VCAP_2)
- net PD0: now reaches U407.81 (PD0)
- net PD1: now reaches U407.82 (PD1)
- net PD2: now reaches U407.83 (PD2)
- net PD3: now reaches U407.84 (PD3)
- net PD4: now reaches U407.85 (PD4)
- net PD5: now reaches U407.86 (PD5)
- net PD6: now reaches U407.87 (PD6)
- net PD7: now reaches U407.88 (PD7)
- net PE0: now reaches U407.97 (PE0)
- net PE1: now reaches U407.98 (PE1)
Other:
- note added: "PB7"
- moved on the sheet: R407, R408, SW402

Commit message: Fix St-link schematic errors
Parts:
- removed C401, C410: 4u7, Capacitor_SMD:C_0402_1005Metric, symbol Device:C_Small
- removed C402, C403, C404, C405, C411: 100nF, Capacitor_SMD:C_0402_1005Metric, symbol Device:C_Small
- removed FB401: 1u, symbol Device:FerriteBead_Small
- added C401, C402, C403, C404, C406, C410, C414: 100nF, PCM_JLCPCB:C_0402, symbol PCM_JLCPCB-Capacitors:0402,100nF,(2)
- added C405, C407, C411: 10uF, PCM_JLCPCB:C_0402, symbol PCM_JLCPCB-Capacitors:0402,10uF
- added C415, C419: 2.2uF, PCM_JLCPCB:C_0402, symbol PCM_JLCPCB-Capacitors:0402,2.2uF
- added FB401: ~, PCM_JLCPCB:FB_0603, symbol PCM_JLCPCB-Inductors:Ferrite,0603
Connections:
- net PB5 is gone; now on net CAN2.RX: U407.91 (PB5)
- net PB6 is gone; now on net CAN2.TX: U407.92 (PB6)
- net PB7 is gone; now on net BOOT_EN: U407.93 (PB7)
- net PB8 is gone; now on net I2C1.SCL: U407.95 (PB8)
- net PB9 is gone; now on net I2C1.SCL: U407.96 (PB9)
- net PD0 is gone; now on net CAN1.RX: U407.81 (PD0)
- net PD1 is gone; now on net CAN1.TX: U407.82 (PD1)
- net +3V3: now also U407.6 (VBAT), C401.1, C402.1, C403.1, C404.1, C405.1, C406.1, C411.1, C414.1, FB401.2
- net GND: now also C401.2, C402.2, C403.2, C404.2, C405.2, C406.2, C407.2, C410.2, C411.2, C414.2, C415.2, C419.2
- net VCAP_1: now also C419.1
- net VCAP_2: now also C415.1
- net at U407.21 (VDDA): now also C407.1, C410.1, FB401.1
Other:
- note added: "CAN1"
- note added: "CAN2"
- note added: "I2C1"
- note added: "I2C2"
- note added: "SWD"
- note added: "USB"
- note removed: "PB7"
- moved on the sheet: C408, C413

Commit message: Add QSPI flash to MCU
Connections:
- net NRST: no longer U407.14 (NRST)
- new net ~{RST}: U407.14 (NRST)
Other:
- removed sheet CAN transceiver 1
- removed sheet CAN transceiver 2
- note added: "(BANK 1)"
- note added: "QSPI1"
