File: mcu.kicad_sch (KiCad schematic)
At the start: 25 parts, among them SW400 TL2243, U400 STM32F750V8Tx, X400 X322512MSB4SI

Commit message: [#2] Replace USB switch and power indicator LEDs
Parts:
- SW400: footprint kicad-footprints:TL2243 -> TL2243:TL2243
Changed lines of the file:
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@@
 			)
 		)
-		(property "Footprint" "kicad-footprints:TL2243"
+		(property "Footprint" "TL2243:TL2243"
 			(at 52.07 166.37 0)
 			(effects
@@
 			)
 		)
-		(property "Footprint" "kicad-footprints:TL2243"
+		(property "Footprint" "TL2243:TL2243"
 			(at 39.37 43.18 0)
 			(effects

Commit message: [#2] WIP: Layout DC-DC converters, MCU
Parts:
- added X300: Q13FC1350000400, PCM_JLCPCB:FC-135R_L3.2-W1.5, symbol PCM_JLCPCB-Crystals:Crystal, 32.768kHz, 13pF
Connections:
- net PH0 is gone; now on net OSC_IN: U400.12 (PH0)
- net PH1 is gone; now on net OSC_OUT: U400.13 (PH1)
- no-connect marks 68 -> 66

Commit message: [#2] Fix MCU model, draft QSPI connection
Parts:
- removed U400: STM32F750V8Tx, Package_QFP:LQFP-100_14x14mm_P0.5mm, symbol MCU_ST_STM32F7:STM32F750V8Tx
- added U400: STM32H750VBTx, Package_QFP:LQFP-100_14x14mm_P0.5mm, symbol MCU_ST_STM32H7:STM32H750VBTx
Connections:
- net +3V3: now also U400.100 (VDD), U400.11 (VDD), U400.27 (VDD), U400.50 (VDD), U400.6 (VBAT), U400.75 (VDD)
- net BOOT0: now also U400.94 (BOOT0)
- net BOOT_EN: now also U400.93 (PB7)
- net CAN1.RX: now also U400.81 (PD0)
- net CAN1.TX: now also U400.82 (PD1)
- net CAN2.RX: now also U400.91 (PB5)
- net CAN2.TX: now also U400.92 (PB6)
- net GND: now also U400.10 (VSS), U400.19 (VSSA), U400.26 (VSS), U400.49 (VSS), U400.74 (VSS), U400.99 (VSS)
- net I2C1.SCL: now also U400.95 (PB8)
- net I2C1.SDA: now also U400.96 (PB9)
- net OSC_IN: now also U400.12 (PH0)
- net OSC_OUT: now also U400.13 (PH1)
- net PA0: now also U400.22 (PA0)
- net PA1: now also U400.23 (PA1)
- net PA10: now also U400.69 (PA10)
- net PA15: now also U400.77 (PA15)
- net PA2: now also U400.24 (PA2)
- net PA3: now also U400.25 (PA3)
- net PA4: now also U400.28 (PA4)
- net PA5: now also U400.29 (PA5)
- net PA6: now also U400.30 (PA6)
- net PA7: now also U400.31 (PA7)
- net PA8: now also U400.67 (PA8)
- net PA9: now also U400.68 (PA9)
- net PB0: now also U400.34 (PB0)
- net PB1: now also U400.35 (PB1)
- net PB11: now also U400.47 (PB11)
- net PB12: now also U400.51 (PB12)
- net PB13: now also U400.52 (PB13)
- net PB14: now also U400.53 (PB14)
- net PB15: now also U400.54 (PB15)
- net PB3: now also U400.89 (PB3)
- net PB4: now also U400.90 (PB4)
- net PC0: now also U400.15 (PC0)
- net PC1: now also U400.16 (PC1)
- net PC10: now also U400.78 (PC10)
- net PC11: now also U400.79 (PC11)
- net PC12: now also U400.80 (PC12)
- net PC13: now also U400.7 (PC13)
- net PC14: now also U400.8 (PC14)
- net PC15: now also U400.9 (PC15)
- net PC2: now also U400.17 (PC2_C)
- net PC3: now also U400.18 (PC3_C)
- net PC4: now also U400.32 (PC4)
- net PC5: now also U400.33 (PC5)
- net PC6: now also U400.63 (PC6)
- net PC7: now also U400.64 (PC7)
- net PC8: now also U400.65 (PC8)
- net PC9: now also U400.66 (PC9)
- net PD10: now also U400.57 (PD10)
- net PD14: now also U400.61 (PD14)
- net PD15: now also U400.62 (PD15)
- net PD2: now also U400.83 (PD2)
- net PD3: now also U400.84 (PD3)
- net PD4: now also U400.85 (PD4)
- net PD5: now also U400.86 (PD5)
- net PD6: now also U400.87 (PD6)
- net PD7: now also U400.88 (PD7)
- net PD8: now also U400.55 (PD8)
- net PD9: now also U400.56 (PD9)
- net PE0: now also U400.97 (PE0)
- net PE1: now also U400.98 (PE1)
- net PE10: now also U400.40 (PE10)
- net PE11: now also U400.41 (PE11)
- net PE12: now also U400.42 (PE12)
- net PE13: now also U400.43 (PE13)
- net PE14: now also U400.44 (PE14)
- net PE15: now also U400.45 (PE15)
- net PE3: now also U400.2 (PE3)
- net PE4: now also U400.3 (PE4)
- net PE5: now also U400.4 (PE5)
- net PE6: now also U400.5 (PE6)
- net PE7: now also U400.37 (PE7)
- net PE8: now also U400.38 (PE8)
- net PE9: now also U400.39 (PE9)
- net QSPI1.CS: now also U400.46 (PB10)
- net QSPI1.IO0: now also U400.58 (PD11)
- net QSPI1.IO1: now also U400.59 (PD12)
- net QSPI1.IO2: now also U400.1 (PE2)
- net QSPI1.IO3: now also U400.60 (PD13)
- net QSPI1.SCLK: now also U400.36 (PB2)
- net SWD.SWCLK: now also U400.76 (PA14)
- net SWD.SWDIO: now also U400.72 (PA13)
- net SWD.~{RST}: now also U400.14 (NRST)
- net USB_MCU.D+: now also U400.71 (PA12)
- net USB_MCU.D-: now also U400.70 (PA11)
- net VCAP_1: now also U400.48 (VCAP)
- net VCAP_2: now also U400.73 (VCAP)
- net VREF+: now also U400.20 (VREF+)
- net at C406.1, C407.1, FB400.1: now also U400.21 (VDDA)
Other:
- moved on the sheet: C400, C401, C402, C403, C404, C405, C406, C407, C408, C409, FB400

Commit message: [#2] Add LSE oscillator, draft CAN RX/TX tracks, ensure copper balance
Parts:
- added C313, C314: 18pF, PCM_JLCPCB:C_0402, symbol PCM_JLCPCB-Capacitors:0402,18pF
Connections:
- net PC14 is gone; now on net OSC32_IN: U400.8 (PC14)
- net PC15 is gone; now on net OSC32_OUT: U400.9 (PC15)
- net GND: now also C313.2, C314.2
- net OSC32_OUT: now reaches X300.1
- net OSC32_OUT: now also C313.1
- net OSC32_IN: now reaches X300.2
- net OSC32_IN: now also C314.1
- no-connect marks 66 -> 64
Other:
- moved on the sheet: X300

Commit message: [#2] Route everything except for some test points, fix LED and button configuration
Parts:
- removed R400: 1kΩ, PCM_JLCPCB:R_0402, symbol PCM_JLCPCB-Resistors:0402,1kΩ
- added C416: 100nF, PCM_JLCPCB:C_0402, symbol PCM_JLCPCB-Capacitors:0402,100nF,(2)
- added LED300, LED301: FixLed307, FixLed307:FixLed307, symbol FixLed307:FixLed307
- added R400, R407: 1.2kΩ, PCM_JLCPCB:R_0402, symbol PCM_JLCPCB-Resistors:0402,1.2kΩ
- added R405: 10kΩ, PCM_JLCPCB:R_0402, symbol PCM_JLCPCB-Resistors:0402,10kΩ
- added R406: 100Ω, PCM_JLCPCB:R_0402, symbol PCM_JLCPCB-Resistors:0402,100Ω
- added R408: 470Ω, PCM_JLCPCB:R_0402, symbol PCM_JLCPCB-Resistors:0402,470Ω
- added R409: 120Ω, PCM_JLCPCB:R_0402, symbol PCM_JLCPCB-Resistors:0402,120Ω
Connections:
- net +3V3: now also R405.1, R409.1; no longer SW400.4
- net GND: now also SW400.1, C416.2, LED300.2, LED300.4, LED301.2, LED301.4
- net PE3 renamed USER_LED_1
- net USER_LED_1: now also R400.1
- net PE4 renamed USER_LED_2
- net USER_LED_2: now also R407.1
- net PE5 renamed STATUS_LED
- net STATUS_LED: now also R408.1
- net PE6 renamed USR_BUTTON
- net USR_BUTTON: now also SW400.4, R406.2
- new net: LED300.3, R407.2
- new net: LED301.3, R409.2
- new net: LED300.1, R400.2
- new net: LED301.1, R408.2
- new net USR_BTN: C416.1, R405.2, R406.1
- no-connect marks 64 -> 60
Other:
- note added: "POWER INDICATOR LEDs"
- note added: "Target I_{LED} = 10mA"
- moved on the sheet: C313, C314, SW400A, X300

Commit message: [#2] Finish layout
Connections:
- net PB12 is gone; now on net CAN2.RX: U400.51 (PB12)
- net PB13 is gone; now on net CAN2.TX: U400.52 (PB13)
- net CAN2.RX: no longer U400.91 (PB5)
- net CAN2.TX: no longer U400.92 (PB6)
- new net PB5: U400.91 (PB5)
- new net PB6: U400.92 (PB6)
Other:
- note added: "Target I_{LED} = 5mA"
- note removed: "Target I_{LED} = 10mA"
Changed lines of the file:
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@@
 	)
 	(no_connect
+		(at 162.56 102.87)
+	)
+	(no_connect
 		(at 162.56 62.23)
 	)
@@
 	)
 	(no_connect
-		(at 162.56 120.65)
-	)
-	(no_connect
 		(at 95.25 97.79)
 	)
@@
 	)
 	(no_connect
+		(at 162.56 105.41)
+	)
+	(no_connect
 		(at 95.25 105.41)
 	)
@@
 	)
 	(no_connect
-		(at 162.56 123.19)
-	)
-	(no_connect
 		(at 95.25 148.59)
 	)
@@
 	(wire
 		(pts
+			(xy 162.56 105.41) (xy 149.86 105.41)
+		)
+		(stroke
+			(width 0)
+			(type default)
+		)
+	)
+	(wire
+		(pts
 			(xy 95.25 120.65) (xy 104.14 120.65)
 		)
@@
 	(wire
 		(pts
+			(xy 162.56 102.87) (xy 149.86 102.87)
+		)
+		(stroke
+			(width 0)
+			(type default)
+		)
+	)
+	(wire
+		(pts
 			(xy 67.31 110.49) (xy 67.31 115.57)
 		)
@@
 	(wire
 		(pts
-			(xy 149.86 105.41) (xy 162.56 105.41)
-		)
-		(stroke
-			(width 0)
-			(type default)
-		)
-	)
-	(wire
-		(pts
 			(xy 85.09 27.94) (xy 85.09 29.21)
 		)
@@
 	(wire
 		(pts
-			(xy 149.86 102.87) (xy 162.56 102.87)
-		)
-		(stroke
-			(width 0)
-			(type default)
-		)
-	)
-	(wire
-		(pts
 			(xy 92.71 80.01) (xy 104.14 80.01)
 		)
@@
 		)
 	)
-	(text "Target I_{LED} = 10mA"
+	(text "Target I_{LED} = 5mA"
 		(exclude_from_sim no)
 		(at 238.506 70.104 0)
@@
 		)
 	)
+	(label "CAN2.RX"
+		(at 162.56 120.65 180)
+		(effects
+			(font
+				(size 1.27 1.27)
+			)
+			(justify right bottom)
+		)
+	)
 	(label "OSC32_IN"
 		(at 219.71 144.78 180)
@@
 		)
 	)
-	(label "PB12"
-		(at 162.56 120.65 180)
-		(effects
-			(font
-				(size 1.27 1.27)
-			)
-			(justify right bottom)
-		)
-	)
 	(label "PE11"
 		(at 95.25 97.79 0)
@@
 		)
 	)
-	(label "CAN2.TX"
-		(at 162.56 105.41 180)
-		(effects
-			(font
-				(size 1.27 1.27)
-			)
-			(justify right bottom)
-		)
-	)
 	(label "QSPI1.IO2"
 		(at 182.88 48.26 0)
@@
 		)
 	)
-	(label "PB13"
-		(at 162.56 123.19 180)
+	(label "BOOT0"
+		(at 95.25 52.07 0)
 		(effects
 			(font
 				(size 1.27 1.27)
 			)
-			(justify right bottom)
+			(justify left bottom)
 		)
 	)
-	(label "BOOT0"
-		(at 95.25 52.07 0)
+	(label "PC10"
+		(at 162.56 158.75 180)
 		(effects
 			(font
 				(size 1.27 1.27)
 			)
-			(justify left bottom)
+			(justify right bottom)
 		)
 	)
-	(label "PC10"
-		(at 162.56 158.75 180)
+	(label "PB6"
+		(at 162.56 105.41 180)
 		(effects
 			(font
@@
 		)
 	)
-	(label "PE9"
-		(at 95.25 92.71 0)
+	(label "PB5"
+		(at 162.56 102.87 180)
 		(effects
 			(font
 				(size 1.27 1.27)
 			)
-			(justify left bottom)
+			(justify right bottom)
 		)
 	)
-	(label "PC7"
-		(at 162.56 151.13 180)
+	(label "PE9"
+		(at 95.25 92.71 0)
 		(effects
 			(font
 				(size 1.27 1.27)
 			)
-			(justify right bottom)
+			(justify left bottom)
 		)
 	)
-	(label "CAN2.RX"
-		(at 162.56 102.87 180)
+	(label "PC7"
+		(at 162.56 151.13 180)
 		(effects
 			(font
@@
 		(effects
 			(font
+				(size 1.27 1.27)
+			)
+			(justify right bottom)
+		)
+	)
+	(label "CAN2.TX"
+		(at 162.56 123.19 180)
+		(effects
+			(font

Commit message: [#4] Remove unnecesary net labels on MCU
Connections:
- net PA0: no longer names the net of U400.22 (PA0)
- net PA1: no longer names the net of U400.23 (PA1)
- net PA10: no longer names the net of U400.69 (PA10)
- net PA15: no longer names the net of U400.77 (PA15)
- net PA2: no longer names the net of U400.24 (PA2)
- net PA3: no longer names the net of U400.25 (PA3)
- net PA4: no longer names the net of U400.28 (PA4)
- net PA5: no longer names the net of U400.29 (PA5)
- net PA6: no longer names the net of U400.30 (PA6)
- net PA7: no longer names the net of U400.31 (PA7)
- net PA8: no longer names the net of U400.67 (PA8)
- net PA9: no longer names the net of U400.68 (PA9)
- net PB0: no longer names the net of U400.34 (PB0)
- net PB1: no longer names the net of U400.35 (PB1)
- net PB11: no longer names the net of U400.47 (PB11)
- net PB14: no longer names the net of U400.53 (PB14)
- net PB15: no longer names the net of U400.54 (PB15)
- net PB3: no longer names the net of U400.89 (PB3)
- net PB4: no longer names the net of U400.90 (PB4)
- net PB5: no longer names the net of U400.91 (PB5)
- net PB6: no longer names the net of U400.92 (PB6)
- net PC0: no longer names the net of U400.15 (PC0)
- net PC1: no longer names the net of U400.16 (PC1)
- net PC10: no longer names the net of U400.78 (PC10)
- net PC11: no longer names the net of U400.79 (PC11)
- net PC12: no longer names the net of U400.80 (PC12)
- net PC13: no longer names the net of U400.7 (PC13)
- net PC2: no longer names the net of U400.17 (PC2_C)
- net PC3: no longer names the net of U400.18 (PC3_C)
- net PC4: no longer names the net of U400.32 (PC4)
- net PC5: no longer names the net of U400.33 (PC5)
- net PC6: no longer names the net of U400.63 (PC6)
- net PC7: no longer names the net of U400.64 (PC7)
- net PC8: no longer names the net of U400.65 (PC8)
- net PC9: no longer names the net of U400.66 (PC9)
- net PD10: no longer names the net of U400.57 (PD10)
- net PD14: no longer names the net of U400.61 (PD14)
- net PD15: no longer names the net of U400.62 (PD15)
- net PD2: no longer names the net of U400.83 (PD2)
- net PD3: no longer names the net of U400.84 (PD3)
- net PD4: no longer names the net of U400.85 (PD4)
- net PD5: no longer names the net of U400.86 (PD5)
- net PD6: no longer names the net of U400.87 (PD6)
- net PD7: no longer names the net of U400.88 (PD7)
- net PD8: no longer names the net of U400.55 (PD8)
- net PD9: no longer names the net of U400.56 (PD9)
- net PE0: no longer names the net of U400.97 (PE0)
- net PE1: no longer names the net of U400.98 (PE1)
- net PE10: no longer names the net of U400.40 (PE10)
- net PE11: no longer names the net of U400.41 (PE11)
- net PE12: no longer names the net of U400.42 (PE12)
- net PE13: no longer names the net of U400.43 (PE13)
- net PE14: no longer names the net of U400.44 (PE14)
- net PE15: no longer names the net of U400.45 (PE15)
- net PE7: no longer names the net of U400.37 (PE7)
- net PE8: no longer names the net of U400.38 (PE8)
- net PE9: no longer names the net of U400.39 (PE9)
- net VREF+: no longer names the net of U400.20 (VREF+)
- no-connect marks 60 -> 58
Other:
- moved on the sheet: C413, C414

Commit message: [#4] Improve schematic aesthetics, color nets
Connections:
- net +VDDA: now reaches C406.1, C407.1, FB400.1, U400.21 (VDDA)
Other:
- note added: "POWER INDICATOR AND USER LEDs"
- note removed: "POWER INDICATOR LEDs"
- moved on the sheet: C400, C401, C402, C403, C404, C405, C406, C407, C408, C409, FB400, LED300A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
