File: mcu.kicad_sch (KiCad schematic)
At the start: 36 parts, among them SW400 TL2243, U400 STM32H750VBTx, X300 Q13FC1350000400, X400 X322512MSB4SI

Commit message: Change MCU and update library
Changed MCU from H7 to H5 series due to programming issues with external
loader. Also updated JLCPCB components (not all tho there are still
arround 18 components to fix)
Parts:
- removed C403, C407, C409: 100nF, PCM_JLCPCB:C_0402, symbol PCM_JLCPCB-Capacitors:0402,100nF,(2)
- removed C406, C408: 10uF, PCM_JLCPCB:C_0402, symbol PCM_JLCPCB-Capacitors:0402,10uF
- removed C411, C412: 22pF, PCM_JLCPCB:C_0402, symbol PCM_JLCPCB-Capacitors:0402,22pF
- removed C413, C414: 2.2uF, PCM_JLCPCB:C_0402, symbol PCM_JLCPCB-Capacitors:0402,2.2uF
- removed FB400: ~, PCM_JLCPCB:FB_0603, symbol PCM_JLCPCB-Inductors:Ferrite,0603
- removed R407: 1.2kΩ, PCM_JLCPCB:R_0402, symbol PCM_JLCPCB-Resistors:0402,1.2kΩ
- removed R408: 470Ω, PCM_JLCPCB:R_0402, symbol PCM_JLCPCB-Resistors:0402,470Ω
- removed R409: 120Ω, PCM_JLCPCB:R_0402, symbol PCM_JLCPCB-Resistors:0402,120Ω
- removed U400: STM32H750VBTx, Package_QFP:LQFP-100_14x14mm_P0.5mm, symbol MCU_ST_STM32H7:STM32H750VBTx
- removed X400: X322512MSB4SI, PCM_JLCPCB:CRYSTAL-SMD_4P-L3.2-W2.5-BL, symbol PCM_JLCPCB-Crystals:Crystal, 12MHz, 20pF
- added C403, C423, C425, C430: 10uF, PCM_JLCPCB:C_0402, symbol PCM_JLCPCB-Capacitors:0402,10uF
- added C420, C421, C422, C424, C426, C432: 100nF, PCM_JLCPCB:C_0402, symbol PCM_JLCPCB-Capacitors:0402,100nF,(2)
- added C427, C434: 2.2uF, PCM_JLCPCB:C_0402, symbol PCM_JLCPCB-Capacitors:0402,2.2uF
- added C431: 15pF, PCM_JLCPCB:C_0402, symbol PCM_JLCPCB-Capacitors:0402,15pF
- added FB401: ~, PCM_JLCPCB:FB_0603, symbol PCM_JLCPCB-Inductors:Ferrite,0603
- added JP302, JP303: SolderJumper_2_Bridged, Jumper:SolderJumper-2_P1.3mm_Open_TrianglePad1.0x1.5mm, symbol Jumper:SolderJumper_2_Bridged
- added R407, R408: 220Ω, PCM_JLCPCB:R_0402, symbol PCM_JLCPCB-Resistors:0402,220Ω
- added R409: 100Ω, PCM_JLCPCB:R_0402, symbol PCM_JLCPCB-Resistors:0402,100Ω
- added U403: STM32H562VGTx, Package_QFP:LQFP-100_14x14mm_P0.5mm, symbol MCU_ST_STM32H5:STM32H562VGTx
- added Y400: ASE-xxxMHz, Oscillator:Oscillator_SMD_Abracon_ASE-4Pin_3.2x2.5mm, symbol Oscillator:ASE-xxxMHz
- C313, C314: Stock 582948 -> 408081
- C400: Price 0.007USD -> 0.008USD; Stock 9197991 -> 1226257
- C401, C402, C404, C405: Stock 5358037 -> 5436546
- C410: Stock 556737 -> 1633861
- C415, C416: Stock 3851753 -> 5436546
- R400: Stock 236021 -> 191144
- R401: Stock 8332962 -> 7947916
- R402, R403, R405: Stock 14017682 -> 13746052
- R404, R406: Stock 1570847 -> 3389382
- X300: Equivalent Series Resistance(Esr) (none) -> 70kΩ; Minimum Qty 1 -> 5; Normal Temperature Frequency Tolerance (none) -> ±20ppm; Price 0.174USD -> 0.188USD; Stock 185543 -> 407326; Type (none) -> Surface Mount Crystal
- renumbered SW400 to BTN400
Connections:
- net +3V3: now also C403.1, C420.1, C421.1, C422.1, C423.1, C424.1, C425.1, C426.1, C430.1, C432.1, FB401.1, FB401.2, JP302.1 (A), R409.1, U403.100 (VDD), U403.11 (VDD), U403.22 (VDDA), U403.28 (VDD), U403.50 (VDD), U403.6 (VBAT), U403.73 (VDDUSB), U403.75 (VDD), Y400.1 (EN), Y400.4 (Vdd)
- net BOOT0: now also U403.94 (BOOT0)
- net BOOT_EN: now also U403.93 (PB7)
- net CAN1.RX: now also U403.81 (PD0)
- net CAN1.TX: now also U403.82 (PD1)
- net CAN2.RX: now also U403.51 (PB12)
- net CAN2.TX: now also U403.52 (PB13)
- net GND: now also C403.2, C420.2, C421.2, C422.2, C423.2, C424.2, C425.2, C426.2, C427.2, C430.2, C431.2, C432.2, C434.2, JP303.1 (A), U403.10 (VSS), U403.19 (VSSA), U403.27 (VSS), U403.49 (VSS), U403.74 (VSS), U403.99 (VSS), Y400.2 (GND)
- net I2C1.SCL: now also U403.95 (PB8)
- net I2C1.SDA: now also U403.96 (PB9)
- net OSC32_IN: now also U403.8 (PC14)
- net OSC32_OUT: now also U403.9 (PC15)
- net OSC_IN: now also C431.1, U403.12 (PH0), Y400.3 (OUT)
- net QSPI1.CS: now also U403.47 (PB10)
- net QSPI1.IO0: now also U403.58 (PD11)
- net QSPI1.IO1: now also U403.59 (PD12)
- net QSPI1.IO2: now also U403.1 (PE2)
- net QSPI1.IO3: now also U403.60 (PD13)
- net QSPI1.SCLK: now also U403.37 (PB2)
- net STATUS_LED: now also R408.1, U403.4 (PE5)
- net SWD.SWCLK: now also U403.76 (PA14(JTCK)
- net SWD.SWDIO: now also U403.72 (PA13(JTMS)
- net SWD.~{RST}: now also U403.14 (NRST)
- net USB_MCU.D+: now also U403.71 (PA12)
- net USB_MCU.D-: now also U403.70 (PA11)
- net USER_LED_1: now also U403.2 (PE3)
- net USER_LED_2: now also R407.1, U403.3 (PE4)
- net USR_BUTTON: now also U403.5 (PE6)
- net VCAP_1: now also C427.1, U403.48 (VCAP)
- net VCAP_2: now also C434.1, U403.98 (VCAP)
- net at LED300.3: now also R407.2
- net at LED301.3: now also R409.2
- net at LED301.1: now also R408.2
- new net VREF+: JP302.2 (B), U403.21 (VREF+)
- new net VREF-: JP303.2 (B), U403.20 (VREF-)
- no-connect marks 60 -> 58
Other:
- note added: "AVDD"
- note added: "BULK"
- note added: "CAN"
- note added: "Design choice due: es0565, sec 2.2.3"
- note added: "NOTE: PLACE CZAPCZATOR AT EVERY PIN"
- note removed: "C = (CL - 4pF) * 2"
- title: ModuCard base module -> ModuCard BM STM32H562VGT6
- moved on the sheet: C313, C314, C410, LED300A, LED300B, LED301A, LED301B, R400, R401, R402, X300

Commit message: [1] Change MCU schematic ERC pass
Connections:
- net +3V3: no longer C423.1, C424.1, FB401.1, U403.22 (VDDA)
- new net VDDA: C423.1, C424.1, FB401.1, U403.22 (VDDA)
Other:
- note added: "NOTE: PLACE CAPACTITOR AT PWR PIN"
- note removed: "NOTE: PLACE CZAPCZATOR AT EVERY PIN"

Commit message: [3] Change layout
Parts:
- removed C430: 10uF, PCM_JLCPCB:C_0402, symbol PCM_JLCPCB-Capacitors:0402,10uF
- removed C431: 15pF, PCM_JLCPCB:C_0402, symbol PCM_JLCPCB-Capacitors:0402,15pF
- removed JP302, JP303: SolderJumper_2_Bridged, Jumper:SolderJumper-2_P1.3mm_Open_TrianglePad1.0x1.5mm, symbol Jumper:SolderJumper_2_Bridged
- added C406: 100nF, PCM_JLCPCB:C_0402, symbol PCM_JLCPCB-Capacitors:0402,100nF,(2)
Connections:
- net VREF+ is gone; now on net +3V3: U403.21 (VREF+)
- net VREF- is gone; now on net GND: U403.20 (VREF-)
- net +3V3: now also C406.1
- net GND: now also C406.2

Commit message: [#5] Add Y400 MPN
Parts:
- Y400: LCSC (none) -> C725989; MPN (none) -> OT322512MJBA4SL

Commit message: [REV2] board finshed, schematics and leyout
Parts:
- added R413, R414: 1.2kΩ, PCM_JLCPCB:R_0402, symbol PCM_JLCPCB-Resistors:0402,1.2kΩ
Connections:
- net +3V3: now also R413.1, R414.1
- net I2C1.SCL: now also R414.2
- net I2C1.SDA: now also R413.2
- net GPS_UART.RX: now reaches U403.23 (PA0)
- net GPS_UART.TX: now reaches U403.24 (PA1)
- net IMU_EXT_NRESET: now reaches U403.39 (PE8)
- net IMU_FSYNC: now reaches U403.42 (PE11)
- net IMU_INT: now reaches U403.43 (PE12)
- net GPS_SPI.CS: now reaches U403.77 (PA15(JTDI))
- net GPS_SPI.CLK: now reaches U403.78 (PC10)
- net GPS_SPI.MISO: now reaches U403.79 (PC11)
- net GPS_SPI.MOSI: now reaches U403.80 (PC12)
- net GPS_NRESET: now reaches U403.83 (PD2)
- net GPS_MODE_SELECT: now reaches U403.84 (PD3)
- net GPS_RTK_STAT: now reaches U403.85 (PD4)
- net GPS_GEOFENCE_STAT: now reaches U403.86 (PD5)
- net GPS_EXINTERUPT: now reaches U403.87 (PD6)
- no-connect marks 58 -> 42
Other:
- note added: "GPS"
- note added: "IMU"
- title: ModuCard BM STM32H562VGT6 -> ModuCard nav module
- moved on the sheet: C313, C314, C423, C424, C425, C426, C427, C432, C434, FB401, LED300A, LED300B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
Changed lines of the file:
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@@
 	(generator "eeschema")
 	(generator_version "9.0")
-	(paper "A4")
+	(paper "A3")
 	(title_block
-		(title "ModuCard BM STM32H562VGT6")
-		(date "2025-04-18")
+		(title "ModuCard nav module")
+		(date "2025-04-20")
 		(rev "1.1.0")
 		(company "KoNaR")
 		(comment 1 "Base project authors: Dominik Pluta, Artem Horiunov")
-		(comment 2 "Project author: <author>")
+		(comment 2 "Project author: Patryk Dudziński")
 	)

Commit message: [mcu] changed mcu from 562VGT6  to 563VGT6
Parts:
- removed U403: STM32H562VGTx, Package_QFP:LQFP-100_14x14mm_P0.5mm, symbol MCU_ST_STM32H5:STM32H562VGTx
- added U403: STM32H563VGTx, Package_QFP:LQFP-100_14x14mm_P0.5mm, symbol MCU_ST_STM32H5:STM32H563VGTx
Connections:
- net +3V3: now also U403.100 (VDD), U403.11 (VDD), U403.21 (VREF+), U403.28 (VDD), U403.50 (VDD), U403.6 (VBAT), U403.73 (VDDUSB), U403.75 (VDD)
- net BOOT0: now also U403.94 (BOOT0)
- net BOOT_EN: now also U403.93 (PB7)
- net CAN1.RX: now also U403.81 (PD0)
- net CAN1.TX: now also U403.82 (PD1)
- net CAN2.RX: now also U403.51 (PB12)
- net CAN2.TX: now also U403.52 (PB13)
- net GND: now also U403.10 (VSS), U403.19 (VSSA), U403.20 (VREF-), U403.27 (VSS), U403.49 (VSS), U403.74 (VSS), U403.99 (VSS)
- net GPS_EXINTERUPT: now also U403.87 (PD6)
- net GPS_GEOFENCE_STAT: now also U403.86 (PD5)
- net GPS_MODE_SELECT: now also U403.84 (PD3)
- net GPS_NRESET: now also U403.83 (PD2)
- net GPS_RTK_STAT: now also U403.85 (PD4)
- net GPS_SPI.CLK: now also U403.78 (PC10)
- net GPS_SPI.CS: now also U403.77 (PA15(JTDI))
- net GPS_SPI.MISO: now also U403.79 (PC11)
- net GPS_SPI.MOSI: now also U403.80 (PC12)
- net GPS_UART.RX: now also U403.23 (PA0)
- net GPS_UART.TX: now also U403.24 (PA1)
- net I2C1.SCL: now also U403.95 (PB8)
- net I2C1.SDA: now also U403.96 (PB9)
- net IMU_EXT_NRESET: now also U403.39 (PE8)
- net IMU_FSYNC: now also U403.42 (PE11)
- net IMU_INT: now also U403.43 (PE12)
- net OSC32_IN: now also U403.8 (PC14)
- net OSC32_OUT: now also U403.9 (PC15)
- net OSC_IN: now also U403.12 (PH0)
- net QSPI1.CS: now also U403.47 (PB10)
- net QSPI1.IO0: now also U403.58 (PD11)
- net QSPI1.IO1: now also U403.59 (PD12)
- net QSPI1.IO2: now also U403.1 (PE2)
- net QSPI1.IO3: now also U403.60 (PD13)
- net QSPI1.SCLK: now also U403.37 (PB2)
- net STATUS_LED: now also U403.4 (PE5)
- net SWD.SWCLK: now also U403.76 (PA14(JTCK)
- net SWD.SWDIO: now also U403.72 (PA13(JTMS)
- net SWD.~{RST}: now also U403.14 (NRST)
- net USB_MCU.D+: now also U403.71 (PA12)
- net USB_MCU.D-: now also U403.70 (PA11)
- net USER_LED_1: now also U403.2 (PE3)
- net USER_LED_2: now also U403.3 (PE4)
- net USR_BUTTON: now also U403.5 (PE6)
- net VCAP_1: now also U403.48 (VCAP)
- net VCAP_2: now also U403.98 (VCAP)
- net VDDA: now also U403.22 (VDDA)

Commit message: changed shity resisrto to smaller one on LEDs  fixed level shifting
Parts:
- removed R400: 1.2kΩ, PCM_JLCPCB:R_0402, symbol PCM_JLCPCB-Resistors:0402,1.2kΩ
- removed R409: 100Ω, PCM_JLCPCB:R_0402, symbol PCM_JLCPCB-Resistors:0402,100Ω
- added R423, R428: 220Ω, PCM_JLCPCB:R_0402, symbol PCM_JLCPCB-Resistors:0402,220Ω
Connections:
- net +3V3: now also R428.1
- net USER_LED_1: now also R423.1
- net at LED301.3: now also R428.2
- net at LED300.1: now also R423.2
