File: power.kicad_sch (KiCad schematic)
At the start: 32 parts, among them Q301 AO3400A, U301 TPS56320x, U302 AMS1117-3.3

Commit message: [3] Change components to parts from LCSC on power sheet
Parts:
- removed C301: 100nF, Capacitor_SMD:C_0402_1005Metric, symbol Device:C_Small
- removed C302, C303, C304, C305, C306, C307: 22uF, symbol Device:C_Small
- removed D301: 5.6 V, symbol Device:D_Zener
- removed D302, D303, D304, D305: Green, symbol Device:LED
- removed F301: 2A FF, symbol Device:Fuse_Small
- removed Q301: AO3400A, Package_TO_SOT_SMD:SOT-23, symbol Transistor_FET:AO3400A
- removed R302: 1k, symbol Device:R_Small
- removed R303, R304: 10k, symbol Device:R_Small
- removed R305, R306: 1K2, symbol Device:R_Small
- removed R307: 480R, symbol Device:R_Small
- removed R308: 120R, symbol Device:R_Small
- added C421, C422, C423, C424, C426, C427: 10uF, PCM_JLCPCB:C_0603, symbol PCM_JLCPCB-Capacitors:0603,10uF,(2)
- added C425: 100nF, PCM_JLCPCB:C_0402, symbol PCM_JLCPCB-Capacitors:0402,100nF,(2)
- added D401: BZT52C5V6S, PCM_JLCPCB:D_SOD-323, symbol PCM_JLCPCB-Diodes:Zener,BZT52C5V6S
- added D402, D403, D404, D405: Green, PCM_JLCPCB:D_0603, symbol PCM_JLCPCB-Diodes:LED,0603,Green
- added F401: 1.5A, PCM_JLCPCB:F_0603, symbol PCM_JLCPCB-Variable-Resistors:Fuse,1.5A
- added Q401: AO3400A, PCM_JLCPCB:Q_SOT-23, symbol PCM_JLCPCB-Transistors:NMOS,AO3400A
- added R417, R418: 10kΩ, PCM_JLCPCB:R_0402, symbol PCM_JLCPCB-Resistors:0402,10kΩ
- added R419: 1kΩ, PCM_JLCPCB:R_0402, symbol PCM_JLCPCB-Resistors:0402,1kΩ
- added R420: 120Ω, PCM_JLCPCB:R_0402, symbol PCM_JLCPCB-Resistors:0402,120Ω
- added R421: 470Ω, PCM_JLCPCB:R_0402, symbol PCM_JLCPCB-Resistors:0402,470Ω
- added R422, R423: 1.2kΩ, PCM_JLCPCB:R_0402, symbol PCM_JLCPCB-Resistors:0402,1.2kΩ
- U301: value TPS56320x -> TPS563201DDCR
Connections:
- net +12V: now also D405.2, F401.1, R419.1
- net +12V_FUSED: now also C421.1, C427.1, D404.2, F401.2
- net +3V3: now also D402.2
- net +5V: now also C422.1, D403.2, Q401.3 (D)
- net 3V3_OUT: now also C426.1
- net 5V_UNPROTEC: now also C423.1, C424.1, D401.1
- net FB: now also R417.1
- net GND: now also C421.2, C422.2, C423.2, C424.2, C426.2, C427.2, D401.2, R417.2, R418.2, R420.2, R421.2, R422.2, R423.2
- net VBST: now also C425.1
- net at L301.1, U301.2 (SW): now also C425.2
- net at JP301.2 (B): now also Q401.2 (S)
- new net: D405.1, R423.1
- new net: Q401.1 (G), R418.1, R419.2
- new net: D403.1, R421.1
- new net: D404.1, R422.1
- new net: D402.1, R420.1
Other:
- moved on the sheet: TP301, TP304, U301

Commit message: [3] Fix schematic sheet descriptions
Other:
- title: ModuCard base module power -> ModuCard base module
Changed lines of the file:
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@@
 	(paper "A4")
 	(title_block
-		(title "ModuCard base module power")
+		(title "ModuCard base module")
 		(date "2024-12-23")
 		(rev "1.0.0")

Commit message: [3] Add second converter
Parts:
- removed C422, C426: 10uF, PCM_JLCPCB:C_0603, symbol PCM_JLCPCB-Capacitors:0603,10uF,(2)
- removed JP302: Test LDO Vout, symbol Jumper:SolderJumper_2_Bridged
- removed TP305: LDO vout, symbol Connector:TestPoint
- removed U302: AMS1117-3.3, Package_TO_SOT_SMD:SOT-223-3_TabPin2, symbol Regulator_Linear:AMS1117-3.3
- added C1, C2: 10uF, PCM_JLCPCB:C_0603, symbol PCM_JLCPCB-Capacitors:0603,10uF,(2)
- added C3: 0.1uF, PCM_JLCPCB:C_0603, symbol PCM_JLCPCB-Capacitors:0603,10uF,(2)
- added C4: 100nF, PCM_JLCPCB:C_0402, symbol PCM_JLCPCB-Capacitors:0402,100nF,(2)
- added C5, C6: 22uF, PCM_JLCPCB:C_0603, symbol PCM_JLCPCB-Capacitors:0603,10uF,(2)
- added D1: BZT52C5V6S, PCM_JLCPCB:D_SOD-323, symbol PCM_JLCPCB-Diodes:Zener,BZT52C5V6S
- added F1: 1.5A, PCM_JLCPCB:F_0603, symbol PCM_JLCPCB-Variable-Resistors:Fuse,1.5A
- added JP1: Test Buck Vout, symbol Jumper:SolderJumper_2_Bridged
- added L1: 2.2uH, symbol Device:L
- added R1: 33k2, symbol Device:R_Small
- added R2: 10kΩ, PCM_JLCPCB:R_0402, symbol PCM_JLCPCB-Resistors:0402,10kΩ
- added TP1: TestPoint, symbol Connector:TestPoint
- added TP2: Buck Feedback, symbol Connector:TestPoint
- added U1: TPS563201DDCR, Package_TO_SOT_SMD:SOT-23-6, symbol Regulator_Switching:TPS563200
Connections:
- net +12V: now also F1.1
- net +3V3: now also JP1.2 (B)
- net FB: now also R1.2, R2.1, TP2.1, U1.4 (VFB)
- net GND: now also C1.2, C2.2, C3.2, C5.2, C6.2, D1.2, R2.2, U1.1 (GND)
- net VBST: now also C4.1, U1.6 (VBST)
- new net: C1.1, C2.1, C3.1, F1.2, TP1.1, U1.3 (VIN), U1.5 (EN)
- new net: C4.2, L1.1, U1.2 (SW)
- new net 3V3_UNPROTEC: C5.1, C6.1, D1.1, JP1.1 (A), L1.2, R1.1
Other:
- note added: "3V3 DC/DC CONVERTER"
- note added: "V_{OUT} = 0.765*(1+33k2/10k) = 3.3V"
- note removed: "3V3 LINEAR REGULATOR"
- moved on the sheet: D402, D403, D404, D405, R420, R421, R422, R423

Commit message: [3] Fix power supply schematic, add test points
Parts:
- removed C3: 0.1uF, PCM_JLCPCB:C_0603, symbol PCM_JLCPCB-Capacitors:0603,10uF,(2)
- removed C5, C6: 22uF, PCM_JLCPCB:C_0603, symbol PCM_JLCPCB-Capacitors:0603,10uF,(2)
- removed D1: BZT52C5V6S, PCM_JLCPCB:D_SOD-323, symbol PCM_JLCPCB-Diodes:Zener,BZT52C5V6S
- removed F1: 1.5A, PCM_JLCPCB:F_0603, symbol PCM_JLCPCB-Variable-Resistors:Fuse,1.5A
- removed Q401: AO3400A, PCM_JLCPCB:Q_SOT-23, symbol PCM_JLCPCB-Transistors:NMOS,AO3400A
- removed R418: 10kΩ, PCM_JLCPCB:R_0402, symbol PCM_JLCPCB-Resistors:0402,10kΩ
- removed R419: 1kΩ, PCM_JLCPCB:R_0402, symbol PCM_JLCPCB-Resistors:0402,1kΩ
- added C306, C307: 22uF, PCM_JLCPCB:C_0603, symbol PCM_JLCPCB-Capacitors:0603,22uF
- added C310: 100nF, PCM_JLCPCB:C_0402, symbol PCM_JLCPCB-Capacitors:0402,100nF,(2)
- added TP305, TP306: TestPoint, symbol Connector:TestPoint
- renumbered C425 to C300, C423 to C301, C424 to C302, C427 to C303, C421 to C304, C4 to C305, C1 to C308, C2 to C309, D401 to D300, D405 to D301, D404 to D302, D403 to D303, D402 to D304, F401 to F300, JP301 to JP300, JP1 to JP301, L301 to L300, L1 to L301, R301 to R300, R417 to R301, R1 to R302, R423 to R303, R422 to R304, R421 to R305, R420 to R306, R2 to R307, TP301 to TP300, TP302 to TP301, TP303 to TP302, TP304 to TP303, TP1 to TP304, TP2 to TP307, U301 to U300, U1 to U301
Connections:
- net +12V_FUSED: now also C308.1, C309.1, TP304.1, U301.3 (VIN), U301.5 (EN), C310.2
- net +3V3: now also TP306.1
- net +5V: now also JP300.2 (B)
- net 3V3_UNPROTEC: now also C306.1, C307.1, TP305.1
- net GND: now also C306.2, C307.2, C310.1
Other:
- moved on the sheet: C305, C308, C309, D301, D302, D303, D304, JP301, L301, R302, R303, R304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

Commit message: [3] Choose 3u3 inductor and solder jumpers footprints on power schematic
[3] Choose 3u3 inductor and testpoint footprints
Parts:
- removed L301: 2.2uH, symbol Device:L
- added L401: 3.3uH, Inductor_SMD:L_Changjiang_FXL0420, symbol Device:L
- JP300, JP301: footprint (none) -> Jumper:SolderJumper-2_P1.3mm_Open_TrianglePad1.0x1.5mm
- L300: footprint (none) -> Inductor_SMD:L_Changjiang_FXL0420
Connections:
- net 3V3_UNPROTEC: now also L401.2
- net at C305.2, U301.2 (SW): now also L401.1
Changed lines of the file:
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@@
 	(label "3V3_UNPROTEC"
 		(at 135.89 95.25 0)
-		(fields_autoplaced yes)
 		(effects
 			(font
@@
 	(label "5V_UNPROTEC"
 		(at 151.13 41.91 0)
-		(fields_autoplaced yes)
 		(effects
 			(font
@@
 	(label "FB"
 		(at 105.41 100.33 180)
-		(fields_autoplaced yes)
 		(effects
 			(font
@@
 	(label "VBST"
 		(at 101.6 97.79 0)
-		(fields_autoplaced yes)
 		(effects
 			(font
@@
 	(label "FB"
 		(at 120.65 46.99 180)
-		(fields_autoplaced yes)
 		(effects
 			(font
@@
 	(label "VBST"
 		(at 116.84 44.45 0)
-		(fields_autoplaced yes)
 		(effects
 			(font
@@
 	)
 	(symbol
+		(lib_id "Device:L")
+		(at 128.27 95.25 90)
+		(unit 1)
+		(exclude_from_sim no)
+		(in_bom yes)
+		(on_board yes)
+		(dnp no)
+		(fields_autoplaced yes)
+		(property "Reference" "L401"
+			(at 128.27 90.17 90)
+			(effects
+				(font
+					(size 1.27 1.27)
+				)
+			)
+		)
+		(property "Value" "3.3uH"
+			(at 128.27 92.71 90)
+			(effects
+				(font
+					(size 1.27 1.27)
+				)
+			)
+		)
+		(property "Footprint" "Inductor_SMD:L_Changjiang_FXL0420"
+			(at 128.27 95.25 0)
+			(effects
+				(font
+					(size 1.27 1.27)
+				)
+				(hide yes)
+			)
+		)
+		(property "Datasheet" "~"
+			(at 128.27 95.25 0)
+			(effects
+				(font
+					(size 1.27 1.27)
+				)
+				(hide yes)
+			)
+		)
+		(property "Description" "DMBJ CXP0420-3R3M-AG(3.3UH)"
+			(at 128.27 95.25 0)
+			(effects
+				(font
+					(size 1.27 1.27)
+				)
+				(hide yes)
+			)
+		)
+		(pin "1"
+		)
+		(pin "2"
+		)
+		(instances
+			(project "base-module"
+				(path "/090a8e41-87a8-4fb1-998b-60a2c0dc4cee/3f372eb1-53a4-4b00-8846-6751dd401eeb"
+					(reference "L401")
+					(unit 1)
+				)
+			)
+		)
+	)
+	(symbol
 		(lib_id "power:GND")
 		(at 242.57 115.57 0)
@@
 			)
 		)
-		(property "Footprint" ""
+		(property "Footprint" "Jumper:SolderJumper-2_P1.3mm_Open_TrianglePad1.0x1.5mm"
 			(at 163.83 95.25 0)
 			(effects
@@
 			)
 		)
-		(property "Footprint" ""
+		(property "Footprint" "Jumper:SolderJumper-2_P1.3mm_Open_TrianglePad1.0x1.5mm"
 			(at 191.77 41.91 0)
 			(effects
@@
 	)
 	(symbol
-		(lib_id "Device:L")
-		(at 128.27 95.25 90)
-		(unit 1)
-		(exclude_from_sim no)
-		(in_bom yes)
-		(on_board yes)
-		(dnp no)
-		(fields_autoplaced yes)
-		(property "Reference" "L301"
-			(at 128.27 90.17 90)
-			(effects
-				(font
-					(size 1.27 1.27)
-				)
-			)
-		)
-		(property "Value" "2.2uH"
-			(at 128.27 92.71 90)
-			(effects
-				(font
-					(size 1.27 1.27)
-				)
-			)
-		)
-		(property "Footprint" ""
-			(at 128.27 95.25 0)
-			(effects
-				(font
-					(size 1.27 1.27)
-				)
-				(hide yes)
-			)
-		)
-		(property "Datasheet" "~"
-			(at 128.27 95.25 0)
-			(effects
-				(font
-					(size 1.27 1.27)
-				)
-				(hide yes)
-			)
-		)
-		(property "Description" "Inductor"
-			(at 128.27 95.25 0)
-			(effects
-				(font
-					(size 1.27 1.27)
-				)
-				(hide yes)
-			)
-		)
-		(pin "1"
-		)
-		(pin "2"
-		)
-		(instances
-			(project "base-module"
-				(path "/090a8e41-87a8-4fb1-998b-60a2c0dc4cee/3f372eb1-53a4-4b00-8846-6751dd401eeb"
-					(reference "L301")
-					(unit 1)
-				)
-			)
-		)
-	)
-	(symbol
 		(lib_id "Device:R_Small")
 		(at 149.86 45.72 0)
@@
 			)
 		)
-		(property "Footprint" ""
+		(property "Footprint" "Inductor_SMD:L_Changjiang_FXL0420"
 			(at 143.51 41.91 0)
 			(effects
@@
 			)
 		)
-		(property "Description" "Inductor"
+		(property "Description" "DMBJ CXP0420-3R3M-AG(3.3UH)"
 			(at 143.51 41.91 0)
 			(effects

Commit message: [3] Add resistor and test points footprints
Parts:
- R300, R302: footprint (none) -> PCM_JLCPCB:R_0402
- TP300, TP301, TP302, TP304, TP305, TP306: footprint (none) -> TestPoint:TestPoint_Pad_D1.0mm
Changed lines of the file:
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@@
 			)
 		)
-		(property "Footprint" ""
+		(property "Footprint" "TestPoint:TestPoint_Pad_D1.0mm"
 			(at 74.93 40.64 0)
 			(effects
@@
 			)
 		)
-		(property "Footprint" ""
+		(property "Footprint" "TestPoint:TestPoint_Pad_D1.0mm"
 			(at 209.55 40.64 0)
 			(effects
@@
 			)
 		)
-		(property "Footprint" ""
+		(property "Footprint" "PCM_JLCPCB:R_0402"
 			(at 149.86 45.72 0)
 			(effects
@@
 			)
 		)
-		(property "Footprint" ""
+		(property "Footprint" "TestPoint:TestPoint_Pad_D1.0mm"
 			(at 175.26 93.98 0)
 			(effects
@@
 			)
 		)
-		(property "Footprint" ""
+		(property "Footprint" "TestPoint:TestPoint_Pad_D1.0mm"
 			(at 74.93 93.98 0)
 			(effects
@@
 			)
 		)
-		(property "Footprint" ""
+		(property "Footprint" "TestPoint:TestPoint_Pad_D1.0mm"
 			(at 179.07 41.91 0)
 			(effects
@@
 			)
 		)
-		(property "Footprint" ""
+		(property "Footprint" "TestPoint:TestPoint_Pad_D1.0mm"
 			(at 162.56 93.98 0)
 			(effects
@@
 			)
 		)
-		(property "Footprint" ""
+		(property "Footprint" "PCM_JLCPCB:R_0402"
 			(at 134.62 99.06 0)
 			(effects
