File: power.kicad_sch (KiCad schematic)
At the start: 39 parts, among them U300 TPS563201DDCR, U301 TPS563201DDCR

Commit message: [#2] Replace USB switch and power indicator LEDs
Parts:
- removed D301, D302, D303, D304: Green, PCM_JLCPCB:D_0603, symbol PCM_JLCPCB-Diodes:LED,0603,Green
- added LED300, LED301: FixLed307, FixLed307:FixLed307, symbol FixLed307:FixLed307
Connections:
- net +12V: now also R303.1
- net +12V_FUSED: now also R304.1
- net +3V3: now also R306.1
- net +5V: now also R305.1
- net GND: now also LED300.2, LED300.4, LED301.2, LED301.4; no longer R303.2, R304.2, R305.2, R306.2
- new net: LED301.3, R306.2
- new net: LED300.3, R304.2
- new net: LED300.1, R303.2
- new net: LED301.1, R305.2
Other:
- moved on the sheet: R303, R304, R305, R306

Commit message: [#2] WIP: Layout DC-DC converters, MCU
Parts:
- added C305: 100nF, PCM_JLCPCB:C_0402, symbol PCM_JLCPCB-Capacitors:0402,100nF,(2)
- renumbered C305 to C306, C306 to C307, C307 to C308, C308 to C309, C309 to C310, C310 to C311, R303 to R302, R304 to R303, R305 to R304, R306 to R305, R302 to R306
Connections:
- net +12V_FUSED: now also C305.2
- net GND: now also C305.1
- net SW_3V3: now reaches C306.2, L301.1, U301.2 (SW)
- net SW_5V0: now reaches C300.2, L300.1, U300.2 (SW)
- net FB renamed FB_3V3
- net FB_3V3: no longer R300.2, R301.1, TP303.1, U300.4 (VFB)
- net VBST renamed VBST_3V3
- net VBST_3V3: no longer C300.1, U300.6 (VBST)
- new net FB_5V0: R300.2, R301.1, TP303.1, U300.4 (VFB)
- new net VBST_5V0: C300.1, U300.6 (VBST)
Other:
- moved on the sheet: C303, C304, C309, C310, C311, F300, TP300, TP304, U300, U301

Commit message: [#2] Connect MCU to ST-LINK, route DC-DC converters
Parts:
- removed TP303, TP307: Buck Feedback, TestPoint:TestPoint_Pad_D1.0mm, symbol Connector:TestPoint
- removed TP304: TestPoint, TestPoint:TestPoint_Pad_D1.0mm, symbol Connector:TestPoint

Commit message: [#2] Fix MCU model, draft QSPI connection
Parts:
- removed D300: BZT52C5V6S, PCM_JLCPCB:D_SOD-323, symbol PCM_JLCPCB-Diodes:Zener,BZT52C5V6S

Commit message: [#2] Route everything except for some test points, fix LED and button configuration
Parts:
- removed LED300, LED301: FixLed307, FixLed307:FixLed307, symbol FixLed307:FixLed307
- removed R302, R303: 1.2kΩ, PCM_JLCPCB:R_0402, symbol PCM_JLCPCB-Resistors:0402,1.2kΩ
- removed R304: 470Ω, PCM_JLCPCB:R_0402, symbol PCM_JLCPCB-Resistors:0402,470Ω
- removed R305: 120Ω, PCM_JLCPCB:R_0402, symbol PCM_JLCPCB-Resistors:0402,120Ω
Other:
- note removed: "POWER INDICATOR LEDs"
- note removed: "Target I_{LED} = 10mA"

Commit message: [#2] Finish layout
Parts:
- removed TP302, TP305: TestPoint, TestPoint:TestPoint_Pad_D1.0mm, symbol Connector:TestPoint
- added D400, D401, D402: Green, PCM_JLCPCB:D_0603, symbol PCM_JLCPCB-Diodes:LED,0603,Green
- added R410, R411, R412: 120Ω, PCM_JLCPCB:R_0402, symbol PCM_JLCPCB-Resistors:0402,120Ω
- renumbered TP306 to TP302
Connections:
- net +12V_FUSED: now also D400.2
- net +3V3: now also D402.2
- net +5V: now also D401.2
- net GND: now also R410.2, R411.2, R412.2
- new net: D400.1, R410.1
- new net: D401.1, R411.1
- new net: D402.1, R412.1

Commit message: [#4] Fix power indicator LEDs resistor values
Parts:
- removed R410, R411, R412: 120Ω, PCM_JLCPCB:R_0402, symbol PCM_JLCPCB-Resistors:0402,120Ω
- added R410: 2.2kΩ, PCM_JLCPCB:R_0402, symbol PCM_JLCPCB-Resistors:0402,2.2kΩ
- added R411: 470Ω, PCM_JLCPCB:R_0402, symbol PCM_JLCPCB-Resistors:0402,470Ω
- added R412: 220Ω, PCM_JLCPCB:R_0402, symbol PCM_JLCPCB-Resistors:0402,220Ω
Connections:
- net GND: now also R410.2, R411.2, R412.2
- net at D400.1: now also R410.1
- net at D401.1: now also R411.1
- net at D402.1: now also R412.1
Other:
- note added: "POWER INDICATOR LEDs"
- note added: "Target I_{LED} = 5mA"
- moved on the sheet: D400, D401, D402

Commit message: [#4] Improve schematic aesthetics, color nets
Connections:
- net 3V3_UNPROTEC renamed +3V3_UNPROTEC
- net 5V_UNPROTEC renamed +5V_UNPROTEC
Changed lines of the file:
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@@
 	(title_block
 		(title "ModuCard base module")
-		(date "2024-12-23")
+		(date "2025-02-18")
 		(rev "1.0.0")
 		(company "KoNaR")
@@
 	(text "Target I_{LED} = 5mA"
 		(exclude_from_sim no)
-		(at 260.858 106.172 0)
+		(at 202.946 143.256 0)
 		(effects
 			(font
@@
 		)
 	)
-	(label "3V3_UNPROTEC"
+	(label "+3V3_UNPROTEC"
 		(at 132.08 113.03 0)
 		(effects
@@
 		)
 	)
-	(label "5V_UNPROTEC"
+	(label "+5V_UNPROTEC"
 		(at 147.32 59.69 0)
 		(effects
