File: power.kicad_sch (KiCad schematic)
At the start: 32 parts, among them U300 TPS563201DDCR, U301 TPS563201DDCR

Commit message: [#12] Add GND testpoint
Parts:
- added TP400: TestPoint, TestPoint:TestPoint_Pad_D1.0mm, symbol Connector:TestPoint
Connections:
- net GND: now also TP400.1
Changed lines of the file:
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@@
 	(wire
 		(pts
+			(xy 33.02 80.01) (xy 33.02 77.47)
+		)
+		(stroke
+			(width 0)
+			(type default)
+		)
+	)
+	(wire
+		(pts
 			(xy 143.51 59.69) (xy 146.05 59.69)
 		)
@@
 	)
 	(symbol
+		(lib_id "Connector:TestPoint")
+		(at 33.02 77.47 0)
+		(unit 1)
+		(exclude_from_sim no)
+		(in_bom yes)
+		(on_board yes)
+		(dnp no)
+		(property "Reference" "TP400"
+			(at 33.02 72.39 0)
+			(effects
+				(font
+					(size 1.27 1.27)
+				)
+			)
+		)
+		(property "Value" "TestPoint"
+			(at 35.56 75.438 0)
+			(effects
+				(font
+					(size 1.27 1.27)
+				)
+				(justify left)
+				(hide yes)
+			)
+		)
+		(property "Footprint" "TestPoint:TestPoint_Pad_D1.0mm"
+			(at 38.1 77.47 0)
+			(effects
+				(font
+					(size 1.27 1.27)
+				)
+				(hide yes)
+			)
+		)
+		(property "Datasheet" "~"
+			(at 38.1 77.47 0)
+			(effects
+				(font
+					(size 1.27 1.27)
+				)
+				(hide yes)
+			)
+		)
+		(property "Description" "test point"
+			(at 33.02 77.47 0)
+			(effects
+				(font
+					(size 1.27 1.27)
+				)
+				(hide yes)
+			)
+		)
+		(pin "1"
+		)
+		(instances
+			(project "base-module"
+				(path "/090a8e41-87a8-4fb1-998b-60a2c0dc4cee/3f372eb1-53a4-4b00-8846-6751dd401eeb"
+					(reference "TP400")
+					(unit 1)
+				)
+			)
+		)
+	)
+	(symbol
 		(lib_id "PCM_JLCPCB-Resistors:0402,470Ω")
 		(at 228.6 127 0)
@@
 					(unit 1)
 				)
+			)
+		)
+	)
+	(symbol
+		(lib_id "power:GND")
+		(at 33.02 80.01 0)
+		(unit 1)
+		(exclude_from_sim no)
+		(in_bom yes)
+		(on_board yes)
+		(dnp no)
+		(property "Reference" "#PWR0415"
+			(at 33.02 86.36 0)
+			(effects
+				(font
+					(size 1.27 1.27)
+				)
+				(hide yes)
+			)
+		)
+		(property "Value" "GND"
+			(at 33.02 83.82 0)
+			(effects
+				(font
+					(size 1.27 1.27)
+				)
+			)
+		)
+		(property "Footprint" ""
+			(at 33.02 80.01 0)
+			(effects
+				(font
+					(size 1.27 1.27)
+				)
+				(hide yes)
+			)
+		)
+		(property "Datasheet" ""
+			(at 33.02 80.01 0)
+			(effects
+				(font
+					(size 1.27 1.27)
+				)
+				(hide yes)
+			)
+		)
+		(property "Description" "Power symbol creates a global label with name \"GND\" , ground"
+			(at 33.02 80.01 0)
+			(effects
+				(font
+					(size 1.27 1.27)
+				)
+				(hide yes)
+			)
+		)
+		(pin "1"
+		)
+		(instances
+			(project "base-module"
+				(path "/090a8e41-87a8-4fb1-998b-60a2c0dc4cee/3f372eb1-53a4-4b00-8846-6751dd401eeb"
+					(reference "#PWR0415")
+					(unit 1)
+				)

Commit message: Change MCU and update library
Changed MCU from H7 to H5 series due to programming issues with external
loader. Also updated JLCPCB components (not all tho there are still
arround 18 components to fix)
Parts:
- C300, C305, C306, C311: Stock 5427590 -> 5436546
- C301, C302, C303, C304, C309, C310: Price 0.017USD -> 0.020USD; Stock 4293394 -> 2203364
- C307, C308: Price 0.010USD -> 0.011USD; Stock 6715457 -> 4784939
- JP300, JP301: value Test Buck Vout -> SolderJumper_2_Bridged
- L300, L301: value 3.3uH -> L
- R300: value 54k9 -> R_Small
- R301, R307: Stock 7034931 -> 13746052
- R306: value 33k2 -> R_Small
- R410: Stock 750885 -> 2234263
- R411: Stock 703987 -> 911336
- R412: Stock 735848 -> 927669
- U300, U301: value TPS563201DDCR -> TPS563200
Other:
- title: ModuCard base module -> ModuCard BM STM32H562VGT6

Commit message: [1] Change MCU schematic ERC pass
Parts:
- removed D400, D401, D402: Green, PCM_JLCPCB:D_0603, symbol PCM_JLCPCB-Diodes:LED,0603,Green
- removed F300: 1.5A, PCM_JLCPCB:F_0603, symbol PCM_JLCPCB-Variable-Resistors:Fuse,1.5A
- added D400, D401, D402: Red, PCM_JLCPCB:D_0603, symbol PCM_JLCPCB-Diodes:LED,0603,Red
- added F300: Fuse, PCM_JLCPCB:R_0603, symbol Device:Fuse
Connections:
- net +12V: now also F300.1
- net +12V_FUSED: now also D400.2, F300.2
- net +3V3: now also D402.2
- net +5V: now also D401.2
- net at R411.1: now also D401.1
- net at R412.1: now also D402.1
- net at R410.1: now also D400.1

Commit message: [REV2] board finshed, schematics and leyout
Other:
- title: ModuCard BM STM32H562VGT6 -> ModuCard nav module
Changed lines of the file:
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@@
 	(paper "A4")
 	(title_block
-		(title "ModuCard BM STM32H562VGT6")
-		(date "2025-04-18")
+		(title "ModuCard nav module")
+		(date "2025-04-20")
 		(rev "1.1.0")
 		(company "KoNaR")
 		(comment 1 "Base project authors: Dominik Pluta, Artem Horiunov")
-		(comment 2 "Project author: <author>")
+		(comment 2 "Project author: Patryk Dudziński")
 	)
 	(rectangle
