File: USB-hub.kicad_sch (KiCad schematic)
At the start: 11 parts, among them U406 CH334R, Y403 12Mhz

Commit message: [3] Rename USB hub sheet
Changed lines of the file:
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@@
-		)
-	)
-	(bus
-		(pts
-			(xy 62.23 91.44) (xy 62.23 93.98)
-		)
-		(stroke
-			(width 0)
-			(type default)
 		)
 	)
@@
 		)
 		(stroke
-			(width 0)
-			(type default)
-		)
-	)
-	(bus
-		(pts
-			(xy 67.31 86.36) (xy 67.31 88.9)
-		)
-		(stroke

Commit message: [3] Fix usb bus issue
Connections:
- net USBOUT2.D+ renamed USB_MCU.+
- net USBOUT2.D- renamed USB_MCU.-
Changed lines of the file:
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@@
 		(comment 1 "Base project authors: Dominik Pluta, Artem Horiunov")
+	)
+	(bus_alias "USB"
+		(members "+" "-")
 	)
 	(junction
@@
 	)
 	(bus_entry
-		(at 69.85 88.9)
-		(size -2.54 -2.54)
-		(stroke
-			(width 0)
-			(type default)
-		)
-	)
-	(bus_entry
-		(at 69.85 86.36)
-		(size -2.54 -2.54)
+		(at 64.77 83.82)
+		(size 2.54 2.54)
 		(stroke
 			(width 0)
@@
 		)
 	)
+	(bus_entry
+		(at 64.77 86.36)
+		(size 2.54 2.54)
+		(stroke
+			(width 0)
+			(type default)
+		)
+	)
+	(bus
+		(pts
+			(xy 64.77 86.36) (xy 64.77 87.63)
+		)
+		(stroke
+			(width 0)
+			(type default)
+		)
+	)
 	(wire
 		(pts
@@
 	(wire
 		(pts
-			(xy 69.85 86.36) (xy 107.95 86.36)
-		)
-		(stroke
-			(width 0)
-			(type default)
-		)
-	)
-	(wire
-		(pts
 			(xy 251.46 81.28) (xy 149.86 81.28)
 		)
@@
 		)
 	)
-	(bus
-		(pts
-			(xy 67.31 80.01) (xy 67.31 83.82)
-		)
-		(stroke
-			(width 0)
-			(type default)
-		)
-	)
 	(wire
 		(pts
@@
 	(bus
 		(pts
-			(xy 46.99 80.01) (xy 67.31 80.01)
+			(xy 59.69 76.2) (xy 64.77 76.2)
 		)
 		(stroke
@@
 	(wire
 		(pts
+			(xy 67.31 86.36) (xy 107.95 86.36)
+		)
+		(stroke
+			(width 0)
+			(type default)
+		)
+	)
+	(wire
+		(pts
 			(xy 149.86 91.44) (xy 163.83 91.44)
 		)
@@
 	(wire
 		(pts
-			(xy 69.85 88.9) (xy 107.95 88.9)
-		)
-		(stroke
-			(width 0)
-			(type default)
-		)
-	)
-	(wire
-		(pts
 			(xy 227.33 96.52) (xy 227.33 93.98)
 		)
@@
 	(bus
 		(pts
-			(xy 67.31 83.82) (xy 67.31 86.36)
+			(xy 64.77 83.82) (xy 64.77 86.36)
 		)
 		(stroke
@@
 	(wire
 		(pts
+			(xy 67.31 88.9) (xy 107.95 88.9)
+		)
+		(stroke
+			(width 0)
+			(type default)
+		)
+	)
+	(wire
+		(pts
 			(xy 233.68 83.82) (xy 233.68 86.36)
 		)
@@
 		(pts
 			(xy 165.1 77.47) (xy 165.1 80.01)
+		)
+		(stroke
+			(width 0)
+			(type default)
+		)
+	)
+	(bus
+		(pts
+			(xy 64.77 76.2) (xy 64.77 83.82)
 		)
 		(stroke
@@
 		)
 	)
-	(label "USBOUT2.D-"
-		(at 90.17 86.36 180)
-		(fields_autoplaced yes)
-		(effects
-			(font
-				(size 1.27 1.27)
-				(italic yes)
-			)
-			(justify right bottom)
+	(label "USB_MCU.+"
+		(at 78.74 88.9 0)
+		(effects
+			(font
+				(size 1.27 1.27)
+			)
+			(justify left bottom)
+		)
+	)
+	(label "USB_MCU.-"
+		(at 78.74 86.36 0)
+		(effects
+			(font
+				(size 1.27 1.27)
+			)
+			(justify left bottom)
 		)
 	)
@@
 	(label "USBOUT1.D-"
 		(at 90.17 91.44 180)
-		(fields_autoplaced yes)
-		(effects
-			(font
-				(size 1.27 1.27)
-				(italic yes)
-			)
-			(justify right bottom)
-		)
-	)
-	(label "USBOUT2.D+"
-		(at 90.17 88.9 180)
 		(fields_autoplaced yes)
 		(effects
@@
 		)
 	)
-	(hierarchical_label "USBOUT1.{+ -}"
+	(hierarchical_label "USBOUT1{USB}"
 		(shape input)
 		(at 46.99 85.09 180)
@@
 		)
 	)
-	(hierarchical_label "USBOUT2.{+ -}"
+	(hierarchical_label "USB_MCU{USB}"
 		(shape input)
-		(at 46.99 80.01 180)
+		(at 59.69 76.2 180)
 		(fields_autoplaced yes)
 		(effects
