File: USB-hub.kicad_sch (KiCad schematic)
At the start: 11 parts, among them U900 CH334R, Y900 12Mhz

Commit message: Change CH334R to CH334P
Parts:
- removed C901: 1uF, PCM_JLCPCB:C_0402, symbol PCM_JLCPCB-Capacitors:0402,1uF
- removed C903: 100nF, PCM_JLCPCB:C_0402, symbol PCM_JLCPCB-Capacitors:0402,100nF,(2)
- removed U900: CH334R, Package_SO:QSOP-16_3.9x4.9mm_P0.635mm, symbol WCH_USB:CH334R
- added D301: Red, PCM_JLCPCB:D_0603, symbol PCM_JLCPCB-Diodes:LED,0603,Red
- added R308: 1kΩ, PCM_JLCPCB:R_0402, symbol PCM_JLCPCB-Resistors:0402,1kΩ
- added U302: CH334P, Package_DFN_QFN:QFN-16-1EP_3x3mm_P0.5mm_EP1.7x1.7mm, symbol CH334P:CH334P
Connections:
- net +5V: now also D301.2, U302.15 (5V)
- net GND: now also U302.17 (GND)
- net USBIN1.D+: now also U302.12 (DPU)
- net USBIN1.D-: now also U302.11 (DMU)
- net at R900.2: now also U302.5 (DM3)
- net at C900.1, C902.1: now also U302.16 (3V3)
- net at R902.2: now also U302.3 (DM4)
- net at R903.2: now also U302.4 (DP4)
- net at R901.2: now also U302.6 (DP3)
- net at Y900.1: now also U302.1 (XO)
- net at Y900.3: now also U302.2 (XI)
- new net: R308.1, U302.14 (PGANG)
- new net: D301.1, R308.2
Other:
- moved on the sheet: C900, C902, C904, R900, R901, R902, R903, Y900

Commit message: [#2] WIP: Layout USB
Connections:
- net USB_MCU_R.D-: now reaches R900.2, U302.5 (DM3)
- net USBOUT1_R.D-: now reaches R902.2, U302.3 (DM4)
- net USBOUT1_R.D+: now reaches R903.2, U302.4 (DP4)
- net USB_MCU_R.D+: now reaches R901.2, U302.6 (DP3)
Other:
- moved on the sheet: C900, C902, C904, R900, R901, R902, R903

Commit message: [#4] Improve schematic aesthetics, color nets
Other:
- title: (none) -> ModuCard base module
Changed lines of the file:
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@@
 	(paper "A4")
 	(title_block
-		(date "2024-12-23")
+		(title "ModuCard base module")
+		(date "2025-02-18")
 		(rev "1.0.0")
 		(company "KoNaR")
 		(comment 1 "Base project authors: Dominik Pluta, Artem Horiunov")
+		(comment 2 "Project author: <author>")
 	)
 	(bus_alias "USB"
@@
 	)
 	(bus_entry
-		(at 57.15 83.82)
-		(size 2.54 2.54)
+		(at 59.69 86.36)
+		(size -2.54 2.54)
 		(stroke
 			(width 0)
@@
 	(bus_entry
 		(at 59.69 95.25)
-		(size -2.54 -2.54)
+		(size -2.54 2.54)
 		(stroke
 			(width 0)
@@
 	(bus_entry
 		(at 59.69 97.79)
-		(size -2.54 -2.54)
+		(size -2.54 2.54)
 		(stroke
 			(width 0)
@@
 	)
 	(bus_entry
-		(at 57.15 86.36)
-		(size 2.54 2.54)
+		(at 59.69 88.9)
+		(size -2.54 2.54)
 		(stroke
 			(width 0)
@@
 		)
 	)
+	(bus
+		(pts
+			(xy 57.15 91.44) (xy 57.15 93.98)
+		)
+		(stroke
+			(width 0)
+			(type default)
+		)
+	)
 	(wire
 		(pts
@@
 		)
 	)
+	(bus
+		(pts
+			(xy 53.34 95.25) (xy 55.88 95.25)
+		)
+		(stroke
+			(width 0)
+			(type default)
+		)
+	)
 	(wire
 		(pts
@@
 		)
 	)
+	(bus
+		(pts
+			(xy 57.15 88.9) (xy 57.15 91.44)
+		)
+		(stroke
+			(width 0)
+			(type default)
+		)
+	)
 	(wire
 		(pts
@@
 		)
 	)
-	(bus
-		(pts
-			(xy 171.45 97.79) (xy 171.45 95.25)
-		)
-		(stroke
-			(width 0)
-			(type default)
-		)
-	)
 	(wire
 		(pts
@@
 	(bus
 		(pts
-			(xy 54.61 81.28) (xy 57.15 81.28)
+			(xy 57.15 100.33) (xy 57.15 102.87)
+		)
+		(stroke
+			(width 0)
+			(type default)
+		)
+	)
+	(bus
+		(pts
+			(xy 172.72 99.06) (xy 171.45 97.79)
+		)
+		(stroke
+			(width 0)
+			(type default)
+		)
+	)
+	(bus
+		(pts
+			(xy 57.15 97.79) (xy 57.15 100.33)
 		)
 		(stroke
@@
 	(bus
 		(pts
-			(xy 57.15 90.17) (xy 57.15 92.71)
+			(xy 53.34 104.14) (xy 55.88 104.14)
 		)
 		(stroke
@@
 		)
 	)
-	(bus
-		(pts
-			(xy 171.45 97.79) (xy 173.99 97.79)
-		)
-		(stroke
-			(width 0)
-			(type default)
-		)
-	)
 	(wire
 		(pts
@@
 		)
 	)
+	(bus
+		(pts
+			(xy 57.15 93.98) (xy 55.88 95.25)
+		)
+		(stroke
+			(width 0)
+			(type default)
+		)
+	)
 	(wire
 		(pts
@@
 		)
 	)
-	(bus
-		(pts
-			(xy 57.15 83.82) (xy 57.15 86.36)
-		)
-		(stroke
-			(width 0)
-			(type default)
-		)
-	)
 	(wire
 		(pts
@@
 		)
 	)
+	(bus
+		(pts
+			(xy 172.72 99.06) (xy 175.26 99.06)
+		)
+		(stroke
+			(width 0)
+			(type default)
+		)
+	)
 	(wire
 		(pts
@@
 		)
 	)
+	(bus
+		(pts
+			(xy 57.15 102.87) (xy 55.88 104.14)
+		)
+		(stroke
+			(width 0)
+			(type default)
+		)
+	)
 	(wire
 		(pts
@@
 		)
 	)
-	(bus
-		(pts
-			(xy 57.15 92.71) (xy 57.15 95.25)
-		)
-		(stroke
-			(width 0)
-			(type default)
-		)
-	)
 	(wire
 		(pts
@@
 	(bus
 		(pts
-			(xy 57.15 81.28) (xy 57.15 83.82)
+			(xy 171.45 95.25) (xy 171.45 97.79)
 		)
 		(stroke
@@
 		(pts
 			(xy 158.75 48.26) (xy 162.56 48.26)
-		)
-		(stroke
-			(width 0)
-			(type default)
-		)
-	)
-	(bus
-		(pts
-			(xy 57.15 90.17) (xy 54.61 90.17)
 		)
 		(stroke
@@
 	(hierarchical_label "USBIN1{USB}"
 		(shape input)
-		(at 173.99 97.79 0)
+		(at 175.26 99.06 0)
 		(effects
 			(font
@@
 	(hierarchical_label "USBOUT1{USB}"
 		(shape input)
-		(at 54.61 90.17 180)
+		(at 53.34 104.14 180)
 		(effects
 			(font
@@
 	(hierarchical_label "USB_MCU{USB}"
 		(shape input)
-		(at 54.61 81.28 180)
-		(effects
-			(font
+		(at 53.34 95.25 180)
+		(effects
+			(font
