File: base-module.kicad_pcb (KiCad board)
At the start: 4 copper layers, 100 x 100 mm, 135 parts, among them J200 09031967921, J900 USB_C_Receptacle_USB2.0_16P, Q700 S9013, SW400 TL2243, U200 IP4234CZ6,115, U300 TPS563201DDCR, U301 TPS563201DDCR, U400 STM32F750V8Tx, U401 W25Q128, U500 TJA1044GTK_3Z, U600 TJA1044GTK_3Z, U700 STM32F103CBTx, U800 IP4234CZ6,115, U801 TS3USB30ERSWR, U900 CH334R, X400 X322512MSB4SI, X700 X50328MSB2GI, Y900 12Mhz

Commit message: [#2] Connect CAN transcievers and TVS to backplane connector, setup differential pairs
Parts:
- moved U200 65.3 mm to (126.0, 155.5), turned to 180 degrees
- moved U600 58.6 mm to (109.6, 155.1), turned to -90 degrees
- moved C601 57.5 mm to (107.4, 155.1), turned to 90 degrees
- moved C600 56.2 mm to (109.6, 152.5), turned to 180 degrees
- moved R600 54.7 mm to (111.8, 155.1), turned to 90 degrees
- moved U500 49.3 mm to (117.2, 155.1), turned to -90 degrees
- moved C501 48.5 mm to (115.0, 155.1), turned to 90 degrees
- moved C500 47.4 mm to (117.2, 152.5), turned to 180 degrees
- moved R500 46.1 mm to (119.4, 155.1), turned to 90 degrees
- moved TP304 7.03 mm to (88.6, 115.2)
- moved TP305 7.03 mm to (88.6, 118.2)
- moved TP300 7.03 mm to (82.5, 115.2)
- moved TP301 7.03 mm to (82.5, 118.2)
- moved TP302 7.03 mm to (85.5, 115.2)
- moved TP303 7.03 mm to (85.5, 118.2)
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Routing:
- net GND: track 3.42 -> 21.1 mm, vias 1 -> 8
- net +5v_stdby: track 0.00 -> 10.6 mm
- net /Backplane/BACKPLANE_U.D+: track 0.00 -> 8.70 mm
- net +5V: track 0.00 -> 3.64 mm, vias 0 -> 2
- net +3V3: track 3.62 -> 6.85 mm, vias 1 -> 3
- net /Backplane/BACKPLANE_U.D-: track 0.00 -> 2.94 mm
- net /Backplane/CAN2.+: track 0.00 -> 2.74 mm
- net /Backplane/CAN2.-: track 0.00 -> 2.74 mm
- net /Backplane/CAN1.-: track 0.00 -> 2.74 mm
- net /Backplane/CAN1.+: track 0.00 -> 2.74 mm
- net /USB/USB2S.D+: track 2.25 -> 0.00 mm, vias 1 -> 0
- net Net-(U600-STB): track 0.00 -> 1.62 mm
- net Net-(U500-STB): track 0.00 -> 1.62 mm
- net /USB/USB2S.D-: track 1.61 -> 0.00 mm
- added copper zone on In1.Cu, net GND

Commit message: [#2] WIP: Layout DC-DC converters, MCU
Parts:
- removed C425: 100nF, PCM_JLCPCB:C_0402
- removed D301, D302, D303, D304: Green, PCM_JLCPCB:D_0603
- removed J900: USB_C_Receptacle_USB2.0_16P, Connector_USB:USB_C_Receptacle_GCT_USB4105-xx-A_16P_TopMnt_Horizontal
- removed R904, R905: 5.1kΩ, PCM_JLCPCB:R_0402
- removed U401: W25Q128, PCM_JLCPCB:SOIC-8_L5.3-W5.3-P1.27-LS8.0-BL
- added C100: 100nF, PCM_JLCPCB:C_0402, F.Cu at (127.6, 77.7)
- added C311: 100nF, PCM_JLCPCB:C_0402, F.Cu at (101.5, 154.8)
- added J800: USB_C_Receptacle_USB2.0_16P, Connector_USB:USB_C_Receptacle_GCT_USB4105-xx-A_16P_TopMnt_Horizontal, F.Cu at (107.0, 72.2)
- added LED300: FixLed307, FixLed307:FixLed307, F.Cu at (77.5, 72.2)
- added LED301: FixLed307, FixLed307:FixLed307, F.Cu at (83.4, 72.2)
- added R803: 22kΩ, PCM_JLCPCB:R_0402, F.Cu at (124.1, 153.6)
- added R804: 10kΩ, PCM_JLCPCB:R_0402, F.Cu at (129.4, 151.2)
- added R805: 330Ω, PCM_JLCPCB:R_0402, F.Cu at (113.7, 74.9)
- added U100: W25Q128, PCM_JLCPCB:SOIC-8_L5.3-W5.3-P1.27-LS8.0-BL, F.Cu at (122.9, 82.0)
- added X300: Q13FC1350000400, PCM_JLCPCB:FC-135R_L3.2-W1.5, F.Cu at (80.3, 122.2)
- C306: value 22uF -> 100nF; footprint PCM_JLCPCB:C_0603 -> PCM_JLCPCB:C_0402
- C308: value 10uF -> 22uF
- C310: value 100nF -> 10uF; footprint PCM_JLCPCB:C_0402 -> PCM_JLCPCB:C_0603
- R302: value 33k2 -> 1.2kΩ
- R304: value 1.2kΩ -> 470Ω
- R305: value 470Ω -> 120Ω
- R306: value 120Ω -> 33k2
- R800, R801: value 10kΩ -> 5.1kΩ
- R802: value 330Ω -> 10kΩ
- SW400: footprint kicad-footprints:TL2243 -> TL2243:TL2243
- U801: value TS3USB30ERSWR -> FSUSB42UMX
- moved TP305 103.6 mm to (188.2, 146.8)
- moved TP306 103.6 mm to (191.2, 143.7)
- moved TP307 103.6 mm to (191.2, 146.8)
- moved R703 85.4 mm to (131.7, 147.2), turned to -90 degrees
- moved R701 84.5 mm to (130.7, 147.2), turned to 90 degrees
- moved R700 83.7 mm to (129.7, 147.2), turned to 90 degrees
- moved C706 82.8 mm to (128.7, 147.2), turned to -90 degrees
- moved L301 77.1 mm to (79.7, 148.3), turned to -90 degrees
- moved X700 76.7 mm to (127.1, 143.1), turned to 0 degrees
- moved C304 75.6 mm to (103.9, 156.2), turned to 0 degrees
- moved R301 75.5 mm to (105.8, 153.7), turned to -90 degrees
- moved F300 75.2 mm to (100.5, 156.6), turned to 180 degrees
- moved C708 74.9 mm to (128.0, 140.8), turned to 180 degrees
- moved R704 74.6 mm to (133.8, 134.8), turned to 0 degrees
- moved FB400 73.9 mm to (48.0, 132.1), turned to -90 degrees
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Connections:
- net Net-(U300-SW) renamed /Power/SW_5V0
- C300 pad 1: /Power/VBST -> /Power/VBST_5V0
- C305 pad 1: /Power/VBST -> GND
- C305 pad 2: Net-(U301-SW) -> +12V_FUSED
- C306 pad 1: /Power/3V3_UNPROTEC -> /Power/VBST_3V3
- C306 pad 2: GND -> /Power/SW_3V3
- C308 pad 1: +12V_FUSED -> /Power/3V3_UNPROTEC
- C310 pad 1: GND -> +12V_FUSED
- C310 pad 2: +12V_FUSED -> GND
- C801 pad 1: Net-(J900-SHIELD) -> Net-(J800-SHIELD)
- L301 pad 1: Net-(U301-SW) -> /Power/SW_3V3
- R300 pad 2: /Power/FB -> /Power/FB_5V0
- R301 pad 1: /Power/FB -> /Power/FB_5V0
- R302 pad 1: /Power/3V3_UNPROTEC -> +12V
- R302 pad 2: /Power/FB -> Net-(LED300-Pad1)
- R303 pad 1: Net-(D301-Pad1) -> +12V_FUSED
- R303 pad 2: GND -> Net-(LED300-Pad3)
- R304 pad 1: Net-(D302-Pad1) -> +5V
- R304 pad 2: GND -> Net-(LED301-Pad1)
- R305 pad 1: Net-(D303-Pad1) -> +3V3
- R305 pad 2: GND -> Net-(LED301-Pad3)
- R306 pad 1: Net-(D304-Pad1) -> /Power/3V3_UNPROTEC
- R306 pad 2: GND -> /Power/FB_3V3
- R307 pad 1: /Power/FB -> /Power/FB_3V3
- R800 pad 1: /USB/VBUS_IN -> /USB/CC2
- R801 pad 1: Net-(U801-~{OE}) -> /USB/CC1
- R802 pad 1: Net-(J900-SHIELD) -> /USB/VBUS_IN
- R802 pad 2: GND -> Net-(U801-SEL)
- TP303 pad 1: /Power/FB -> /Power/FB_5V0
- TP307 pad 1: /Power/FB -> /Power/FB_3V3
- U200 pad 1: /Backplane/BACKPLANE_U.D- -> /Backplane/BACKPLANE_U.D+
- U200 pad 3: /Backplane/BACKPLANE.D- -> /Backplane/BACKPLANE.D+
- U200 pad 4: /Backplane/BACKPLANE.D+ -> /Backplane/BACKPLANE.D-
- U200 pad 6: /Backplane/BACKPLANE_U.D+ -> /Backplane/BACKPLANE_U.D-
- U300 pad 4: /Power/FB -> /Power/FB_5V0
- U300 pad 6: /Power/VBST -> /Power/VBST_5V0
- U301 pad 2: Net-(U301-SW) -> /Power/SW_3V3
- U301 pad 4: /Power/FB -> /Power/FB_3V3
- U301 pad 6: /Power/VBST -> /Power/VBST_3V3
- U400 pad 12: /MCU/PH0 -> /MCU/OSC_IN
- U400 pad 13: /MCU/PH1 -> /MCU/OSC_OUT
- U801 pad 1: /USB/USB2S.D+ -> /USB-hub/USBIN1.D+
- U801 pad 10: /USB/VBUS_IN -> Net-(U801-SEL)
- U801 pad 2: /Backplane/BACKPLANE.D+ -> /USB-hub/USBIN1.D-
- U801 pad 3: /USB-hub/USBIN1.D+ -> GND
- U801 pad 4: GND -> /Backplane/BACKPLANE.D-
- U801 pad 5: /USB-hub/USBIN1.D- -> /Backplane/BACKPLANE.D+
- U801 pad 6: /Backplane/BACKPLANE.D- -> /USB/USB2S.D-
- U801 pad 7: /USB/USB2S.D- -> /USB/USB2S.D+
- U801 pad 9: +5V -> +3V3
Routing:
- net GND: track 21.1 -> 33.8 mm, vias 8 -> 18
- net +3V3: track 6.85 -> 17.0 mm, vias 3 -> 6
- net /USB/USB2U.D-: track 0.00 -> 5.15 mm
- net /Backplane/CAN2.-: track 2.74 -> 7.82 mm
- net /Backplane/CAN2.+: track 2.74 -> 7.82 mm
- net /Backplane/CAN1.-: track 2.74 -> 7.82 mm
- net /Backplane/CAN1.+: track 2.74 -> 7.82 mm
- net /USB/USB2U.D+: track 0.00 -> 4.38 mm
- net /Power/FB_5V0: track 0.00 -> 3.97 mm
- net /Power/5V_UNPROTEC: track 0.00 -> 3.27 mm
- net /Power/SW_5V0: track 0.00 -> 3.24 mm
- net +12V_FUSED: track 0.00 -> 2.90 mm
- net /Backplane/BACKPLANE.D+: track 0.00 -> 2.27 mm
- net /Backplane/BACKPLANE.D-: track 0.00 -> 2.27 mm
- net /Power/VBST_5V0: track 0.00 -> 1.53 mm
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- added copper zone on F.Cu, net +12V
- added copper zone on F.Cu, net /Power/5V_UNPROTEC
- added copper zone on F.Cu, net /Power/SW_5V0
- added copper zone on F.Cu, net GND

Commit message: Change CH334R to CH334P
Parts:
- removed C901: 1uF, PCM_JLCPCB:C_0402
- removed C903: 100nF, PCM_JLCPCB:C_0402
- removed U900: CH334R, Package_SO:QSOP-16_3.9x4.9mm_P0.635mm
- added D301: Red, PCM_JLCPCB:D_0603, F.Cu at (143.1, 157.2)
- added R308: 1kΩ, PCM_JLCPCB:R_0402, F.Cu at (146.5, 156.8)
- added U302: CH334P, Package_DFN_QFN:QFN-16-1EP_3x3mm_P0.5mm_EP1.7x1.7mm, F.Cu at (143.7, 153.2)
- moved R304 2.52 mm to (77.7, 79.8)
- moved R303 2.02 mm to (81.3, 79.4)
- moved R306 2.02 mm to (80.1, 79.2)
- moved R305 2.02 mm to (78.7, 79.2)
- moved LED301 1.42 mm to (83.7, 73.6)
- moved LED300 1.42 mm to (77.8, 73.6)

Commit message: [#2] WIP: Layout USB
Parts:
- added C312: 100nF, PCM_JLCPCB:C_0402, F.Cu at (132.1, 153.6)
- moved R901 30.8 mm to (124.1, 153.1)
- moved R903 30.3 mm to (126.4, 149.9), turned to -90 degrees
- moved C100 29.6 mm to (98.8, 84.4)
- moved TP700 29.6 mm to (90.0, 96.1)
- moved TP701 29.6 mm to (90.0, 99.1)
- moved U100 29.6 mm to (94.1, 88.7)
- moved R902 28.8 mm to (127.3, 149.9), turned to -90 degrees
- moved R900 25.8 mm to (124.1, 152.2)
- moved C800 18.6 mm to (128.3, 78.1)
- moved J800 18.6 mm to (125.5, 72.8)
- moved R800 18.6 mm to (120.8, 78.8)
- moved R801 18.6 mm to (130.0, 78.6)
- moved U800 18.6 mm to (125.0, 79.3)
- moved C801 18.6 mm to (132.2, 76.5)
- moved R805 18.6 mm to (132.2, 75.5)
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Connections:
- net Net-(U302-DM3) renamed /USB-hub/USB_MCU_R.D-
- net Net-(U302-DM4) renamed /USB-hub/USBOUT1_R.D-
- net Net-(U302-DP3) renamed /USB-hub/USB_MCU_R.D+
- net Net-(U302-DP4) renamed /USB-hub/USBOUT1_R.D+
- J800 pad A6: /USB/USB2U.D- -> /USB/USB2U.D+
- J800 pad A7: /USB/USB2U.D+ -> /USB/USB2U.D-
- J800 pad B6: /USB/USB2U.D- -> /USB/USB2U.D+
- J800 pad B7: /USB/USB2U.D+ -> /USB/USB2U.D-
- U800 pad 1: /USB/USB2U.D- -> /USB/USB2U.D+
- U800 pad 3: /USB/USB2S.D- -> /USB/USB2S.D+
- U800 pad 4: /USB/USB2S.D+ -> /USB/USB2S.D-
- U800 pad 6: /USB/USB2U.D+ -> /USB/USB2U.D-
Routing:
- net /USB/USB2S.D-: track 1.40 -> 87.2 mm
- net /USB/USB2S.D+: track 1.40 -> 86.6 mm
- net Net-(U801-SEL): track 0.00 -> 5.98 mm
- net Net-(U302-XO): track 0.00 -> 5.03 mm
- net +5v_stdby: track 9.90 -> 14.8 mm
- net /USB-hub/USBIN1.D-: track 0.62 -> 4.80 mm
- net Net-(U302-XI): track 0.00 -> 3.95 mm
- net Net-(U801-~{OE}): track 0.00 -> 3.90 mm, vias 0 -> 2
- net /USB-hub/USBIN1.D+: track 1.17 -> 4.67 mm
- net /Backplane/BACKPLANE_U.D-: track 3.34 -> 6.01 mm
- net GND: track 33.8 -> 35.4 mm, vias 18 -> 24
- net /USB-hub/USBOUT1_R.D+: track 0.00 -> 1.41 mm
- net /USB-hub/USB_MCU_R.D+: track 0.00 -> 1.41 mm
- net /USB-hub/USBOUT1_R.D-: track 0.00 -> 1.41 mm
- net /USB-hub/USB_MCU_R.D-: track 0.00 -> 1.41 mm
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
Commit message: [#2] WIP: Layout USB, ST-LINK, move CAN transcievers
Parts:
- removed X700: X50328MSB2GI, PCM_JLCPCB:CRYSTAL-SMD_L5.0-W3.2
- added Y700: 8 MHz, PCM_JLCPCB:CRYSTAL-SMD_4P-L3.2-W2.5-BL, F.Cu at (127.5, 130.7)
- TP702, TP703, TP704, TP705, TP706: moved to B.Cu
- moved TP700 45.9 mm to (122.2, 128.7)
- moved R713 30.9 mm to (100.1, 126.1), turned to -90 degrees
- moved R707 30.8 mm to (100.1, 124.1), turned to -90 degrees
- moved D700 26.9 mm to (102.0, 124.0), turned to 180 degrees
- moved D701 26.8 mm to (102.1, 126.0), turned to 0 degrees
- moved TP302 21.7 mm to (94.5, 149.7)
- moved TP300 21.7 mm to (91.4, 149.7)
- moved TP301 21.7 mm to (91.4, 152.7)
- moved Q700 20.5 mm to (114.2, 139.9), turned to 0 degrees
- moved R712 20.4 mm to (130.1, 145.8), turned to 180 degrees
- moved R714 19.4 mm to (123.0, 144.6), turned to 90 degrees
- moved R715 18.7 mm to (123.9, 144.6), turned to 90 degrees
- moved C900 18.7 mm to (130.3, 151.9), turned to 90 degrees
- moved D301 18.4 mm to (124.8, 155.4), turned to 90 degrees
- moved R703 18.3 mm to (120.0, 131.0), turned to 90 degrees
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Connections:
- U200 pad 5: +5v_stdby -> +5V
Routing:
- net GND: track 35.4 -> 55.0 mm, vias 24 -> 40
- net +5v_stdby: track 14.8 -> 5.08 mm
- net /Backplane/CAN2.+: track 7.82 -> 15.3 mm
- net /Backplane/CAN2.-: track 7.82 -> 15.3 mm
- net +3V3: track 18.2 -> 25.3 mm, vias 6 -> 11
- net /ST-LINK/ST-LINK.D+: track 0.00 -> 6.94 mm, vias 0 -> 2
- net /ST-LINK/ST-LINK.D-: track 0.00 -> 6.78 mm, vias 0 -> 2
- net Net-(U302-PGANG): track 0.00 -> 5.66 mm, vias 0 -> 2
- net +5V: track 3.64 -> 8.36 mm, vias 2 -> 5
- net /Backplane/CAN1.+: track 7.82 -> 12.3 mm
- net /Backplane/CAN1.-: track 7.82 -> 12.3 mm
- net /ST-LINK/STLINK-OSC_OUT: track 6.49 -> 3.32 mm
- net Net-(U700-PA0): track 0.00 -> 3.04 mm
- net Net-(U700-PC13): track 3.02 -> 6.03 mm, vias 0 -> 2
- net /USB-hub/USB_MCU_R.D+: track 1.41 -> 3.54 mm
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- added copper zone on In2.Cu, net +3V3

Commit message: [#2] Connect MCU to ST-LINK, route DC-DC converters
Parts:
- removed TP303, TP307: Buck Feedback, TestPoint:TestPoint_Pad_D1.0mm
- removed TP304: TestPoint, TestPoint:TestPoint_Pad_D1.0mm
- Q700: value S9013 -> MMST3904; footprint PCM_JLCPCB:Q_SOT-23 -> PCM_JLCPCB:Q_SOT-323
- moved TP306 120.6 mm to (71.1, 154.7)
- moved TP305 112.6 mm to (75.8, 153.2)
- moved R306 79.6 mm to (114.0, 151.1), turned to -90 degrees
- moved R302 67.9 mm to (76.5, 79.1)
- moved TP701 47.6 mm to (120.0, 136.1)
- moved R307 42.4 mm to (114.0, 153.0), turned to -90 degrees
- moved JP301 40.7 mm to (113.6, 148.1), turned to 0 degrees
- moved C309 38.5 mm to (112.1, 155.6)
- moved C310 37.3 mm to (112.1, 154.3), turned to 0 degrees
- moved U301 36.7 mm to (111.5, 151.9), turned to 0 degrees
- moved C306 36.3 mm to (112.9, 149.8), turned to 180 degrees
- moved C308 35.5 mm to (111.3, 148.8), turned to -90 degrees
- moved C307 34.7 mm to (110.0, 148.8), turned to -90 degrees
- moved L301 27.4 mm to (107.0, 150.2), turned to 90 degrees
- moved C305 23.0 mm to (96.0, 152.4), turned to -90 degrees
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Routing:
- net GND: track 55.0 -> 62.3 mm, vias 40 -> 61
- net Net-(U700-PB14): track 1.82 -> 8.55 mm
- net +24V: track 0.00 -> 5.08 mm
- net Net-(Q700-B): track 0.00 -> 4.94 mm
- net /ST-LINK/USB_RENUM: track 0.00 -> 4.46 mm
- net /Power/SW_3V3: track 0.00 -> 3.24 mm
- net /Power/3V3_UNPROTEC: track 0.00 -> 3.05 mm
- net +12V_FUSED: track 2.90 -> 5.81 mm, vias 0 -> 7
- net /Power/FB_3V3: track 0.00 -> 2.43 mm
- net +3V3: track 25.3 -> 27.6 mm, vias 11 -> 14
- net /USB-hub/USBOUT1_R.D+: track 3.23 -> 1.38 mm
- net /USB-hub/USBOUT1_R.D-: track 3.23 -> 1.38 mm
- net /ST-LINK/ST-LINK.D-: track 6.78 -> 8.57 mm, vias 2 -> 0
- net /ST-LINK/ST-LINK.D+: track 6.94 -> 8.70 mm, vias 2 -> 0
- net /Power/FB_5V0: track 4.00 -> 2.43 mm
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- added copper zone on F.Cu, net +12V_FUSED
- added copper zone on In2.Cu, net +12V_FUSED
- added copper zone on F.Cu, net +5V
- added copper zone on F.Cu, net /Power/3V3_UNPROTEC
- added copper zone on F.Cu, net /Power/SW_3V3

Commit message: [#2] Fix MCU model, draft QSPI connection
Parts:
- removed D300: BZT52C5V6S, PCM_JLCPCB:D_SOD-323
- U400: value STM32F750V8Tx -> STM32H750VBTx
- moved C405 69.1 mm to (121.2, 130.1), turned to -90 degrees
- moved C410 67.1 mm to (121.4, 136.8)
- moved C400 66.0 mm to (115.5, 126.4), turned to 90 degrees
- moved C401 63.2 mm to (113.2, 126.9), turned to 0 degrees
- moved FB400 59.0 mm to (106.5, 124.8), turned to 180 degrees
- moved C406 58.5 mm to (107.4, 126.0), turned to 180 degrees
- moved C407 57.5 mm to (107.4, 126.8), turned to 180 degrees
- moved C404 57.0 mm to (118.9, 144.3), turned to -90 degrees
- moved C409 56.8 mm to (105.5, 126.0), turned to 0 degrees
- moved C408 55.8 mm to (105.5, 126.8), turned to 0 degrees
- moved C414 54.7 mm to (117.5, 145.3), turned to 0 degrees
- moved U400 53.6 mm to (112.0, 136.1), turned to -90 degrees
- moved C402 49.8 mm to (102.8, 130.1), turned to 90 degrees
- moved U100 47.8 mm to (99.7, 136.1), turned to 180 degrees
- moved C413 38.5 mm to (102.8, 141.6), turned to -90 degrees
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Routing:
- net /MCU/QSPI1.IO1: track 0.00 -> 30.5 mm
- net /MCU/QSPI1.CS: track 0.00 -> 30.2 mm
- net /MCU/QSPI1.IO2: track 0.00 -> 30.2 mm
- net /MCU/QSPI1.IO0: track 0.00 -> 29.2 mm
- net /MCU/QSPI1.SCLK: track 0.00 -> 28.4 mm
- net /MCU/QSPI1.IO3: track 0.00 -> 16.6 mm
- net /MCU/USB_MCU.D+: track 0.00 -> 16.0 mm
- net /MCU/USB_MCU.D-: track 0.00 -> 14.4 mm
- net /CAN transceiver 1/CAN.TX: track 0.00 -> 7.05 mm
- net /CAN transceiver 2/CAN.RX: track 0.00 -> 4.54 mm
- net /CAN transceiver 1/CAN.RX: track 0.00 -> 4.39 mm
- net /CAN transceiver 2/CAN.TX: track 0.00 -> 3.05 mm
- net +3V3: vias 14 -> 18
- added copper zone on F.Cu, net +3V3

Commit message: [#2] Length match QSPI
Routing:
- net /MCU/QSPI1.IO3: track 16.6 -> 29.9 mm
- net /MCU/QSPI1.SCLK: track 28.4 -> 29.4 mm
- net /MCU/QSPI1.IO0: track 29.2 -> 30.0 mm
