File: base-module.kicad_pcb (KiCad board)
At the start: 4 copper layers, 100 x 100 mm, 133 parts, among them J200 09031967921, J800 USB_C_Receptacle_USB2.0_16P, Q700 MMST3904, SW400 TL2243, U100 W25Q128, U200 IP4234CZ6,115, U300 TPS563201DDCR, U301 TPS563201DDCR, U302 CH334P, U400 STM32H750VBTx, U500 TJA1044GTK_3Z, U600 TJA1044GTK_3Z, U700 STM32F103CBTx, U800 IP4234CZ6,115, U801 FSUSB42UMX, X300 Q13FC1350000400, X400 X322512MSB4SI, Y700 8 MHz, Y900 12Mhz

Commit message: [#2] Shield power supply section from MCU
Parts:
- moved C400 1.43 mm to (115.5, 125.0)
- moved C401 1.43 mm to (113.2, 125.5)
- moved C403 1.43 mm to (103.7, 141.6)
- moved C414 1.43 mm to (117.5, 143.9)
- moved C406 1.43 mm to (107.4, 124.5)
- moved C407 1.43 mm to (107.4, 125.4)
- moved C408 1.43 mm to (105.5, 125.4)
- moved C409 1.43 mm to (105.5, 124.5)
- moved FB400 1.43 mm to (106.4, 123.3)
- moved X300 1.43 mm to (115.0, 122.0)
- moved X400 1.43 mm to (110.4, 121.8)
- moved C404 1.43 mm to (118.9, 142.9)
- moved C405 1.43 mm to (121.2, 128.7)
- moved C410 1.43 mm to (121.3, 135.4)
- moved U100 1.43 mm to (99.7, 134.7)
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Routing:
- net GND: track 62.3 -> 81.5 mm, vias 61 -> 73
- net /MCU/USB_MCU.D-: track 14.4 -> 15.9 mm
- net /MCU/USB_MCU.D+: track 16.0 -> 17.4 mm

Commit message: [#2] Add LSE oscillator, draft CAN RX/TX tracks, ensure copper balance
Parts:
- added C313: 18pF, PCM_JLCPCB:C_0402, F.Cu at (113.8, 123.1)
- added C314: 18pF, PCM_JLCPCB:C_0402, F.Cu at (115.6, 123.7)
- moved R401 85.1 mm to (126.7, 122.9)
- moved R400 85.1 mm to (126.7, 121.0)
- moved R402 85.1 mm to (126.7, 124.7)
- moved R403 77.7 mm to (119.5, 124.8), turned to 180 degrees
- moved R404 59.5 mm to (119.5, 122.9), turned to 180 degrees
- moved C415 56.6 mm to (119.5, 123.8)
- moved C100 54.0 mm to (102.8, 138.2), turned to 90 degrees
- moved C412 34.5 mm to (109.4, 124.8), turned to 180 degrees
- moved C411 30.9 mm to (111.3, 124.8), turned to 0 degrees
- moved C410 10.7 mm to (126.8, 126.2), turned to 180 degrees
- moved R708 7.43 mm to (121.8, 139.0), turned to -90 degrees
- moved X400 1.01 mm to (110.7, 122.8)
- moved R704 0.85 mm to (121.5, 145.7), turned to 0 degrees
- moved C400 0.71 mm to (116.0, 125.5), turned to 0 degrees
- moved X300 0.49 mm to (114.8, 121.5), turned to 0 degrees
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Connections:
- U400 pad 8: /MCU/PC14 -> /MCU/OSC32_IN
- U400 pad 9: /MCU/PC15 -> /MCU/OSC32_OUT
- X300 pad 1: unconnected-(X300-Pad1) -> /MCU/OSC32_OUT
- X300 pad 2: unconnected-(X300-Pad2) -> /MCU/OSC32_IN
Routing:
- net /CAN transceiver 2/CAN.TX: track 3.05 -> 24.7 mm, vias 0 -> 2
- net /CAN transceiver 2/CAN.RX: track 4.54 -> 24.1 mm, vias 0 -> 2
- net /CAN transceiver 1/CAN.RX: track 4.39 -> 18.6 mm, vias 0 -> 2
- net /CAN transceiver 1/CAN.TX: track 7.05 -> 19.6 mm, vias 0 -> 2
- net /MCU/SWD.SWDIO: track 0.00 -> 10.1 mm
- net /MCU/SWD.SWCLK: track 0.00 -> 7.44 mm
- net GND: track 81.5 -> 87.3 mm, vias 73 -> 81
- net +3V3: track 27.6 -> 32.4 mm, vias 18 -> 20
- net /MCU/OSC32_OUT: track 0.00 -> 3.25 mm
- net /MCU/OSC32_IN: track 0.00 -> 2.53 mm
- net Net-(U700-PB0): track 0.00 -> 1.59 mm
- net /MCU/USB_MCU.D-: track 15.9 -> 15.1 mm
- net /MCU/USB_MCU.D+: track 17.4 -> 16.7 mm

Commit message: [#2] Position front panel parts, add 3d models, continue layout
Parts:
- added kibuzzard-67B20BD5: G***, kibuzzard-67B20BD5, F.Cu at (129.1, 129.2)
- added kibuzzard-67B2198C: G***, kibuzzard-67B2198C, F.Cu at (134.5, 129.2)
- added kibuzzard-67B219C6: G***, kibuzzard-67B219C6, F.Cu at (134.5, 131.2)
- moved TP302 105.9 mm to (179.1, 142.9)
- moved TP300 101.8 mm to (172.3, 140.8)
- moved TP306 101.8 mm to (172.2, 143.0)
- moved TP301 101.8 mm to (174.7, 142.8)
- moved TP305 101.7 mm to (176.9, 142.8)
- moved LED300 30.3 mm to (108.0, 73.6)
- moved R302 29.4 mm to (106.0, 79.1)
- moved R305 29.4 mm to (108.2, 79.2)
- moved LED301 29.4 mm to (113.1, 73.6)
- moved R303 29.4 mm to (110.8, 79.4)
- moved R304 29.4 mm to (107.2, 79.8)
- moved R805 18.5 mm to (114.8, 82.0)
- moved C801 16.3 mm to (117.2, 83.1)
- moved R400 11.3 mm to (123.9, 131.9), turned to -90 degrees
- moved R707 10.7 mm to (123.2, 127.2), turned to 0 degrees
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Routing:
- net /USB/VBUS_IN: track 0.86 -> 81.0 mm, vias 1 -> 2
- net /ST-LINK/LED: track 0.00 -> 18.7 mm, vias 0 -> 2
- net GND: track 87.3 -> 100.8 mm, vias 81 -> 93
- net /ST-LINK/STLINK_RX: track 0.00 -> 12.5 mm, vias 0 -> 2
- net /ST-LINK/STLINK_TX: track 0.00 -> 12.5 mm, vias 0 -> 2
- net Net-(U700-PA5): track 0.00 -> 11.1 mm, vias 0 -> 2
- net /ST-LINK/STLINK-RST: track 0.00 -> 8.37 mm
- net /MCU/OSC_IN: track 0.00 -> 6.80 mm
- net /MCU/OSC_OUT: track 0.00 -> 5.25 mm
- net /MCU/BOOT0: track 0.00 -> 4.83 mm
- net +3V3: track 32.4 -> 37.1 mm, vias 20 -> 25
- net Net-(U400-VDDA): track 0.00 -> 4.50 mm
- net /USB/USB2S.D-: track 87.2 -> 90.8 mm
- net /USB/USB2S.D+: track 86.6 -> 90.2 mm
- net /MCU/OSC32_IN: track 2.53 -> 5.20 mm
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- added copper zone on B.Cu, net +5V

Commit message: [#2] Route front panel components
Parts:
- added kibuzzard-67B222E6: G***, kibuzzard-67B222E6, F.Cu at (125.7, 85.4)
- moved TP306 93.8 mm to (103.3, 79.4)
- moved TP302 89.3 mm to (111.0, 85.0)
- moved TP305 89.2 mm to (109.0, 85.0)
- moved TP301 89.1 mm to (107.0, 85.0)
- moved TP300 88.9 mm to (103.0, 85.0)
- moved R304 8.13 mm to (115.2, 79.0), turned to 90 degrees
- moved R302 7.47 mm to (113.5, 79.0)
- moved R305 6.17 mm to (114.3, 79.0)
- moved C801 4.20 mm to (116.2, 79.0), turned to -90 degrees
- moved R805 3.69 mm to (117.0, 79.0), turned to -90 degrees
- moved R404 2.77 mm to (118.5, 125.5)
- moved R303 1.80 mm to (112.5, 79.0)
- moved C415 1.03 mm to (118.5, 123.7)
- moved R403 1.03 mm to (118.5, 124.6)
- moved R801 0.79 mm to (127.0, 78.2), turned to 180 degrees
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Routing:
- net /MCU/SWD.~{RST}: track 0.00 -> 122.6 mm, vias 0 -> 3
- net Net-(R400-Pad1): track 0.00 -> 96.9 mm, vias 0 -> 1
- net Net-(J800-SHIELD): track 0.00 -> 20.7 mm
- net Net-(LED300-Pad1): track 0.00 -> 9.79 mm
- net /USB/CC1: track 0.00 -> 9.26 mm
- net /USB/VBUS_IN: track 81.0 -> 90.2 mm
- net GND: track 100.8 -> 107.9 mm, vias 93 -> 100
- net Net-(LED301-Pad1): track 0.00 -> 6.83 mm
- net Net-(LED300-Pad3): track 0.00 -> 6.78 mm
- net Net-(LED301-Pad3): track 0.00 -> 3.76 mm
- net /USB/CC2: track 0.00 -> 3.48 mm
- net /MCU/NRST: track 0.00 -> 2.25 mm
- net +3V3: track 37.1 -> 38.4 mm, vias 25 -> 27
- net +5V: track 8.96 -> 9.61 mm, vias 10 -> 11
- net +12V_FUSED: track 5.81 -> 6.46 mm, vias 7 -> 8
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
Commit message: [#2] Route everything except for some test points, fix LED and button configuration
Parts:
- removed R302, R303: 1.2kΩ, PCM_JLCPCB:R_0402
- removed R304: 470Ω, PCM_JLCPCB:R_0402
- removed R305: 120Ω, PCM_JLCPCB:R_0402
- removed kibuzzard-67B222E6: G***, kibuzzard-67B222E6
- added C416: 100nF, PCM_JLCPCB:C_0402, F.Cu at (100.5, 76.6)
- added R405: 10kΩ, PCM_JLCPCB:R_0402, F.Cu at (100.5, 77.5)
- added R406: 100Ω, PCM_JLCPCB:R_0402, F.Cu at (100.5, 75.7)
- added R407: 1.2kΩ, PCM_JLCPCB:R_0402, F.Cu at (112.5, 79.0)
- added R408: 470Ω, PCM_JLCPCB:R_0402, F.Cu at (115.2, 79.0)
- added R409: 120Ω, PCM_JLCPCB:R_0402, F.Cu at (114.3, 79.0)
- R400: value 1kΩ -> 1.2kΩ
- moved R400 53.9 mm to (113.5, 79.0), turned to 90 degrees
- moved TP306 6.32 mm to (97.9, 82.6)
- moved R801 3.25 mm to (124.8, 80.5), turned to 0 degrees
- moved C415 0.88 mm to (119.4, 123.7)
- moved R403 0.88 mm to (119.4, 124.6)
- moved R404 0.88 mm to (119.3, 125.5)
- moved C800 0.25 mm to (124.8, 78.3)
Connections:
- R400 pad 1: Net-(R400-Pad1) -> /MCU/USER_LED_1
- R400 pad 2: /MCU/BOOT0 -> Net-(LED300-Pad1)
- SW400 pad 1: Net-(R400-Pad1) -> GND
- SW400 pad 4: +3V3 -> /MCU/USR_BUTTON
- U400 pad 2: /MCU/PE3 -> /MCU/USER_LED_1
- U400 pad 3: /MCU/PE4 -> /MCU/USER_LED_2
- U400 pad 4: /MCU/PE5 -> /MCU/STATUS_LED
- U400 pad 5: /MCU/PE6 -> /MCU/USR_BUTTON
Routing:
- net /MCU/USR_BUTTON: track 0.00 -> 107.7 mm, vias 0 -> 2
- net Net-(R400-Pad1): track 96.9 -> 0.00 mm, vias 1 -> 0
- net /MCU/STATUS_LED: track 0.00 -> 84.8 mm, vias 0 -> 2
- net /MCU/USER_LED_1: track 0.00 -> 83.9 mm, vias 0 -> 2
- net /MCU/USER_LED_2: track 0.00 -> 83.6 mm, vias 0 -> 2
- net /USB/VBUS_IN: track 90.2 -> 95.2 mm
- net /MCU/SWD.~{RST}: track 122.6 -> 126.2 mm
- net /USB/CC1: track 9.26 -> 6.67 mm, vias 0 -> 2
- net GND: track 107.9 -> 110.1 mm, vias 100 -> 102
- net /MCU/USR_BTN: track 0.00 -> 1.80 mm
- net /MCU/BOOT0: track 4.83 -> 3.50 mm
- net +5V: track 9.61 -> 8.96 mm, vias 11 -> 10
- net +12V_FUSED: track 6.46 -> 5.81 mm, vias 8 -> 7
- net +12V: track 0.65 -> 0.00 mm, vias 1 -> 0
- net +3V3: track 38.4 -> 39.0 mm, vias 27 -> 28
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
Commit message: [#2] Finish layout
Parts:
- removed TP305, TP306: TestPoint, TestPoint:TestPoint_Pad_D1.0mm
- added D400: Green, PCM_JLCPCB:D_0603, F.Cu at (129.1, 125.7)
- added D401: Green, PCM_JLCPCB:D_0603, F.Cu at (130.7, 125.7)
- added D402: Green, PCM_JLCPCB:D_0603, F.Cu at (132.1, 125.7)
- added R410: 120Ω, PCM_JLCPCB:R_0402, F.Cu at (127.8, 125.7)
- added R411: 120Ω, PCM_JLCPCB:R_0402, F.Cu at (126.8, 125.7)
- added R412: 120Ω, PCM_JLCPCB:R_0402, F.Cu at (126.0, 125.7)
- added kibuzzard-67B37005: G***, kibuzzard-67B37005, F.Cu at (132.7, 121.6)
- added kibuzzard-67B37418: G***, kibuzzard-67B37418, F.Cu at (128.7, 121.6)
- added kibuzzard-67B37472: G***, kibuzzard-67B37472, F.Cu at (130.7, 121.6)
- moved TP300 46.0 mm to (128.7, 123.2)
- moved TP301 44.9 mm to (130.7, 123.2)
- moved TP302 43.9 mm to (132.7, 123.2)
- moved TP706 4.33 mm to (131.8, 140.8)
- moved TP705 3.96 mm to (129.4, 140.8)
- moved TP702 1.61 mm to (127.0, 138.6)
- moved TP704 0.99 mm to (127.0, 140.8)
- moved TP703 0.89 mm to (129.4, 138.6)
- moved TP700 0.32 mm to (133.2, 129.6)
- moved TP701 0.32 mm to (133.2, 131.6)
- moved kibuzzard-67B2198C 0.32 mm to (134.4, 129.6)
- moved kibuzzard-67B219C6 0.32 mm to (134.4, 131.6)
Connections:
- TP302 pad 1: /Power/5V_UNPROTEC -> +3V3
- U400 pad 51: /MCU/PB12 -> /CAN transceiver 2/CAN.RX
- U400 pad 52: /MCU/PB13 -> /CAN transceiver 2/CAN.TX
- U400 pad 91: /CAN transceiver 2/CAN.RX -> /MCU/PB5
- U400 pad 92: /CAN transceiver 2/CAN.TX -> /MCU/PB6
Routing:
- net +12V_FUSED: track 5.81 -> 95.1 mm, vias 7 -> 8
- net +5V: track 8.96 -> 39.5 mm, vias 10 -> 11
- net Net-(D402-Pad1): track 0.00 -> 7.31 mm
- net Net-(D401-Pad1): track 0.00 -> 4.59 mm
- net GND: track 110.1 -> 114.0 mm, vias 102 -> 101
- net +3V3: track 39.0 -> 42.6 mm, vias 28 -> 29
- net /CAN transceiver 2/CAN.RX: track 24.0 -> 20.7 mm
- net /ST-LINK/DIO: track 1.63 -> 4.11 mm
- net /ST-LINK/LED: track 19.1 -> 16.7 mm
- net /CAN transceiver 2/CAN.TX: track 23.4 -> 21.8 mm
- net /ST-LINK/CLK: track 1.67 -> 3.22 mm
- net Net-(D400-Pad1): track 0.00 -> 1.51 mm
- net /ST-LINK/STLINK-BOOT0: track 2.62 -> 3.97 mm
- net /USB/VBUS_IN: track 95.2 -> 96.0 mm
- added copper zone on B.Cu, net +12V_FUSED

Commit message: [#2] Add grid and drill origin
Parts:
- moved C301 17.8 mm to (101.4, 136.2)
- moved C302 17.8 mm to (101.4, 134.9)
- moved C305 17.8 mm to (96.1, 134.6)
- moved C309 17.8 mm to (112.2, 137.7)
- moved C310 17.8 mm to (112.2, 136.5)
- moved C402 17.8 mm to (102.9, 110.8)
- moved C404 17.8 mm to (119.0, 125.1)
- moved C405 17.8 mm to (121.3, 110.8)
- moved C410 17.8 mm to (123.1, 114.1)
- moved C413 17.8 mm to (102.9, 122.3)
- moved C501 17.8 mm to (119.1, 137.6)
- moved C601 17.8 mm to (114.5, 137.6)
- moved C707 17.8 mm to (130.0, 116.2)
- moved C900 17.8 mm to (130.4, 134.1)
- moved C902 17.8 mm to (131.3, 134.1)
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Other:
- outline, holes or cut-outs redrawn
