File: base-module.kicad_pcb (KiCad board)
At the start: 4 copper layers, 100 x 100 mm, 161 parts, among them J200 09031967921, J800 USB_C_Receptacle_USB2.0_16P, Q700 MMST3904, SW400 TL2243, U100 W25Q128, U200 PESD5V0S2BT, U300 TPS563201DDCR, U301 TPS563201DDCR, U302 CH334P, U400 STM32H750VBTx, U500 TJA1044GTK_3Z, U600 TJA1044GTK_3Z, U700 STM32F103CBTx, U801 FSUSB42UMX, U802 PESD5V0S2BT, X300 Q13FC1350000400, X400 X322512MSB4SI, Y700 8 MHz, Y900 12Mhz

Commit message: Fix revision on the silkscreen
Other:
- board text added: "PROJECT Rev. 1.0.0 TEMPLATE Rev. 1.0.1"
- board text removed: "PROJECT Rev. ${REVISION} TEMPLATE Rev. 1.0.0"
Changed lines of the file:
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@@
 			(net 198 "unconnected-(U400-PB0-Pad34)")
 			(pinfunction "PB0")
-			(pintype "bidirectional")
+			(pintype "bidirectional+no_connect")
 		)
 		(pad "35" smd roundrect
@@
 			(net 40 "unconnected-(U400-PB1-Pad35)")
 			(pinfunction "PB1")
-			(pintype "bidirectional")
+			(pintype "bidirectional+no_connect")
 		)
 		(pad "36" smd roundrect
@@
 		)
 	)
-	(gr_text "PROJECT  Rev. ${REVISION} \nTEMPLATE Rev. 1.0.0\n"
+	(gr_text "PROJECT  Rev. 1.0.0\nTEMPLATE Rev. 1.0.1\n"
 		(at 118.97 74.085001 0)
 		(layer "F.SilkS")

Commit message: [#12] Add GND testpoint
Parts:
- added TP400: TestPoint, TestPoint:TestPoint_Pad_D1.0mm, F.Cu at (126.8, 105.3)
- added kibuzzard-67E7D86B: G***, kibuzzard-67E7D86B, F.Cu at (126.8, 103.8)
Routing:
- net GND: track 114.0 -> 115.4 mm

Commit message: [#12] Change USB TVS
Parts:
- removed U200, U802: PESD5V0S2BT, Package_TO_SOT_SMD:SOT-23
- added U401: TPD2E2U06DCK, Package_TO_SOT_SMD:SOT-323_SC-70, F.Cu at (121.5, 61.8)
- added U402: TPD2E2U06DCK, Package_TO_SOT_SMD:SOT-323_SC-70, F.Cu at (132.7, 142.2)
Routing:
- net /Backplane/BACKPLANE.D-: track 9.68 -> 11.5 mm
- net GND: track 115.4 -> 114.8 mm

Commit message: [#12] Fix typo on silkscreen
Other:
- board text added: "ESD SENSITIVE DEVICE"
- board text removed: "ESD SENSETIVE DEVICE"
Changed lines of the file:
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@@
 		)
 	)
-	(gr_text "ESD SENSETIVE DEVICE"
+	(gr_text "ESD SENSITIVE DEVICE"
 		(at 102.57 127.885001 0)
 		(layer "F.SilkS")
