File: QSPI FLASH.kicad_sch (KiCad schematic)
At the start: 2 parts, among them U401 W25Q128

Commit message: [#2] Replace USB switch and power indicator LEDs
Parts:
- renumbered C425 to C100, U401 to U100
Changed lines of the file:
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@@
 		(on_board yes)
 		(dnp no)
-		(property "Reference" "#PWR0485"
+		(property "Reference" "#PWR0101"
 			(at 172.72 107.95 0)
 			(effects
@@
 			(project "base-module"
 				(path "/090a8e41-87a8-4fb1-998b-60a2c0dc4cee/e8ac371f-5104-4cae-bf76-5dce1f5864c3"
-					(reference "#PWR0485")
+					(reference "#PWR0101")
 					(unit 1)
 				)
@@
 		(dnp no)
 		(fields_autoplaced yes)
-		(property "Reference" "U401"
+		(property "Reference" "U100"
 			(at 140.97 85.09 0)
 			(effects
@@
 			(project "base-module"
 				(path "/090a8e41-87a8-4fb1-998b-60a2c0dc4cee/e8ac371f-5104-4cae-bf76-5dce1f5864c3"
-					(reference "U401")
+					(reference "U100")
 					(unit 1)
 				)
@@
 		(on_board yes)
 		(dnp no)
-		(property "Reference" "#PWR0483"
+		(property "Reference" "#PWR0102"
 			(at 115.57 109.22 0)
 			(effects
@@
 			(project ""
 				(path "/090a8e41-87a8-4fb1-998b-60a2c0dc4cee/e8ac371f-5104-4cae-bf76-5dce1f5864c3"
-					(reference "#PWR0483")
+					(reference "#PWR0102")
 					(unit 1)
 				)
@@
 		(on_board yes)
 		(dnp no)
-		(property "Reference" "#PWR0484"
+		(property "Reference" "#PWR0100"
 			(at 172.72 95.25 0)
 			(effects
@@
 			(project ""
 				(path "/090a8e41-87a8-4fb1-998b-60a2c0dc4cee/e8ac371f-5104-4cae-bf76-5dce1f5864c3"
-					(reference "#PWR0484")
+					(reference "#PWR0100")
 					(unit 1)
 				)
@@
 		(dnp no)
 		(fields_autoplaced yes)
-		(property "Reference" "C425"
+		(property "Reference" "C100"
 			(at 175.26 95.25 0)
 			(effects
@@
 			(project ""
 				(path "/090a8e41-87a8-4fb1-998b-60a2c0dc4cee/e8ac371f-5104-4cae-bf76-5dce1f5864c3"
-					(reference "C425")
+					(reference "C100")
 					(unit 1)
 				)

Commit message: [#4] Improve schematic aesthetics, color nets
Other:
- title: (none) -> ModuCard base module
Changed lines of the file:
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@@
 	(paper "A4")
 	(title_block
-		(date "2024-12-23")
+		(title "ModuCard base module")
+		(date "2025-02-18")
 		(rev "1.0.0")
 		(company "KoNaR")
 		(comment 1 "Base project authors: Dominik Pluta, Artem Horiunov")
+		(comment 2 "Project author: <author>")
 	)
 	(junction
@@
 	(bus
 		(pts
+			(xy 71.12 109.22) (xy 72.39 107.95)
+		)
+		(stroke
+			(width 0)
+			(type default)
+		)
+	)
+	(bus
+		(pts
 			(xy 72.39 105.41) (xy 72.39 107.95)
 		)
@@
 		)
 	)
+	(bus
+		(pts
+			(xy 68.58 109.22) (xy 71.12 109.22)
+		)
+		(stroke
+			(width 0)
+			(type default)
+		)
+	)
 	(wire
 		(pts
 			(xy 172.72 100.33) (xy 172.72 101.6)
-		)
-		(stroke
-			(width 0)
-			(type default)
-		)
-	)
-	(bus
-		(pts
-			(xy 69.85 107.95) (xy 72.39 107.95)
 		)
 		(stroke
@@
 	(hierarchical_label "QSPI{QSPI}"
 		(shape bidirectional)
-		(at 69.85 107.95 180)
-		(effects
-			(font
+		(at 68.58 109.22 180)
+		(effects
+			(font
