File: QSPI FLASH.kicad_sch (KiCad schematic)
At the start: 2 parts, among them U100 W25Q128

Commit message: Change MCU and update library
Changed MCU from H7 to H5 series due to programming issues with external
loader. Also updated JLCPCB components (not all tho there are still
arround 18 components to fix)
Parts:
- C100: Stock 5358037 -> 5436546
- U100: Price 0.552USD -> 0.545USD; Stock 198408 -> 69526
Other:
- title: ModuCard base module -> ModuCard BM STM32H562VGT6
Changed lines of the file:
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@@
 (kicad_sch
-	(version 20231120)
+	(version 20250114)
 	(generator "eeschema")
-	(generator_version "8.0")
+	(generator_version "9.0")
 	(paper "A4")
 	(title_block
-		(title "ModuCard base module")
-		(date "2025-02-25")
-		(rev "1.0.1")
+		(title "ModuCard BM STM32H562VGT6")
+		(date "2025-04-18")
+		(rev "1.0.0")
 		(company "KoNaR")
 		(comment 1 "Base project authors: Dominik Pluta, Artem Horiunov")
@@
 	(wire
 		(pts
-			(xy 115.57 100.33) (xy 128.27 100.33)
+			(xy 113.03 100.33) (xy 128.27 100.33)
 		)
 		(stroke
@@
 	(wire
 		(pts
-			(xy 115.57 100.33) (xy 115.57 102.87)
+			(xy 113.03 100.33) (xy 113.03 102.87)
 		)
 		(stroke
@@
 	(wire
 		(pts
-			(xy 115.57 92.71) (xy 128.27 92.71)
+			(xy 113.03 92.71) (xy 128.27 92.71)
 		)
 		(stroke
@@
 	(wire
 		(pts
-			(xy 115.57 95.25) (xy 128.27 95.25)
+			(xy 113.03 95.25) (xy 128.27 95.25)
 		)
 		(stroke
@@
 	(wire
 		(pts
-			(xy 115.57 97.79) (xy 128.27 97.79)
+			(xy 113.03 97.79) (xy 128.27 97.79)
 		)
 		(stroke
@@
 	)
 	(label "QSPI.IO2"
-		(at 115.57 97.79 0)
+		(at 113.03 97.79 0)
 		(effects
 			(font
@@
 	)
 	(label "QSPI.IO1"
-		(at 115.57 95.25 0)
+		(at 113.03 95.25 0)
 		(effects
 			(font
@@
 	)
 	(label "QSPI.CS"
-		(at 115.57 92.71 0)
+		(at 113.03 92.71 0)
 		(effects
 			(font
@@
 		(on_board yes)
 		(dnp no)
-		(property "Reference" "#PWR0101"
+		(property "Reference" "#PWR101"
 			(at 172.72 107.95 0)
 			(effects
@@
 			(project "base-module"
 				(path "/090a8e41-87a8-4fb1-998b-60a2c0dc4cee/e8ac371f-5104-4cae-bf76-5dce1f5864c3"
-					(reference "#PWR0101")
+					(reference "#PWR101")
 					(unit 1)
 				)
@@
 			)
 		)
-		(property "Stock" "198408"
-			(at 140.97 97.79 0)
-			(effects
-				(font
-					(size 1.27 1.27)
-				)
-				(hide yes)
-			)
-		)
-		(property "Price" "0.552USD"
+		(property "Stock" "69526"
+			(at 140.97 97.79 0)
+			(effects
+				(font
+					(size 1.27 1.27)
+				)
+				(hide yes)
+			)
+		)
+		(property "Price" "0.545USD"
 			(at 140.97 97.79 0)
 			(effects
@@
 	(symbol
 		(lib_id "power:GND")
-		(at 115.57 102.87 0)
+		(at 113.03 102.87 0)
 		(unit 1)
 		(exclude_from_sim no)
@@
 		(on_board yes)
 		(dnp no)
-		(property "Reference" "#PWR0102"
-			(at 115.57 109.22 0)
+		(property "Reference" "#PWR102"
+			(at 113.03 109.22 0)
 			(effects
 				(font
@@
 		)
 		(property "Value" "GND"
-			(at 115.57 106.934 0)
+			(at 113.03 106.934 0)
 			(effects
 				(font
@@
 		)
 		(property "Footprint" ""
-			(at 115.57 102.87 0)
+			(at 113.03 102.87 0)
 			(effects
 				(font
@@
 		)
 		(property "Datasheet" ""
-			(at 115.57 102.87 0)
+			(at 113.03 102.87 0)
 			(effects
 				(font
@@
 		)
 		(property "Description" "Power symbol creates a global label with name \"GND\" , ground"
-			(at 115.57 102.87 0)
+			(at 113.03 102.87 0)
 			(effects
 				(font
@@
 			(project ""
 				(path "/090a8e41-87a8-4fb1-998b-60a2c0dc4cee/e8ac371f-5104-4cae-bf76-5dce1f5864c3"
-					(reference "#PWR0102")
+					(reference "#PWR102")
 					(unit 1)
 				)
@@
 		(on_board yes)
 		(dnp no)
-		(property "Reference" "#PWR0100"
+		(property "Reference" "#PWR100"
 			(at 172.72 95.25 0)
 			(effects
@@
 			(project ""
 				(path "/090a8e41-87a8-4fb1-998b-60a2c0dc4cee/e8ac371f-5104-4cae-bf76-5dce1f5864c3"
-					(reference "#PWR0100")
+					(reference "#PWR100")
 					(unit 1)
 				)
@@
 			)
 		)
-		(property "Stock" "5358037"
+		(property "Stock" "5436546"
 			(at 172.72 96.52 0)
 			(effects

Commit message: [1] Change MCU schematic ERC pass
Changed lines of the file:
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@@
+		)
+	)
+	(wire
+		(pts
+			(xy 172.72 86.36) (xy 172.72 92.71)
+		)
+		(stroke
+			(width 0)
+			(type default)
 		)
 	)
@@
 	(wire
 		(pts
-			(xy 172.72 92.71) (xy 172.72 91.44)
+			(xy 172.72 104.14) (xy 172.72 100.33)
 		)
 		(stroke
@@
 		(pts
 			(xy 68.58 109.22) (xy 71.12 109.22)
-		)
-		(stroke
-			(width 0)
-			(type default)
-		)
-	)
-	(wire
-		(pts
-			(xy 172.72 100.33) (xy 172.72 101.6)
 		)
 		(stroke
@@
 	(symbol
 		(lib_id "power:GND")
-		(at 172.72 101.6 0)
+		(at 113.03 102.87 0)
 		(unit 1)
 		(exclude_from_sim no)
@@
 		(on_board yes)
 		(dnp no)
-		(property "Reference" "#PWR101"
-			(at 172.72 107.95 0)
+		(fields_autoplaced yes)
+		(property "Reference" "#PWR0402"
+			(at 113.03 109.22 0)
 			(effects
 				(font
@@
 		)
 		(property "Value" "GND"
-			(at 172.72 105.41 0)
+			(at 113.03 107.95 0)
 			(effects
 				(font
@@
 		)
 		(property "Footprint" ""
-			(at 172.72 101.6 0)
+			(at 113.03 102.87 0)
 			(effects
 				(font
@@
 		)
 		(property "Datasheet" ""
-			(at 172.72 101.6 0)
+			(at 113.03 102.87 0)
 			(effects
 				(font
@@
 		)
 		(property "Description" "Power symbol creates a global label with name \"GND\" , ground"
-			(at 172.72 101.6 0)
+			(at 113.03 102.87 0)
 			(effects
 				(font
@@
 			(project "base-module"
 				(path "/090a8e41-87a8-4fb1-998b-60a2c0dc4cee/e8ac371f-5104-4cae-bf76-5dce1f5864c3"
-					(reference "#PWR101")
+					(reference "#PWR0402")
 					(unit 1)
 				)
@@
 	(symbol
 		(lib_id "power:GND")
-		(at 113.03 102.87 0)
+		(at 172.72 104.14 0)
 		(unit 1)
 		(exclude_from_sim no)
@@
 		(on_board yes)
 		(dnp no)
-		(property "Reference" "#PWR102"
-			(at 113.03 109.22 0)
+		(fields_autoplaced yes)
+		(property "Reference" "#PWR0401"
+			(at 172.72 110.49 0)
 			(effects
 				(font
@@
 		)
 		(property "Value" "GND"
-			(at 113.03 106.934 0)
+			(at 172.72 109.22 0)
 			(effects
 				(font
@@
 		)
 		(property "Footprint" ""
-			(at 113.03 102.87 0)
+			(at 172.72 104.14 0)
 			(effects
 				(font
@@
 		)
 		(property "Datasheet" ""
-			(at 113.03 102.87 0)
+			(at 172.72 104.14 0)
 			(effects
 				(font
@@
 		)
 		(property "Description" "Power symbol creates a global label with name \"GND\" , ground"
-			(at 113.03 102.87 0)
+			(at 172.72 104.14 0)
 			(effects
 				(font
@@
 			(project ""
 				(path "/090a8e41-87a8-4fb1-998b-60a2c0dc4cee/e8ac371f-5104-4cae-bf76-5dce1f5864c3"
-					(reference "#PWR102")
+					(reference "#PWR0401")
 					(unit 1)
 				)
@@
 	(symbol
 		(lib_id "power:+3V3")
-		(at 172.72 91.44 0)
+		(at 172.72 86.36 0)
 		(unit 1)
 		(exclude_from_sim no)
@@
 		(dnp no)
 		(property "Reference" "#PWR100"
-			(at 172.72 95.25 0)
+			(at 172.72 90.17 0)
 			(effects
 				(font
@@
 		)
 		(property "Value" "+3V3"
-			(at 172.466 87.63 0)
+			(at 172.466 82.55 0)
 			(effects
 				(font
@@
 		)
 		(property "Footprint" ""
-			(at 172.72 91.44 0)
+			(at 172.72 86.36 0)
 			(effects
 				(font
@@
 		)
 		(property "Datasheet" ""
-			(at 172.72 91.44 0)
+			(at 172.72 86.36 0)
 			(effects
 				(font
@@
 		)
 		(property "Description" "Power symbol creates a global label with name \"+3V3\""
-			(at 172.72 91.44 0)
-			(effects
-				(font
+			(at 172.72 86.36 0)
+			(effects
+				(font

Commit message: [REV2] board finshed, schematics and leyout
Other:
- title: ModuCard BM STM32H562VGT6 -> ModuCard nav module
Changed lines of the file:
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@@
 	(paper "A4")
 	(title_block
-		(title "ModuCard BM STM32H562VGT6")
-		(date "2025-04-18")
+		(title "ModuCard nav module")
+		(date "2025-04-20")
 		(rev "1.1.0")
 		(company "KoNaR")
 		(comment 1 "Base project authors: Dominik Pluta, Artem Horiunov")
-		(comment 2 "Project author: <author>")
+		(comment 2 "Project author: Patryk Dudziński")
 	)
 	(junction
