File: ModuCard-navigation-module.kicad_pcb (KiCad board)
At the start: 4 copper layers, 100 x 100 mm, 221 parts, among them J1100 Conn_Coaxial, J200 09031967921, J400 Adafruit garbage connector, J800 USB_C_Receptacle_USB2.0_16P, Q700 MMST3904, U100 W25Q128, U1100 ZED-F9P, U1300 BMP280, U300 TPS563200, U301 TPS563200, U302 CH334P, U400 ICM-20948, U401 TPD2E2U06DCK, U402 TPD2E2U06DCK, U403 STM32H562VGTx, U500 TJA1044GTK_3Z, U600 TJA1044GTK_3Z, U700 STM32F103CBTx, U801 FSUSB42UMX, X300 Q13FC1350000400, Y400 ASE-xxxMHz, Y700 Crystal_GND24, Y900 Crystal_GND24

Commit message: addd nice silkinfo
Parts:
- removed kibuzzard-67B69E78: G***, kibuzzard-67B69E78
- removed kibuzzard-68057AEC: G***, kibuzzard-68057AEC
- added kibuzzard-6807DF1D: G***, kibuzzard-6807DF1D, F.Cu at (61.8, 124.7)
- added kibuzzard-6807DFFB: G***, kibuzzard-6807DFFB, F.Cu at (60.6, 100.8)
- added kibuzzard-6807E003: G***, kibuzzard-6807E003, F.Cu at (50.6, 95.3)

Commit message: update for imu
Parts:
- removed kibuzzard-6807DFFB: G***, kibuzzard-6807DFFB
- removed kibuzzard-6807E003: G***, kibuzzard-6807E003
- added kibuzzard-68091D50: G***, kibuzzard-68091D50, F.Cu at (50.6, 95.3)
- moved kibuzzard-68057139 1.41 mm to (54.4, 59.3)
Routing:
- net /IMU/IMU_FSYNC: track 87.5 -> 88.3 mm
Other:
- board text added: "Are you shure about that?"
- board text added: "Is your debuger not working?"

Commit message: fixed 5v line and drc
Routing:
- net +5V: track 131.8 -> 115.2 mm
Changed lines of the file:
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@@
 	)
 	(segment
-		(start 49.709999 137.025)
+		(start 95.060767 129.285001)
+		(end 95.071768 129.274)
+		(width 0.3)
+		(layer "B.Cu")
+		(net 6)
+	)
+	(segment
+		(start 103.471768 133.976)
+		(end 103.726 133.976)
+		(width 0.3)
+		(layer "B.Cu")
+		(net 6)
+	)
+	(segment
+		(start 99.035001 129.285001)
+		(end 103.149 133.399)
+		(width 0.3)
+		(layer "B.Cu")
+		(net 6)
+	)
+	(segment
+		(start 103.726 133.976)
 		(end 106.775 137.025)
 		(width 0.3)
@@
 	)
 	(segment
-		(start 52.93 106.685001)
-		(end 50.17 106.685001)
+		(start 55.27 127.085001)
+		(end 57.47 129.285001)
 		(width 0.3)
 		(layer "B.Cu")
@@
 	)
 	(segment
-		(start 50.17 106.685001)
-		(end 45.87 110.985001)
+		(start 95.539233 129.285001)
+		(end 99.035001 129.285001)
 		(width 0.3)
 		(layer "B.Cu")
@@
 	)
 	(segment
-		(start 45.87 110.985001)
-		(end 45.87 133.185001)
+		(start 95.071768 129.274)
+		(end 95.528232 129.274)
+		(width 0.3)
+		(layer "B.Cu")
+		(net 6)
+	)
+	(segment
+		(start 95.528232 129.274)
+		(end 95.539233 129.285001)
+		(width 0.3)
+		(layer "B.Cu")
+		(net 6)
+	)
+	(segment
+		(start 55.27 110.985001)
+		(end 55.27 127.085001)
+		(width 0.3)
+		(layer "B.Cu")
+		(net 6)
+	)
+	(segment
+		(start 57.47 129.285001)
+		(end 95.060767 129.285001)
 		(width 0.3)
 		(layer "B.Cu")
@@
 	)
 	(segment
-		(start 45.87 133.185001)
-		(end 49.709999 137.025)
+		(start 103.149 133.653232)
+		(end 103.471768 133.976)
 		(width 0.3)
 		(layer "B.Cu")
+		(net 6)
+	)
+	(segment
+		(start 53.47 109.185001)
+		(end 55.27 110.985001)
+		(width 0.3)
+		(layer "B.Cu")
+		(net 6)
+	)
+	(segment
+		(start 53.47 106.685001)
+		(end 53.47 109.185001)
+		(width 0.3)
+		(layer "B.Cu")
+		(net 6)
+	)
+	(segment
+		(start 103.149 133.399)
+		(end 103.149 133.653232)
+		(width 0.3)
+		(layer "B.Cu")

Commit message: [mcu] changed mcu from 562VGT6  to 563VGT6
Parts:
- U403: value STM32H562VGTx -> STM32H563VGTx
Changed lines of the file:
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@@
 			)
 		)
-		(property "Value" "STM32H562VGTx"
+		(property "Value" "STM32H563VGTx"
 			(at 0 9.42 90)
 			(layer "F.Fab")
@@
 			)
 		)
-		(property "Datasheet" "https://www.st.com/resource/en/datasheet/stm32h562vg.pdf"
+		(property "Datasheet" "https://www.st.com/resource/en/datasheet/stm32h563vg.pdf"
 			(at 0 0 90)
 			(layer "F.Fab")
@@
 			)
 		)
-		(property "Description" "STMicroelectronics Arm Cortex-M33 MCU, 1024KB flash, 640KB RAM, 80 GPIO, LQFP100"
+		(property "Description" "STMicroelectronics Arm Cortex-M33 MCU, 1024KB flash, 640KB RAM, 250 MHz, 1.62-3.6V, 80 GPIO, LQFP100"
 			(at 0 0 90)
 			(layer "F.Fab")
@@
 			(keep_text_aligned yes)
 		)
-		(gr_text "88,9000 mm"
+		(gr_text "88.9000 mm"
 			(at 89.37 44.875001 0)
 			(layer "Cmts.User")
@@
 			(keep_text_aligned yes)
 		)
-		(gr_text "3,5600 mm"
+		(gr_text "3.5600 mm"
 			(at 38.383656 53.083348 -89.83905722)
 			(layer "Cmts.User")
@@
 			(keep_text_aligned yes)
 		)
-		(gr_text "5,5500 mm"
+		(gr_text "5.5500 mm"
 			(at 42.1092 44.920599 0.2064703838)
 			(layer "Cmts.User")
@@
 			(keep_text_aligned yes)
 		)
-		(gr_text "100,0000 mm"
+		(gr_text "100.0000 mm"
 			(at 89.37 167.215 0)
 			(layer "Cmts.User")
@@
 			(keep_text_aligned yes)
 		)
-		(gr_text "3,5600 mm"
+		(gr_text "3.5600 mm"
 			(at 140.53 53.065001 90)
 			(layer "Cmts.User")
@@
 			(keep_text_aligned yes)
 		)
-		(gr_text "100,0000 mm"
+		(gr_text "100.0000 mm"
 			(at 146.06 104.285001 90)
 			(layer "Cmts.User")
@@
 			(keep_text_aligned yes)
 		)
-		(gr_text "5,5500 mm"
+		(gr_text "5.5500 mm"
 			(at 136.577069 44.888119 0.103235527)
 			(layer "Cmts.User")
