File: ModuCard-navigation-module.kicad_pcb (KiCad board)
At the start: 4 copper layers, 100 x 100 mm, 221 parts, among them J1100 Conn_Coaxial, J200 09031967921, J400 Adafruit garbage connector, J800 USB_C_Receptacle_USB2.0_16P, Q700 MMST3904, U100 W25Q128, U1100 ZED-F9P, U1300 BMP280, U300 TPS563200, U301 TPS563200, U302 CH334P, U400 ICM-20948, U401 TPD2E2U06DCK, U402 TPD2E2U06DCK, U403 STM32H563VGTx, U500 TJA1044GTK_3Z, U600 TJA1044GTK_3Z, U700 STM32F103CBTx, U801 FSUSB42UMX, X300 Q13FC1350000400, Y400 ASE-xxxMHz, Y700 Crystal_GND24, Y900 Crystal_GND24

Commit message: [imu] added ligic lever shifter and 1.8V power supply
Parts:
- added C407: 10uF, PCM_JLCPCB:C_0603, F.Cu at (54.1, 99.8)
- added C408: 100nF, PCM_JLCPCB:C_0402, F.Cu at (55.6, 98.0)
- added C409: 100nF, PCM_JLCPCB:C_0402, F.Cu at (60.4, 100.5)
- added C411: 1uF, PCM_JLCPCB:C_0402, F.Cu at (59.5, 100.5)
- added IC400: RT9013-18GB, kicad-footprints:SOT94P279X130-5N, F.Cu at (56.9, 100.2)
- added Q400: BSS138, Package_TO_SOT_SMD:SOT-23, F.Cu at (64.1, 98.1)
- added Q401: BSS138, Package_TO_SOT_SMD:SOT-23, F.Cu at (64.1, 94.6)
- added R421: 4.7kΩ, PCM_JLCPCB:R_0402, F.Cu at (61.8, 98.2)
- added R422: 4.7kΩ, PCM_JLCPCB:R_0402, F.Cu at (65.6, 96.6)
- added R424: 4.7kΩ, PCM_JLCPCB:R_0402, F.Cu at (66.5, 94.2)
- added R425: 0Ω, PCM_JLCPCB:R_0402, F.Cu at (61.3, 100.5)
- added R426: 4.7kΩ, PCM_JLCPCB:R_0402, F.Cu at (61.8, 95.3)
- added R427: 0Ω, PCM_JLCPCB:R_0402, F.Cu at (62.2, 100.5)
- moved U1300 5.78 mm to (68.7, 96.7)
- moved C1302 5.78 mm to (68.0, 94.8)
- moved R414 5.78 mm to (67.0, 98.5)
- moved C1300 5.78 mm to (70.9, 96.9)
- moved C1301 5.78 mm to (69.9, 94.8)
- moved R413 5.78 mm to (68.9, 98.5)
- moved C1107 4.12 mm to (55.2, 96.0), turned to -90 degrees
Connections:
- R420 pad 1: +3V3 -> /IMU/VDDIO
- U400 pad 22: +3V3 -> /IMU/VDDIO
- U400 pad 23: /Barometer/BAROMETR_I2C.SCL -> /IMU/L_SCL
- U400 pad 24: /Barometer/BAROMETR_I2C.SDA -> /IMU/L_SDA
- U400 pad 8: +3V3 -> /IMU/VDDIO
Routing:
- net +3V3: track 76.8 -> 84.1 mm, vias 47 -> 49
- net GND: track 329.9 -> 334.9 mm, vias 206 -> 209
- net /Barometer/BAROMETR_I2C.SDA: track 91.3 -> 96.3 mm
- net /IMU/L_SDA: track 0.00 -> 4.61 mm
- net /IMU/L_SCL: track 0.00 -> 4.40 mm
- net /IMU/VDDIO_1V8: track 0.00 -> 3.94 mm
- net /Barometer/BAROMETR_I2C.SCL: track 92.9 -> 96.1 mm
- net /IMU/VDDIO: track 0.00 -> 1.86 mm
- added copper zone on F.Cu, net /IMU/VDDIO

Commit message: changed shity resisrto to smaller one on LEDs  fixed level shifting
Parts:
- removed R400: 1.2kΩ, PCM_JLCPCB:R_0402
- removed R425, R427: 0Ω, PCM_JLCPCB:R_0402
- removed R707, R713: 10kΩ, PCM_JLCPCB:R_0402
- added R423: 220Ω, PCM_JLCPCB:R_0402, F.Cu at (113.6, 61.2)
- added R428: 220Ω, PCM_JLCPCB:R_0402, F.Cu at (114.5, 61.2)
- added R429: 220Ω, PCM_JLCPCB:R_0402, F.Cu at (125.3, 109.4)
- R409: value 100Ω -> 220Ω
- moved R409 49.0 mm to (123.3, 109.4), turned to 0 degrees
Connections:
- C409 pad 1: /IMU/VDDIO_1V8 -> /IMU/VDDIO
- C411 pad 1: /IMU/VDDIO_1V8 -> /IMU/VDDIO
- IC400 pad 5: /IMU/VDDIO_1V8 -> /IMU/VDDIO
- R409 pad 2: Net-(LED301-Pad3) -> Net-(D700-Pad2)
Routing:
- net /IMU/VDDIO_1V8: track 3.94 -> 0.00 mm
- net +3V3: track 84.1 -> 83.2 mm, vias 49 -> 48
Other:
- board text added: "PROJECT Rev. 2.1.0 TEMPLATE Rev. 2.0.0"
- board text removed: "PROJECT Rev. 2.0.0 TEMPLATE Rev. 2.0.0"
