File: IMU.kicad_sch (KiCad schematic)
At the start: 11 parts, among them J400 Adafruit garbage connector, U400 ICM-20948

Commit message: [imu] added ligic lever shifter and 1.8V power supply
Parts:
- added C407: 10uF, PCM_JLCPCB:C_0603, symbol PCM_JLCPCB-Capacitors:0603,10uF,(2)
- added C408, C409: 100nF, PCM_JLCPCB:C_0402, symbol PCM_JLCPCB-Capacitors:0402,100nF,(2)
- added C411: 1uF, PCM_JLCPCB:C_0402, symbol PCM_JLCPCB-Capacitors:0402,1uF
- added IC400: RT9013-18GB, kicad-footprints:SOT94P279X130-5N, symbol RT9013-18GB:RT9013-18GB
- added Q400, Q401: BSS138, Package_TO_SOT_SMD:SOT-23, symbol Transistor_FET:BSS138
- added R421, R422, R424, R426: 4.7kΩ, PCM_JLCPCB:R_0402, symbol PCM_JLCPCB-Resistors:0402,4.7kΩ
- added R425, R427: 0Ω, PCM_JLCPCB:R_0402, symbol PCM_JLCPCB-Resistors:0402,0Ω
- R419: now not fitted
Connections:
- net +3V3: now also C407.1, C408.1, IC400.1 (VIN), IC400.3 (EN), R422.1, R424.1, R427.1; no longer R420.1, U400.22 (~{CS}), U400.8 (VDDIO)
- net GND: now also C407.2, C408.2, C409.2, C411.2, IC400.2 (GND)
- net IMU_I2C.SCL: now also Q400.3 (D), R422.2; no longer U400.23 (SCL/SCLK)
- net IMU_I2C.SDA: now also Q401.3 (D), R424.2; no longer U400.24 (SDA/SDI)
- new net L_SCL: Q400.2 (S), R421.2, U400.23 (SCL/SCLK)
- new net L_SDA: Q401.2 (S), R426.2, U400.24 (SDA/SDI)
- new net VDDIO: Q400.1 (G), Q401.1 (G), R420.1, R421.1, R425.2, R426.1, R427.2, U400.22 (~{CS}), U400.8 (VDDIO)
- new net VDDIO_1V8: C409.1, C411.1, IC400.5 (VOUT), R425.1
Other:
- moved on the sheet: C1106, C1107, C1108, H400, H401, H402, H403, J400, R420, U400

Commit message: changed shity resisrto to smaller one on LEDs  fixed level shifting
Parts:
- removed R425, R427: 0Ω, PCM_JLCPCB:R_0402, symbol PCM_JLCPCB-Resistors:0402,0Ω
Connections:
- net VDDIO_1V8 is gone; now on net VDDIO: C409.1, C411.1, IC400.5 (VOUT)
